File: PCB/7SegClock.sch (KiCad schematic (older format))
At the start: 4 parts

Commit message: Schematic work.
Parts:
- removed U?: 24LC256, symbol 24C16
- added C?: 10nF, symbol C
- added Q?: NPN, Transistors_SMD:sot23, symbol NPN
- added R? (x2): 10K, symbol R
- added U2: 24LC256, SMD_Packages:SOIC-8-N, symbol 24LC256
- added U3: FT232RL, symbol FT232RL
- CON1: renamed from CON?; footprint (none) -> Connect:USB_Mini-B
- U1: renamed from U?; footprint (none) -> SMD_Packages:TQFP-44
- X1: renamed from X?; footprint (none) -> Crystals_Oscillators_SMD:Q_49U3HMS
Connections:
- net labels added: +3V3, +5V, DTR
- wire segments 18 -> 72
- no-connect marks 0 -> 3
Other:
- moved on the sheet: CON1, U1, X1

Commit message: Updated schematic.
Connections:
- net +3V3: now also U2.8 (VCC)
- net GND: now also U1.6 (BOEn)
Changed lines of the file:
@@
 $EndDescr
-$Comp
-L GND #PWR1
-U 1 1 549F470E
-P 1550 900
-F 0 "#PWR1" H 1550 650 60  0001 C CNN
-F 1 "GND" H 1550 750 60  0000 C CNN
-F 2 "" H 1550 900 60  0000 C CNN
-F 3 "" H 1550 900 60  0000 C CNN
-	1    1550 900
-	-1   0    0    1
-$EndComp
 $Comp
 L P8X32A U1
@@
 	1    0    0    -1
 $EndComp
-Text GLabel 1550 1000 3    60   Input ~ 0
-GND
 $Comp
 L CRYSTAL X1
@@
 L +3V3 #PWR?
 U 1 1 549F87F3
-P 2500 2000
-F 0 "#PWR?" H 2500 1850 60  0001 C CNN
-F 1 "+3V3" H 2500 2140 60  0000 C CNN
-F 2 "" H 2500 2000 60  0000 C CNN
-F 3 "" H 2500 2000 60  0000 C CNN
-	1    2500 2000
-	-1   0    0    1
+P 2500 1700
+F 0 "#PWR?" H 2500 1550 60  0001 C CNN
+F 1 "+3V3" H 2500 1840 60  0000 C CNN
+F 2 "" H 2500 1700 60  0000 C CNN
+F 3 "" H 2500 1700 60  0000 C CNN
+	1    2500 1700
+	1    0    0    -1
 $EndComp
 $Comp
@@
 $EndComp
 Wire Wire Line
-	1550 900  1550 1000
-Wire Wire Line
 	3800 4400 4050 4400
 Wire Wire Line
@@
 Wire Wire Line
 	3200 1850 2500 1850
-Wire Wire Line
-	2500 1850 2500 2000
 Wire Wire Line
 	2900 2000 2900 1850
@@
 	1    0    0    -1
 $EndComp
+Wire Wire Line
+	3000 4400 3000 4800
+$Comp
+L GND #PWR?
+U 1 1 549F9839
+P 3000 4800
+F 0 "#PWR?" H 3000 4550 60  0001 C CNN
+F 1 "GND" H 3000 4650 60  0000 C CNN
+F 2 "" H 3000 4800 60  0000 C CNN
+F 3 "" H 3000 4800 60  0000 C CNN
+	1    3000 4800
+	1    0    0    -1
+$EndComp
+$Comp
+L +3V3 #PWR?
+U 1 1 549F993F
+P 4100 5450
+F 0 "#PWR?" H 4100 5300 60  0001 C CNN
+F 1 "+3V3" H 4100 5590 60  0000 C CNN
+F 2 "" H 4100 5450 60  0000 C CNN
+F 3 "" H 4100 5450 60  0000 C CNN
+	1    4100 5450
+	1    0    0    -1
+$EndComp
+Wire Wire Line
+	4100 5450 4100 5550
+Wire Wire Line
+	4100 5550 3950 5550
+Wire Wire Line
+	2500 1850 2500 1700
 $EndSCHEMATC

Commit message: Worked on schematic.
Parts:
- added D? (x2): LED, symbol LED
- added R?: 1K, Resistors_SMD:R_0805_HandSoldering, symbol R
Connections:
- net +5V: now also R?.2
- net at U3.22 (RXLED): now also D?.2 (K)
- net at U3.23 (TXLED): now also D?.2 (K)
- new net: D?.1 (A), D?.1 (A), R?.1
Changed lines of the file:
@@
 	1    0    0    -1
 $EndComp
-Wire Wire Line
-	3800 4400 4050 4400
-Wire Wire Line
-	4050 4400 4050 4750
-Wire Wire Line
-	3700 4400 3450 4400
-Wire Wire Line
-	3450 4400 3450 4750
-Wire Wire Line
-	4200 2650 4350 2650
-Wire Wire Line
-	4200 2750 4350 2750
-Wire Wire Line
-	2750 5550 2600 5550
-Wire Wire Line
-	2600 5550 2600 5950
-Wire Wire Line
-	2750 5850 2600 5850
-Connection ~ 2600 5850
-Wire Wire Line
-	2750 5750 2600 5750
-Connection ~ 2600 5750
-Wire Wire Line
-	2750 5650 2600 5650
-Connection ~ 2600 5650
-Wire Wire Line
-	4150 5750 3950 5750
-Wire Wire Line
-	4150 5850 3950 5850
-Wire Wire Line
-	3950 5650 4450 5650
-Wire Wire Line
-	4450 5650 4450 5950
-Wire Wire Line
-	5450 3400 4950 3400
-Wire Wire Line
-	4950 3400 4950 2450
-Wire Wire Line
-	4950 2450 4200 2450
-Wire Wire Line
-	4200 2550 4850 2550
-Wire Wire Line
-	4850 2550 4850 3500
-Wire Wire Line
-	4850 3500 5450 3500
-Wire Wire Line
-	6800 3450 6950 3450
-Wire Wire Line
-	6950 3450 6950 4050
-Wire Wire Line
-	6800 3550 6950 3550
-Connection ~ 6950 3550
-Wire Wire Line
-	6800 3650 6950 3650
-Connection ~ 6950 3650
-Wire Wire Line
-	6800 3750 6950 3750
-Connection ~ 6950 3750
-Wire Wire Line
-	6800 3850 6950 3850
-Connection ~ 6950 3850
-Wire Wire Line
-	5450 3100 5300 3100
-Wire Wire Line
-	5300 3100 5300 3200
-Wire Wire Line
-	5300 3200 5450 3200
-Wire Wire Line
-	3500 2000 3500 1850
-Wire Wire Line
-	3500 1850 4200 1850
-Wire Wire Line
-	4200 1850 4200 2000
-Wire Wire Line
-	3600 2000 3600 1850
-Connection ~ 3600 1850
-Wire Wire Line
-	3700 2000 3700 1850
-Connection ~ 3700 1850
-Wire Wire Line
-	3800 2000 3800 1850
-Connection ~ 3800 1850
-Wire Wire Line
-	5500 4400 5500 4500
-Wire Wire Line
-	5500 4500 5650 4500
-Wire Wire Line
-	5650 4600 5300 4600
-Wire Wire Line
-	5300 4600 5300 3850
-Wire Wire Line
-	5300 3850 5450 3850
-Wire Wire Line
-	5450 3750 5200 3750
-Wire Wire Line
-	5200 3750 5200 4700
-Wire Wire Line
-	5200 4700 5650 4700
-Wire Wire Line
-	6650 4500 6800 4500
-Wire Wire Line
-	6800 4500 6800 5050
-Wire Wire Line
-	6650 4900 6800 4900
-Connection ~ 6800 4900
-Wire Wire Line
-	6650 4800 6800 4800
-Connection ~ 6800 4800
-Wire Wire Line
-	6650 4600 6800 4600
-Connection ~ 6800 4600
-Wire Wire Line
-	5650 4900 5500 4900
-Wire Wire Line
-	5500 4900 5500 5050
-Wire Wire Line
-	5300 2450 5300 2650
-Wire Wire Line
-	5300 2650 5450 2650
-Wire Wire Line
-	5450 2550 5300 2550
-Connection ~ 5300 2550
-Wire Wire Line
-	3200 2000 3200 1850
-Wire Wire Line
-	3200 1850 2500 1850
-Wire Wire Line
-	2900 2000 2900 1850
-Connection ~ 2900 1850
-Wire Wire Line
-	3000 2000 3000 1850
-Connection ~ 3000 1850
-Wire Wire Line
-	3100 2000 3100 1850
-Connection ~ 3100 1850
-Wire Wire Line
-	7250 2750 6800 2750
-Wire Wire Line
-	7650 2750 8000 2750
-Wire Wire Line
-	8300 2950 8300 3700
-Wire Wire Line
-	8300 3550 7850 3550
-Wire Wire Line
-	7850 3550 7850 3450
-Wire Wire Line
-	7850 2950 7850 2750
-Connection ~ 7850 2750
-Connection ~ 8300 3550
 $Comp
 L GND #PWR?
@@
 Text GLabel 3100 4550 3    50   Input ~ 0
 DTR
-Wire Wire Line
-	3100 4400 3100 4550
 Text GLabel 8300 2250 1    50   Input ~ 0
 DTR
-Wire Wire Line
-	8300 2250 8300 2550
 $Comp
 L R R?
@@
 	1    0    0    -1
 $EndComp
-Wire Wire Line
-	7850 2350 7850 2450
-Wire Wire Line
-	7850 2450 8300 2450
-Connection ~ 8300 2450
-Wire Wire Line
-	7850 1850 7850 1700
 $Comp
 L +3V3 #PWR?
@@
 	1    0    0    -1
 $EndComp
-Wire Wire Line
-	3000 4400 3000 4800
 $Comp
 L GND #PWR?
@@
 	1    0    0    -1
 $EndComp
+$Comp
+L LED D?
+U 1 1 549F9252
+P 7300 3650
+F 0 "D?" H 7300 3750 50  0000 C CNN
+F 1 "LED" H 7300 3550 50  0000 C CNN
+F 2 "" H 7300 3650 60  0000 C CNN
+F 3 "" H 7300 3650 60  0000 C CNN
+	1    7300 3650
+	0    -1   -1   0
+$EndComp
+$Comp
+L LED D?
+U 1 1 549F92C9
+P 7600 3650
+F 0 "D?" H 7600 3750 50  0000 C CNN
+F 1 "LED" H 7600 3550 50  0000 C CNN
+F 2 "" H 7600 3650 60  0000 C CNN
+F 3 "" H 7600 3650 60  0000 C CNN
+	1    7600 3650
+	0    -1   -1   0
+$EndComp
+$Comp
+L R R?
+U 1 1 549F945E
+P 7450 4300
+F 0 "R?" V 7530 4300 40  0000 C CNN
+F 1 "1K" V 7457 4301 40  0000 C CNN
+F 2 "Resistors_SMD:R_0805_HandSoldering" V 7380 4300 30  0001 C CNN
+F 3 "" H 7450 4300 30  0000 C CNN
+	1    7450 4300
+	1    0    0    -1
+$EndComp
+Wire Wire Line
+	3800 4400 4050 4400
+Wire Wire Line
+	4050 4400 4050 4750
+Wire Wire Line
+	3700 4400 3450 4400
+Wire Wire Line
+	3450 4400 3450 4750
+Wire Wire Line
+	4200 2650 4350 2650
+Wire Wire Line
+	4200 2750 4350 2750
+Wire Wire Line
+	2750 5550 2600 5550
+Wire Wire Line
+	2600 5550 2600 5950
+Wire Wire Line
+	2750 5850 2600 5850
+Connection ~ 2600 5850
+Wire Wire Line
+	2750 5750 2600 5750
+Connection ~ 2600 5750
+Wire Wire Line
+	2750 5650 2600 5650
+Connection ~ 2600 5650
+Wire Wire Line
+	4150 5750 3950 5750
+Wire Wire Line
+	4150 5850 3950 5850
+Wire Wire Line
+	3950 5650 4450 5650
+Wire Wire Line
+	4450 5650 4450 5950
+Wire Wire Line
+	6800 3450 6950 3450
+Wire Wire Line
+	6950 3450 6950 4050
+Wire Wire Line
+	6800 3550 6950 3550
+Connection ~ 6950 3550
+Wire Wire Line
+	6800 3650 6950 3650
+Connection ~ 6950 3650
+Wire Wire Line
+	6800 3750 6950 3750
+Connection ~ 6950 3750
+Wire Wire Line
+	6800 3850 6950 3850
+Connection ~ 6950 3850
+Wire Wire Line
+	5450 3100 5300 3100
+Wire Wire Line
+	5300 3100 5300 3200
+Wire Wire Line
+	5300 3200 5450 3200
+Wire Wire Line
+	3500 2000 3500 1850
+Wire Wire Line
+	3500 1850 4200 1850
+Wire Wire Line
+	4200 1850 4200 2000
+Wire Wire Line
+	3600 2000 3600 1850
+Connection ~ 3600 1850
+Wire Wire Line
+	3700 2000 3700 1850
+Connection ~ 3700 1850
+Wire Wire Line
+	3800 2000 3800 1850
+Connection ~ 3800 1850
+Wire Wire Line
+	5500 4400 5500 4500
+Wire Wire Line
+	5500 4500 5650 4500
+Wire Wire Line
+	5650 4600 5300 4600
+Wire Wire Line
+	5300 4600 5300 3850
+Wire Wire Line
+	5300 3850 5450 3850
+Wire Wire Line
+	5450 3750 5200 3750
+Wire Wire Line
+	5200 3750 5200 4700
+Wire Wire Line
+	5200 4700 5650 4700
+Wire Wire Line
+	6650 4500 6800 4500
+Wire Wire Line
+	6800 4500 6800 5050
+Wire Wire Line
+	6650 4900 6800 4900
+Connection ~ 6800 4900
+Wire Wire Line
+	6650 4800 6800 4800
+Connection ~ 6800 4800
+Wire Wire Line
+	6650 4600 6800 4600
+Connection ~ 6800 4600
+Wire Wire Line
+	5650 4900 5500 4900
+Wire Wire Line
+	5500 4900 5500 5050
+Wire Wire Line
+	5300 2450 5300 2650
+Wire Wire Line
+	5300 2650 5450 2650
+Wire Wire Line
+	5450 2550 5300 2550
+Connection ~ 5300 2550
+Wire Wire Line
+	3200 2000 3200 1850
+Wire Wire Line
+	3200 1850 2500 1850
+Wire Wire Line
+	2900 2000 2900 1850
+Connection ~ 2900 1850
+Wire Wire Line
+	3000 2000 3000 1850
+Connection ~ 3000 1850
+Wire Wire Line
+	3100 2000 3100 1850
+Connection ~ 3100 1850
+Wire Wire Line
+	7250 2750 6800 2750
+Wire Wire Line
+	7650 2750 8000 2750
+Wire Wire Line
+	8300 2950 8300 3700
+Wire Wire Line
+	8300 3550 7850 3550
+Wire Wire Line
+	7850 3550 7850 3450
+Wire Wire Line
+	7850 2950 7850 2750
+Connection ~ 7850 2750
+Connection ~ 8300 3550
+Wire Wire Line
+	3100 4400 3100 4550
+Wire Wire Line
+	8300 2250 8300 2550
+Wire Wire Line
+	7850 2350 7850 2450
+Wire Wire Line
+	7850 2450 8300 2450
+Connection ~ 8300 2450
+Wire Wire Line
+	7850 1850 7850 1700
+Wire Wire Line
+	3000 4400 3000 4800
 Wire Wire Line
 	4100 5450 4100 5550
@@
 Wire Wire Line
 	2500 1850 2500 1700
+Wire Wire Line
+	6800 3100 7600 3100
+Wire Wire Line
+	7600 3100 7600 3450
+Wire Wire Line
+	6800 3200 7300 3200
+Wire Wire Line
+	7300 3200 7300 3450
+Wire Wire Line
+	7300 3850 7300 3950
+Wire Wire Line
+	7300 3950 7600 3950
+Wire Wire Line
+	7600 3950 7600 3850
+Wire Wire Line
+	7450 4050 7450 3950
+Connection ~ 7450 3950
+Wire Wire Line
+	7450 4550 7450 4700
+$Comp
+L +5V #PWR?
+U 1 1 549F97BA
+P 7450 4700
+F 0 "#PWR?" H 7450 4550 60  0001 C CNN
+F 1 "+5V" H 7450 4840 60  0000 C CNN
+F 2 "" H 7450 4700 60  0000 C CNN
+F 3 "" H 7450 4700 60  0000 C CNN
+	1    7450 4700
+	-1   0    0    1
+$EndComp
+Wire Wire Line
+	4200 2450 5100 2450
+Wire Wire Line
+	5100 2450 5100 3400
+Wire Wire Line
+	5100 3400 5450 3400
+Wire Wire Line
+	5450 3500 5000 3500
+Wire Wire Line
+	5000 3500 5000 2550
+Wire Wire Line
+	5000 2550 4200 2550
 $EndSCHEMATC

Commit message: Updated files.
Parts:
- added R? (x2): 10K, Resistors_SMD:R_0805_HandSoldering, symbol R
Connections:
- net +3V3: now also R?.1, R?.1
- net SCL: now also R?.2
- net SDA: now also R?.2
Changed lines of the file:
@@
 Connection ~ 5300 2550
 Wire Wire Line
-	3200 2000 3200 1850
+	3200 1850 3200 2000
 Wire Wire Line
-	3200 1850 2500 1850
+	2500 1850 3200 1850
 Wire Wire Line
 	2900 2000 2900 1850
@@
 Wire Wire Line
 	5000 2550 4200 2550
+$Comp
+L R R?
+U 1 1 54A04352
+P 2000 5700
+F 0 "R?" V 2080 5700 40  0000 C CNN
+F 1 "10K" V 2007 5701 40  0000 C CNN
+F 2 "Resistors_SMD:R_0805_HandSoldering" V 1930 5700 30  0001 C CNN
+F 3 "" H 2000 5700 30  0000 C CNN
+	1    2000 5700
+	1    0    0    -1
+$EndComp
+$Comp
+L R R?
+U 1 1 54A043D7
+P 1750 5700
+F 0 "R?" V 1830 5700 40  0000 C CNN
+F 1 "10K" V 1757 5701 40  0000 C CNN
+F 2 "Resistors_SMD:R_0805_HandSoldering" V 1680 5700 30  0001 C CNN
+F 3 "" H 1750 5700 30  0000 C CNN
+	1    1750 5700
+	1    0    0    -1
+$EndComp
+$Comp
+L +3V3 #PWR?
+U 1 1 54A044E3
+P 1750 5300
+F 0 "#PWR?" H 1750 5150 60  0001 C CNN
+F 1 "+3V3" H 1750 5440 60  0000 C CNN
+F 2 "" H 1750 5300 60  0000 C CNN
+F 3 "" H 1750 5300 60  0000 C CNN
+	1    1750 5300
+	1    0    0    -1
+$EndComp
+$Comp
+L +3V3 #PWR?
+U 1 1 54A044FC
+P 2000 5300
+F 0 "#PWR?" H 2000 5150 60  0001 C CNN
+F 1 "+3V3" H 2000 5440 60  0000 C CNN
+F 2 "" H 2000 5300 60  0000 C CNN
+F 3 "" H 2000 5300 60  0000 C CNN
+	1    2000 5300
+	1    0    0    -1
+$EndComp
+Wire Wire Line
+	2000 5300 2000 5450
+Wire Wire Line
+	1750 5300 1750 5450
+Text GLabel 2000 6100 3    50   Input ~ 0
+SDA
+Text GLabel 1750 6100 3    50   Input ~ 0
+SCL
+Wire Wire Line
+	1750 5950 1750 6100
+Wire Wire Line
+	2000 5950 2000 6100
 $EndSCHEMATC

Commit message: Worked on schematic.
Parts:
- added BT?: BATTERY, symbol BATTERY
- added C? (x2): 0.1uF, symbol C
- added R?: 10K, Resistors_SMD:R_0805_HandSoldering, symbol R
- added U?: DS3231, SMD_Packages:SO-16-W, symbol DS3231
- U3: footprint (none) -> SMD_Packages:SSOP-28
Connections:
- net +3V3: now also C?.2, C?.2, R?.1, U?.2 (VCC)
- net GND: now also BT?.2 (-), C?.1, C?.1, U?.10 (NC), U?.11 (NC), U?.12 (NC), U?.13 (GND), U?.5 (NC), U?.6 (NC), U?.7 (NC), U?.8 (NC), U?.9 (NC)
- net SCL: now also U?.16 (SCL)
- net SDA: now also U?.15 (SDA)
- new net: BT?.1 (+), U?.14 (VBAT)
- new net CLK_INT: R?.2, U?.3 (~INT)
- no-connect marks 3 -> 5
Other:
- moved on the sheet: C?, CON1, D?, Q?, R?, U1, U2, U3, X1

Commit message: Updated files.
Parts:
- C1, C2, C3: renamed from C?; footprint (none) -> Capacitors_SMD:C_0805_HandSoldering
- D1, D2: renamed from D?; footprint (none) -> LEDs:LED-0805
- R5, R6: renamed from R?; footprint (none) -> Resistors_SMD:R_0805_HandSoldering
- gave numbers to parts that had none: 7
Changed lines of the file:
@@
 $EndComp
 $Comp
-L GND #PWR2
+L GND #PWR01
 U 1 1 549F6A6A
 P 1500 5300
-F 0 "#PWR2" H 1500 5050 60  0001 C CNN
+F 0 "#PWR01" H 1500 5050 60  0001 C CNN
 F 1 "GND" H 1500 5150 60  0000 C CNN
 F 2 "" H 1500 5300 60  0000 C CNN
@@
 SDA
 $Comp
-L GND #PWR4
+L GND #PWR02
 U 1 1 549F6C2C
 P 3350 5300
-F 0 "#PWR4" H 3350 5050 60  0001 C CNN
+F 0 "#PWR02" H 3350 5050 60  0001 C CNN
 F 1 "GND" H 3350 5150 60  0000 C CNN
 F 2 "" H 3350 5300 60  0000 C CNN
@@
 $EndComp
 $Comp
-L GND #PWR5
+L GND #PWR03
 U 1 1 549F7C95
 P 5850 3400
-F 0 "#PWR5" H 5850 3150 60  0001 C CNN
+F 0 "#PWR03" H 5850 3150 60  0001 C CNN
 F 1 "GND" H 5850 3250 60  0000 C CNN
 F 2 "" H 5850 3400 60  0000 C CNN
@@
 $EndComp
 $Comp
-L GND #PWR3
+L GND #PWR04
 U 1 1 549F8071
 P 3100 1350
-F 0 "#PWR3" H 3100 1100 60  0001 C CNN
+F 0 "#PWR04" H 3100 1100 60  0001 C CNN
 F 1 "GND" H 3100 1200 60  0000 C CNN
 F 2 "" H 3100 1350 60  0000 C CNN
@@
 $EndComp
 $Comp
-L +5V #PWR?
+L +5V #PWR05
 U 1 1 549F8247
 P 4200 1800
-F 0 "#PWR?" H 4200 1650 60  0001 C CNN
+F 0 "#PWR05" H 4200 1650 60  0001 C CNN
 F 1 "+5V" H 4200 1940 60  0000 C CNN
 F 2 "" H 4200 1800 60  0000 C CNN
@@
 $EndComp
 $Comp
-L +5V #PWR?
+L +5V #PWR06
 U 1 1 549F825B
 P 4400 3750
-F 0 "#PWR?" H 4400 3600 60  0001 C CNN
+F 0 "#PWR06" H 4400 3600 60  0001 C CNN
 F 1 "+5V" H 4400 3890 60  0000 C CNN
 F 2 "" H 4400 3750 60  0000 C CNN
@@
 $EndComp
 $Comp
-L GND #PWR?
+L GND #PWR07
 U 1 1 549F8426
 P 5700 4400
-F 0 "#PWR?" H 5700 4150 60  0001 C CNN
+F 0 "#PWR07" H 5700 4150 60  0001 C CNN
 F 1 "GND" H 5700 4250 60  0000 C CNN
 F 2 "" H 5700 4400 60  0000 C CNN
@@
 $EndComp
 $Comp
-L GND #PWR?
+L GND #PWR08
 U 1 1 549F84C5
 P 4400 4400
-F 0 "#PWR?" H 4400 4150 60  0001 C CNN
+F 0 "#PWR08" H 4400 4150 60  0001 C CNN
 F 1 "GND" H 4400 4250 60  0000 C CNN
 F 2 "" H 4400 4400 60  0000 C CNN
@@
 NoConn ~ 4550 4150
 $Comp
-L +3V3 #PWR?
+L +3V3 #PWR09
 U 1 1 549F87F3
 P 1400 1050
-F 0 "#PWR?" H 1400 900 60  0001 C CNN
+F 0 "#PWR09" H 1400 900 60  0001 C CNN
 F 1 "+3V3" H 1400 1190 60  0000 C CNN
 F 2 "" H 1400 1050 60  0000 C CNN
@@
 $EndComp
 $Comp
-L C C?
+L C C3
 U 1 1 549F88B8
 P 6350 2100
-F 0 "C?" H 6350 2200 40  0000 L CNN
+F 0 "C3" H 6350 2200 40  0000 L CNN
 F 1 "10nF" H 6356 2015 40  0000 L CNN
-F 2 "" H 6388 1950 30  0000 C CNN
+F 2 "Capacitors_SMD:C_0805_HandSoldering" H 6388 1950 30  0001 C CNN
 F 3 "" H 6350 2100 60  0000 C CNN
 	1    6350 2100
@@
 $EndComp
 $Comp
-L NPN Q?
+L NPN Q1
 U 1 1 549F89D8
 P 7100 2100
-F 0 "Q?" H 7100 1950 50  0000 R CNN
+F 0 "Q1" H 7100 1950 50  0000 R CNN
 F 1 "NPN" H 7100 2250 50  0000 R CNN
 F 2 "Transistors_SMD:sot23" H 7100 2100 60  0001 C CNN
@@
 $EndComp
 $Comp
-L R R?
+L R R6
 U 1 1 549F8BBE
 P 6750 2550
-F 0 "R?" V 6830 2550 40  0000 C CNN
+F 0 "R6" V 6830 2550 40  0000 C CNN
 F 1 "10K" V 6757 2551 40  0000 C CNN
-F 2 "" V 6680 2550 30  0000 C CNN
+F 2 "Resistors_SMD:R_0805_HandSoldering" V 6680 2550 30  0001 C CNN
 F 3 "" H 6750 2550 30  0000 C CNN
 	1    6750 2550
@@
 $EndComp
 $Comp
-L GND #PWR?
+L GND #PWR010
 U 1 1 549F8E76
 P 7200 3050
-F 0 "#PWR?" H 7200 2800 60  0001 C CNN
+F 0 "#PWR010" H 7200 2800 60  0001 C CNN
 F 1 "GND" H 7200 2900 60  0000 C CNN
 F 2 "" H 7200 3050 60  0000 C CNN
@@
 DTR
 $Comp
-L R R?
+L R R5
 U 1 1 549F93DF
 P 6750 1450
-F 0 "R?" V 6830 1450 40  0000 C CNN
+F 0 "R5" V 6830 1450 40  0000 C CNN
 F 1 "10K" V 6757 1451 40  0000 C CNN
-F 2 "" V 6680 1450 30  0000 C CNN
+F 2 "Resistors_SMD:R_0805_HandSoldering" V 6680 1450 30  0001 C CNN
 F 3 "" H 6750 1450 30  0000 C CNN
 	1    6750 1450
@@
 $EndComp
 $Comp
-L +3V3 #PWR?
+L +3V3 #PWR011
 U 1 1 549F951B
 P 6750 1050
-F 0 "#PWR?" H 6750 900 60  0001 C CNN
+F 0 "#PWR011" H 6750 900 60  0001 C CNN
 F 1 "+3V3" H 6750 1190 60  0000 C CNN
 F 2 "" H 6750 1050 60  0000 C CNN
@@
 $EndComp
 $Comp
-L GND #PWR?
+L GND #PWR012
 U 1 1 549F9839
 P 1900 4150
-F 0 "#PWR?" H 1900 3900 60  0001 C CNN
+F 0 "#PWR012" H 1900 3900 60  0001 C CNN
 F 1 "GND" H 1900 4000 60  0000 C CNN
 F 2 "" H 1900 4150 60  0000 C CNN
@@
 $EndComp
 $Comp
-L +3V3 #PWR?
+L +3V3 #PWR013
 U 1 1 549F993F
 P 3000 4800
-F 0 "#PWR?" H 3000 4650 60  0001 C CNN
+F 0 "#PWR013" H 3000 4650 60  0001 C CNN
 F 1 "+3V3" H 3000 4940 60  0000 C CNN
 F 2 "" H 3000 4800 60  0000 C CNN
@@
 $EndComp
 $Comp
-L LED D?
+L LED D1
 U 1 1 549F9252
 P 6200 3000
-F 0 "D?" H 6200 3100 50  0000 C CNN
+F 0 "D1" H 6200 3100 50  0000 C CNN
 F 1 "LED" H 6200 2900 50  0000 C CNN
-F 2 "" H 6200 3000 60  0000 C CNN
+F 2 "LEDs:LED-0805" H 6200 3000 60  0001 C CNN
 F 3 "" H 6200 3000 60  0000 C CNN
 	1    6200 3000
@@
 $EndComp
 $Comp
-L LED D?
+L LED D2
 U 1 1 549F92C9
 P 6500 3000
-F 0 "D?" H 6500 3100 50  0000 C CNN
+F 0 "D2" H 6500 3100 50  0000 C CNN
 F 1 "LED" H 6500 2900 50  0000 C CNN
-F 2 "" H 6500 3000 60  0000 C CNN
+F 2 "LEDs:LED-0805" H 6500 3000 60  0001 C CNN
 F 3 "" H 6500 3000 60  0000 C CNN
 	1    6500 3000
@@
 $EndComp
 $Comp
-L R R?
+L R R4
 U 1 1 549F945E
 P 6350 3650
-F 0 "R?" V 6430 3650 40  0000 C CNN
+F 0 "R4" V 6430 3650 40  0000 C CNN
 F 1 "1K" V 6357 3651 40  0000 C CNN
 F 2 "Resistors_SMD:R_0805_HandSoldering" V 6280 3650 30  0001 C CNN
@@
 	6350 3900 6350 4050
 $Comp
-L +5V #PWR?
+L +5V #PWR014
 U 1 1 549F97BA
 P 6350 4050
-F 0 "#PWR?" H 6350 3900 60  0001 C CNN
+F 0 "#PWR014" H 6350 3900 60  0001 C CNN
 F 1 "+5V" H 6350 4190 60  0000 C CNN
 F 2 "" H 6350 4050 60  0000 C CNN
@@
 	3900 1900 3100 1900
 $Comp
-L R R?
+L R R2
 U 1 1 54A04352
 P 2400 6500
-F 0 "R?" V 2480 6500 40  0000 C CNN
+F 0 "R2" V 2480 6500 40  0000 C CNN
 F 1 "10K" V 2407 6501 40  0000 C CNN
 F 2 "Resistors_SMD:R_0805_HandSoldering" V 2330 6500 30  0001 C CNN
@@
 $EndComp
 $Comp
-L R R?
+L R R1
 U 1 1 54A043D7
 P 2150 6500
-F 0 "R?" V 2230 6500 40  0000 C CNN
+F 0 "R1" V 2230 6500 40  0000 C CNN
 F 1 "10K" V 2157 6501 40  0000 C CNN
 F 2 "Resistors_SMD:R_0805_HandSoldering" V 2080 6500 30  0001 C CNN
@@
 $EndComp
 $Comp
-L +3V3 #PWR?
+L +3V3 #PWR015
 U 1 1 54A044E3
 P 2150 6100
-F 0 "#PWR?" H 2150 5950 60  0001 C CNN
+F 0 "#PWR015" H 2150 5950 60  0001 C CNN
 F 1 "+3V3" H 2150 6240 60  0000 C CNN
 F 2 "" H 2150 6100 60  0000 C CNN
@@
 $EndComp
 $Comp
-L +3V3 #PWR?
+L +3V3 #PWR016
 U 1 1 54A044FC
 P 2400 6100
-F 0 "#PWR?" H 2400 5950 60  0001 C CNN
+F 0 "#PWR016" H 2400 5950 60  0001 C CNN
 F 1 "+3V3" H 2400 6240 60  0000 C CNN
 F 2 "" H 2400 6100 60  0000 C CNN
@@
 	2400 6750 2400 6900
 $Comp
-L DS3231 U?
+L DS3231 U4
 U 1 1 54A09D3F
 P 5050 5650
-F 0 "U?" H 5200 4900 60  0000 C CNN
+F 0 "U4" H 5200 4900 60  0000 C CNN
 F 1 "DS3231" H 5300 6100 60  0000 C CNN
 F 2 "SMD_Packages:SO-16-W" H 5050 5650 60  0001 C CNN
@@
 NoConn ~ 4450 5700
 $Comp
-L BATTERY BT?
+L BATTERY BT1
 U 1 1 54A0A224
 P 6250 6100
-F 0 "BT?" H 6250 6300 50  0000 C CNN
+F 0 "BT1" H 6250 6300 50  0000 C CNN
 F 1 "BATTERY" H 6250 5910 50  0000 C CNN
-F 2 "" H 6250 6100 60  0000 C CNN
+F 2 "" H 6250 6100 60  0001 C CNN
 F 3 "" H 6250 6100 60  0000 C CNN
 	1    6250 6100
@@
 Connection ~ 5800 6150
 $Comp
-L GND #PWR?
+L GND #PWR017
 U 1 1 54A0A7A2
 P 5050 6850
-F 0 "#PWR?" H 5050 6600 60  0001 C CNN
+F 0 "#PWR017" H 5050 6600 60  0001 C CNN
 F 1 "GND" H 5050 6700 60  0000 C CNN
 F 2 "" H 5050 6850 60  0000 C CNN
@@
 $EndComp
 $Comp
-L GND #PWR?
+L GND #PWR018
 U 1 1 54A0A7CD
 P 6250 6550
-F 0 "#PWR?" H 6250 6300 60  0001 C CNN
+F 0 "#PWR018" H 6250 6300 60  0001 C CNN
 F 1 "GND" H 6250 6400 60  0000 C CNN
 F 2 "" H 6250 6550 60  0000 C CNN
@@
 $EndComp
 $Comp
-L +3V3 #PWR?
+L +3V3 #PWR019
 U 1 1 54A0A98E
 P 5050 4900
-F 0 "#PWR?" H 5050 4750 60  0001 C CNN
+F 0 "#PWR019" H 5050 4750 60  0001 C CNN
 F 1 "+3V3" H 5050 5040 60  0000 C CNN
 F 2 "" H 5050 4900 60  0000 C CNN
@@
 	5050 4900 5050 5050
 $Comp
-L C C?
+L C C2
 U 1 1 54A0AA7F
 P 5600 4950
-F 0 "C?" H 5600 5050 40  0000 L CNN
+F 0 "C2" H 5600 5050 40  0000 L CNN
 F 1 "0.1uF" H 5606 4865 40  0000 L CNN
-F 2 "" H 5638 4800 30  0000 C CNN
+F 2 "Capacitors_SMD:C_0805_HandSoldering" H 5638 4800 30  0001 C CNN
 F 3 "" H 5600 4950 60  0000 C CNN
 	1    5600 4950
@@
 NoConn ~ 5650 5550
 $Comp
-L GND #PWR?
+L GND #PWR020
 U 1 1 54A0AFDC
 P 5900 5050
-F 0 "#PWR?" H 5900 4800 60  0001 C CNN
+F 0 "#PWR020" H 5900 4800 60  0001 C CNN
 F 1 "GND" H 5900 4900 60  0000 C CNN
 F 2 "" H 5900 5050 60  0000 C CNN
@@
 $EndComp
 $Comp
-L C C?
+L C C1
 U 1 1 54A0B1CB
 P 3550 4850
-F 0 "C?" H 3550 4950 40  0000 L CNN
+F 0 "C1" H 3550 4950 40  0000 L CNN
 F 1 "0.1uF" H 3556 4765 40  0000 L CNN
-F 2 "" H 3588 4700 30  0000 C CNN
+F 2 "Capacitors_SMD:C_0805_HandSoldering" H 3588 4700 30  0001 C CNN
 F 3 "" H 3550 4850 60  0000 C CNN
 	1    3550 4850
@@
 $EndComp
 $Comp
-L GND #PWR?
+L GND #PWR021
 U 1 1 54A0B233
 P 3900 4950
-F 0 "#PWR?" H 3900 4700 60  0001 C CNN
+F 0 "#PWR021" H 3900 4700 60  0001 C CNN
 F 1 "GND" H 3900 4800 60  0000 C CNN
 F 2 "" H 3900 4950 60  0000 C CNN
@@
 CLK_INT
 $Comp
-L R R?
+L R R3
 U 1 1 54A0C1E4
 P 6300 5050
-F 0 "R?" V 6380 5050 40  0000 C CNN
+F 0 "R3" V 6380 5050 40  0000 C CNN
 F 1 "10K" V 6307 5051 40  0000 C CNN
 F 2 "Resistors_SMD:R_0805_HandSoldering" V 6230 5050 30  0001 C CNN
@@
 $EndComp
 $Comp
-L +3V3 #PWR?
+L +3V3 #PWR022
 U 1 1 54A0C24B
 P 6300 4650
-F 0 "#PWR?" H 6300 4500 60  0001 C CNN
+F 0 "#PWR022" H 6300 4500 60  0001 C CNN
 F 1 "+3V3" H 6300 4790 60  0000 C CNN
 F 2 "" H 6300 4650 60  0000 C CNN
