File: PCB/7SegClock.sch (KiCad schematic (older format))
At the start: 19 parts, among them CON1 USB-MINI-B, Q1 NPN, U1 P8X32A, U2 24LC256, U3 FT232RL, U4 DS3231, X1 5mhz CRYSTAL

Commit message: Schematic progress.
Parts:
- added F?: FUSE, symbol FUSE
- added U?: TPS62172DSGT, symbol TPS62172DSGT
Connections:
- net +5V: now also F?.2; no longer CON1.1 (VBUS)
- new net VIN: CON1.1 (VBUS), F?.1
Changed lines of the file:
@@
 L +5V #PWR06
 U 1 1 549F825B
-P 4400 3750
-F 0 "#PWR06" H 4400 3600 60  0001 C CNN
-F 1 "+5V" H 4400 3890 60  0000 C CNN
-F 2 "" H 4400 3750 60  0000 C CNN
-F 3 "" H 4400 3750 60  0000 C CNN
-	1    4400 3750
-	1    0    0    -1
+P 5450 1000
+F 0 "#PWR06" H 5450 850 60  0001 C CNN
+F 1 "+5V" H 5450 1140 60  0000 C CNN
+F 2 "" H 5450 1000 60  0000 C CNN
+F 3 "" H 5450 1000 60  0000 C CNN
+	1    5450 1000
+	0    1    1    0
 $EndComp
 $Comp
@@
 Connection ~ 2700 1200
 Wire Wire Line
-	4400 3750 4400 3850
-Wire Wire Line
-	4400 3850 4550 3850
-Wire Wire Line
-	4550 3950 4200 3950
-Wire Wire Line
-	4200 3950 4200 3200
-Wire Wire Line
-	4200 3200 4350 3200
-Wire Wire Line
-	4350 3100 4100 3100
-Wire Wire Line
-	4100 3100 4100 4050
-Wire Wire Line
-	4100 4050 4550 4050
-Wire Wire Line
 	5550 3850 5700 3850
 Wire Wire Line
@@
 Wire Wire Line
 	5900 4950 5900 5050
+$Comp
+L FUSE F?
+U 1 1 54A0D025
+P 5050 1000
+F 0 "F?" H 5150 1050 40  0000 C CNN
+F 1 "FUSE" H 4950 950 40  0000 C CNN
+F 2 "" H 5050 1000 60  0000 C CNN
+F 3 "" H 5050 1000 60  0000 C CNN
+	1    5050 1000
+	1    0    0    -1
+$EndComp
+$Comp
+L TPS62172DSGT U?
+U 1 1 54A0D0C2
+P 9500 2450
+F 0 "U?" H 9500 2150 60  0000 C CNN
+F 1 "TPS62172DSGT" H 9500 2750 60  0000 C CNN
+F 2 "" H 9500 2450 60  0000 C CNN
+F 3 "" H 9500 2450 60  0000 C CNN
+	1    9500 2450
+	1    0    0    -1
+$EndComp
+Wire Wire Line
+	5450 1000 5300 1000
+Text GLabel 4650 1000 0    50   Input ~ 0
+VIN
+Wire Wire Line
+	4800 1000 4650 1000
+Text GLabel 4400 3850 0    50   Input ~ 0
+VIN
+Wire Wire Line
+	4550 3850 4400 3850
+Wire Wire Line
+	4550 3950 4100 3950
+Wire Wire Line
+	4100 3950 4100 3200
+Wire Wire Line
+	4100 3200 4350 3200
+Wire Wire Line
+	4350 3100 4000 3100
+Wire Wire Line
+	4000 3100 4000 4050
+Wire Wire Line
+	4000 4050 4550 4050
 $EndSCHEMATC

Commit message: Worked on schematic.
Parts:
- gave numbers to parts that had none: 2
Connections:
- net P16: now reaches U1.19 (P16)
Changed lines of the file:
@@
 $Descr A4 11693 8268
 encoding utf-8
-Sheet 1 1
+Sheet 1 2
 Title "4 Digit 7 Segment Clock"
 Date "12/27/14"
@@
 	5900 4950 5900 5050
 $Comp
-L FUSE F?
+L FUSE F1
 U 1 1 54A0D025
 P 5050 1000
-F 0 "F?" H 5150 1050 40  0000 C CNN
+F 0 "F1" H 5150 1050 40  0000 C CNN
 F 1 "FUSE" H 4950 950 40  0000 C CNN
-F 2 "" H 5050 1000 60  0000 C CNN
+F 2 "" H 5050 1000 60  0001 C CNN
 F 3 "" H 5050 1000 60  0000 C CNN
 	1    5050 1000
@@
 $EndComp
 $Comp
-L TPS62172DSGT U?
+L TPS62172DSGT U5
 U 1 1 54A0D0C2
 P 9500 2450
-F 0 "U?" H 9500 2150 60  0000 C CNN
+F 0 "U5" H 9500 2150 60  0000 C CNN
 F 1 "TPS62172DSGT" H 9500 2750 60  0000 C CNN
-F 2 "" H 9500 2450 60  0000 C CNN
+F 2 "" H 9500 2450 60  0001 C CNN
 F 3 "" H 9500 2450 60  0000 C CNN
 	1    9500 2450
@@
 Wire Wire Line
 	4000 4050 4550 4050
+$Sheet
+S 9600 4600 1000 800
+U 54A9B3AB
+F0 "Lattice MACHXO2" 60
+F1 "FPGA.sch" 60
+$EndSheet
+Wire Wire Line
+	3100 3300 3350 3300
+Text Label 3250 3300 0    39   ~ 0
+P16
 $EndSCHEMATC
