File: PCB/7SegClock.sch (KiCad schematic (older format))
At the start: 25 parts, among them CON1 USB-MINI-B, Q1 NPN, U1 P8X32A, U2 24LC256, U3 FT232RL, U4 DS3231, U5 TPS62172DSGT, X1 5mhz CRYSTAL

Commit message: Added additional mosfets.
Parts:
- U1: renamed from U5; footprint SMD_Packages:WSON-8-1EP -> SMD_Packages:TQFP-44
- U2: renamed from U1; footprint SMD_Packages:TQFP-44 -> SMD_Packages:SOIC-8-N
- U4: renamed from U2; footprint SMD_Packages:SOIC-8-N -> SMD_Packages:SO-16-W
- U5: renamed from U4; footprint SMD_Packages:SO-16-W -> SMD_Packages:WSON-8-1EP
- renumbered C3 to C1, C1 to C2, C2 to C3, R5 to R1, R6 to R2, R4 to R3, R3 to R4, R1 to R5, R2 to R6
Changed lines of the file:
@@
 $EndDescr
 $Comp
-L P8X32A U1
+L P8X32A U2
 U 1 1 549F5799
 P 2250 2550
-F 0 "U1" H 2250 2400 60  0000 C CNN
+F 0 "U2" H 2250 2400 60  0000 C CNN
 F 1 "P8X32A" H 2250 2700 60  0000 C CNN
-F 2 "SMD_Packages:TQFP-44" H 1950 2950 60  0001 C CNN
+F 2 "SMD_Packages:SOIC-8-N" H 1950 2950 60  0001 C CNN
 F 3 "" H 1950 2950 60  0000 C CNN
 	1    2250 2550
@@
 $EndComp
 $Comp
-L 24LC256 U2
+L 24LC256 U4
 U 1 1 549F6837
 P 2250 5050
-F 0 "U2" H 2250 4700 60  0000 C CNN
+F 0 "U4" H 2250 4700 60  0000 C CNN
 F 1 "24LC256" H 2250 5400 60  0000 C CNN
-F 2 "SMD_Packages:SOIC-8-N" H 2250 5050 60  0001 C CNN
+F 2 "SMD_Packages:SO-16-W" H 2250 5050 60  0001 C CNN
 F 3 "" H 2250 5050 60  0000 C CNN
 	1    2250 5050
@@
 NoConn ~ 4550 4150
 $Comp
-L C C3
+L C C1
 U 1 1 549F88B8
 P 6350 2100
-F 0 "C3" H 6350 2200 40  0000 L CNN
+F 0 "C1" H 6350 2200 40  0000 L CNN
 F 1 "10nF" H 6356 2015 40  0000 L CNN
 F 2 "Capacitors_SMD:C_0603_HandSoldering" H 6388 1950 30  0001 C CNN
@@
 $EndComp
 $Comp
-L R R6
+L R R2
 U 1 1 549F8BBE
 P 6750 2550
-F 0 "R6" V 6830 2550 40  0000 C CNN
+F 0 "R2" V 6830 2550 40  0000 C CNN
 F 1 "10K" V 6757 2551 40  0000 C CNN
 F 2 "Resistors_SMD:R_0603_HandSoldering" V 6680 2550 30  0001 C CNN
@@
 DTR
 $Comp
-L R R5
+L R R1
 U 1 1 549F93DF
 P 6750 1450
-F 0 "R5" V 6830 1450 40  0000 C CNN
+F 0 "R1" V 6830 1450 40  0000 C CNN
 F 1 "10K" V 6757 1451 40  0000 C CNN
 F 2 "Resistors_SMD:R_0603_HandSoldering" V 6680 1450 30  0001 C CNN
@@
 $EndComp
 $Comp
-L R R4
+L R R3
 U 1 1 549F945E
 P 6350 3650
-F 0 "R4" V 6430 3650 40  0000 C CNN
+F 0 "R3" V 6430 3650 40  0000 C CNN
 F 1 "1K" V 6357 3651 40  0000 C CNN
 F 2 "Resistors_SMD:R_0603_HandSoldering" V 6280 3650 30  0001 C CNN
@@
 	3750 1900 3100 1900
 $Comp
-L R R2
+L R R6
 U 1 1 54A04352
 P 1200 6700
-F 0 "R2" V 1280 6700 40  0000 C CNN
+F 0 "R6" V 1280 6700 40  0000 C CNN
 F 1 "10K" V 1207 6701 40  0000 C CNN
 F 2 "Resistors_SMD:R_0603_HandSoldering" V 1130 6700 30  0001 C CNN
@@
 $EndComp
 $Comp
-L R R1
+L R R5
 U 1 1 54A043D7
 P 950 6700
-F 0 "R1" V 1030 6700 40  0000 C CNN
+F 0 "R5" V 1030 6700 40  0000 C CNN
 F 1 "10K" V 957 6701 40  0000 C CNN
 F 2 "Resistors_SMD:R_0603_HandSoldering" V 880 6700 30  0001 C CNN
@@
 	1200 6950 1200 7100
 $Comp
-L DS3231 U4
+L DS3231 U5
 U 1 1 54A09D3F
 P 5050 5650
-F 0 "U4" H 5200 4900 60  0000 C CNN
+F 0 "U5" H 5200 4900 60  0000 C CNN
 F 1 "DS3231" H 5300 6100 60  0000 C CNN
-F 2 "SMD_Packages:SO-16-W" H 5050 5650 60  0001 C CNN
+F 2 "SMD_Packages:WSON-8-1EP" H 5050 5650 60  0001 C CNN
 F 3 "" H 5050 5650 60  0000 C CNN
 	1    5050 5650
@@
 	5050 4900 5050 5050
 $Comp
-L C C2
+L C C3
 U 1 1 54A0AA7F
 P 5600 4950
-F 0 "C2" H 5600 5050 40  0000 L CNN
+F 0 "C3" H 5600 5050 40  0000 L CNN
 F 1 "0.1uF" H 5606 4865 40  0000 L CNN
 F 2 "Capacitors_SMD:C_0603_HandSoldering" H 5638 4800 30  0001 C CNN
@@
 $EndComp
 $Comp
-L C C1
+L C C2
 U 1 1 54A0B1CB
 P 3550 4850
-F 0 "C1" H 3550 4950 40  0000 L CNN
+F 0 "C2" H 3550 4950 40  0000 L CNN
 F 1 "0.1uF" H 3556 4765 40  0000 L CNN
 F 2 "Capacitors_SMD:C_0603_HandSoldering" H 3588 4700 30  0001 C CNN
@@
 CLK_INT
 $Comp
-L R R3
+L R R4
 U 1 1 54A0C1E4
 P 6350 5050
-F 0 "R3" V 6430 5050 40  0000 C CNN
+F 0 "R4" V 6430 5050 40  0000 C CNN
 F 1 "10K" V 6357 5051 40  0000 C CNN
 F 2 "Resistors_SMD:R_0603_HandSoldering" V 6280 5050 30  0001 C CNN
@@
 $EndComp
 $Comp
-L TPS62172DSGT U5
+L TPS62172DSGT U1
 U 1 1 54A0D0C2
 P 9500 2450
-F 0 "U5" H 9500 2150 60  0000 C CNN
+F 0 "U1" H 9500 2150 60  0000 C CNN
 F 1 "TPS62172DSGT" H 9500 2750 60  0000 C CNN
-F 2 "SMD_Packages:WSON-8-1EP" H 9500 2450 60  0001 C CNN
+F 2 "SMD_Packages:TQFP-44" H 9500 2450 60  0001 C CNN
 F 3 "" H 9500 2450 60  0000 C CNN
 	1    9500 2450

Commit message: Edit PCB.
Parts:
- R3: value 1K -> 150
Changed lines of the file:
@@
 P 6350 3650
 F 0 "R3" V 6430 3650 40  0000 C CNN
-F 1 "1K" V 6357 3651 40  0000 C CNN
+F 1 "150" V 6357 3651 40  0000 C CNN
 F 2 "Resistors_SMD:R_0603_HandSoldering" V 6280 3650 30  0001 C CNN
 F 3 "" H 6350 3650 30  0000 C CNN
@@
 	2100 1200 2100 1350
 Wire Wire Line
-	1500 1200 2100 1200
-Wire Wire Line
-	1800 1350 1800 1200
+	1800 1000 1800 1350
 Connection ~ 1800 1200
 Wire Wire Line
@@
 	2000 1350 2000 1200
 Connection ~ 2000 1200
-Text Label 1500 1200 0    50   ~ 0
-VDD
 Wire Wire Line
 	9600 5350 9200 5350
@@
 Entry Wire Line
 	9450 -400 9550 -300
+Wire Wire Line
+	1800 1200 2100 1200
+$Comp
+L +3V3 #PWR023
+U 1 1 55A05889
+P 1800 1000
+F 0 "#PWR023" H 1800 850 60  0001 C CNN
+F 1 "+3V3" H 1800 1140 60  0000 C CNN
+F 2 "" H 1800 1000 60  0000 C CNN
+F 3 "" H 1800 1000 60  0000 C CNN
+	1    1800 1000
+	1    0    0    -1
+$EndComp
 $EndSCHEMATC

Commit message: PCB work.
Parts:
- removed CON1: USB-MINI-B, Connect:USB_Mini-B, symbol USB-MINI-B
- added CON1: USB_Micro_Vertical, Custom:MicroSD_Vertical, symbol USB_Micro_Vertical
- added U7: Electric_Imp, Custom:SD_Card, symbol Electric_Imp
- BT1: footprint (none) -> Custom:SuperCap_604-1020-1-ND
- F1: footprint (none) -> Fuse_Holders_and_Fuses:Fuse_SMD1206_HandSoldering
- R1, R2, R3, R4, R5, R6: footprint Resistors_SMD:R_0603_HandSoldering -> Resistors_SMD:R_0402
- U1: footprint SMD_Packages:TQFP-44 -> Custom:WSON-8-1EP
- U2: footprint SMD_Packages:SOIC-8-N -> Custom:TQFP-44
- U4: footprint SMD_Packages:SO-16-W -> SMD_Packages:SOIC-8-N
- U5: footprint SMD_Packages:WSON-8-1EP -> SMD_Packages:SO-16-L
Connections:
- wire segments 136 -> 135
- no-connect marks 5 -> 4
Other:
- moved on the sheet: U1
Changed lines of the file:
@@
 F 0 "U2" H 2250 2400 60  0000 C CNN
 F 1 "P8X32A" H 2250 2700 60  0000 C CNN
-F 2 "SMD_Packages:SOIC-8-N" H 1950 2950 60  0001 C CNN
+F 2 "Custom:TQFP-44" H 1950 2950 60  0001 C CNN
 F 3 "" H 1950 2950 60  0000 C CNN
 	1    2250 2550
@@
 SDA
 $Comp
-L USB-MINI-B CON1
-U 1 1 549F617F
-P 5050 4050
-F 0 "CON1" H 4750 4400 50  0000 C CNN
-F 1 "USB-MINI-B" H 4900 3700 50  0000 C CNN
-F 2 "Connect:USB_Mini-B" H 5050 3950 50  0001 C CNN
-F 3 "" H 5050 3950 50  0000 C CNN
-	1    5050 4050
-	1    0    0    -1
-$EndComp
-$Comp
 L 24LC256 U4
 U 1 1 549F6837
@@
 F 0 "U4" H 2250 4700 60  0000 C CNN
 F 1 "24LC256" H 2250 5400 60  0000 C CNN
-F 2 "SMD_Packages:SO-16-W" H 2250 5050 60  0001 C CNN
+F 2 "SMD_Packages:SOIC-8-N" H 2250 5050 60  0001 C CNN
 F 3 "" H 2250 5050 60  0000 C CNN
 	1    2250 5050
@@
 L GND #PWR07
 U 1 1 549F8426
-P 5700 4400
-F 0 "#PWR07" H 5700 4150 60  0001 C CNN
-F 1 "GND" H 5700 4250 60  0000 C CNN
-F 2 "" H 5700 4400 60  0000 C CNN
-F 3 "" H 5700 4400 60  0000 C CNN
-	1    5700 4400
+P 5700 4225
+F 0 "#PWR07" H 5700 3975 60  0001 C CNN
+F 1 "GND" H 5700 4075 60  0000 C CNN
+F 2 "" H 5700 4225 60  0000 C CNN
+F 3 "" H 5700 4225 60  0000 C CNN
+	1    5700 4225
 	1    0    0    -1
 $EndComp
@@
 L GND #PWR08
 U 1 1 549F84C5
-P 4400 4400
-F 0 "#PWR08" H 4400 4150 60  0001 C CNN
-F 1 "GND" H 4400 4250 60  0000 C CNN
-F 2 "" H 4400 4400 60  0000 C CNN
-F 3 "" H 4400 4400 60  0000 C CNN
-	1    4400 4400
+P 4400 4225
+F 0 "#PWR08" H 4400 3975 60  0001 C CNN
+F 1 "GND" H 4400 4075 60  0000 C CNN
+F 2 "" H 4400 4225 60  0000 C CNN
+F 3 "" H 4400 4225 60  0000 C CNN
+	1    4400 4225
 	1    0    0    -1
 $EndComp
 NoConn ~ 5700 1900
 NoConn ~ 5700 2000
-NoConn ~ 4550 4150
 $Comp
 L C C1
@@
 F 0 "R2" V 6830 2550 40  0000 C CNN
 F 1 "10K" V 6757 2551 40  0000 C CNN
-F 2 "Resistors_SMD:R_0603_HandSoldering" V 6680 2550 30  0001 C CNN
+F 2 "Resistors_SMD:R_0402" V 6680 2550 30  0001 C CNN
 F 3 "" H 6750 2550 30  0000 C CNN
 	1    6750 2550
@@
 F 0 "R1" V 6830 1450 40  0000 C CNN
 F 1 "10K" V 6757 1451 40  0000 C CNN
-F 2 "Resistors_SMD:R_0603_HandSoldering" V 6680 1450 30  0001 C CNN
+F 2 "Resistors_SMD:R_0402" V 6680 1450 30  0001 C CNN
 F 3 "" H 6750 1450 30  0000 C CNN
 	1    6750 1450
@@
 F 0 "R3" V 6430 3650 40  0000 C CNN
 F 1 "150" V 6357 3651 40  0000 C CNN
-F 2 "Resistors_SMD:R_0603_HandSoldering" V 6280 3650 30  0001 C CNN
+F 2 "Resistors_SMD:R_0402" V 6280 3650 30  0001 C CNN
 F 3 "" H 6350 3650 30  0000 C CNN
 	1    6350 3650
@@
 	2700 1350 2700 1200
 Connection ~ 2700 1200
-Wire Wire Line
-	5550 3850 5700 3850
-Wire Wire Line
-	5700 3850 5700 4400
-Wire Wire Line
-	5550 4250 5700 4250
-Connection ~ 5700 4250
-Wire Wire Line
-	5550 4150 5700 4150
-Connection ~ 5700 4150
-Wire Wire Line
-	5550 3950 5700 3950
-Connection ~ 5700 3950
-Wire Wire Line
-	4550 4250 4400 4250
-Wire Wire Line
-	4400 4250 4400 4400
 Wire Wire Line
 	4200 1800 4200 2000
@@
 F 0 "R6" V 1280 6700 40  0000 C CNN
 F 1 "10K" V 1207 6701 40  0000 C CNN
-F 2 "Resistors_SMD:R_0603_HandSoldering" V 1130 6700 30  0001 C CNN
+F 2 "Resistors_SMD:R_0402" V 1130 6700 30  0001 C CNN
 F 3 "" H 1200 6700 30  0000 C CNN
 	1    1200 6700
@@
 F 0 "R5" V 1030 6700 40  0000 C CNN
 F 1 "10K" V 957 6701 40  0000 C CNN
-F 2 "Resistors_SMD:R_0603_HandSoldering" V 880 6700 30  0001 C CNN
+F 2 "Resistors_SMD:R_0402" V 880 6700 30  0001 C CNN
 F 3 "" H 950 6700 30  0000 C CNN
 	1    950  6700
@@
 F 0 "U5" H 5200 4900 60  0000 C CNN
 F 1 "DS3231" H 5300 6100 60  0000 C CNN
-F 2 "SMD_Packages:WSON-8-1EP" H 5050 5650 60  0001 C CNN
+F 2 "SMD_Packages:SO-16-L" H 5050 5650 60  0001 C CNN
 F 3 "" H 5050 5650 60  0000 C CNN
 	1    5050 5650
@@
 F 0 "BT1" H 6250 6300 50  0000 C CNN
 F 1 "BATTERY" H 6250 5910 50  0000 C CNN
-F 2 "" H 6250 6100 60  0001 C CNN
+F 2 "Custom:SuperCap_604-1020-1-ND" H 6250 6100 60  0001 C CNN
 F 3 "" H 6250 6100 60  0000 C CNN
 	1    6250 6100
@@
 F 0 "R4" V 6430 5050 40  0000 C CNN
 F 1 "10K" V 6357 5051 40  0000 C CNN
-F 2 "Resistors_SMD:R_0603_HandSoldering" V 6280 5050 30  0001 C CNN
+F 2 "Resistors_SMD:R_0402" V 6280 5050 30  0001 C CNN
 F 3 "" H 6350 5050 30  0000 C CNN
 	1    6350 5050
@@
 F 0 "F1" H 5100 1050 40  0000 C CNN
 F 1 "FUSE" H 4900 950 40  0000 C CNN
-F 2 "" H 5000 1000 60  0001 C CNN
+F 2 "Fuse_Holders_and_Fuses:Fuse_SMD1206_HandSoldering" H 5000 1000 60  0001 C CNN
 F 3 "" H 5000 1000 60  0000 C CNN
 	1    5000 1000
@@
 L TPS62172DSGT U1
 U 1 1 54A0D0C2
-P 9500 2450
-F 0 "U1" H 9500 2150 60  0000 C CNN
-F 1 "TPS62172DSGT" H 9500 2750 60  0000 C CNN
-F 2 "SMD_Packages:TQFP-44" H 9500 2450 60  0001 C CNN
-F 3 "" H 9500 2450 60  0000 C CNN
-	1    9500 2450
+P 9500 1500
+F 0 "U1" H 9500 1200 60  0000 C CNN
+F 1 "TPS62172DSGT" H 9500 1800 60  0000 C CNN
+F 2 "Custom:WSON-8-1EP" H 9500 1500 60  0001 C CNN
+F 3 "" H 9500 1500 60  0000 C CNN
+	1    9500 1500
 	1    0    0    -1
 $EndComp
@@
 VIN
 Wire Wire Line
-	4550 3850 4400 3850
-Wire Wire Line
-	4550 3950 4100 3950
-Wire Wire Line
-	4100 3950 4100 3200
-Wire Wire Line
 	4100 3200 4350 3200
 Wire Wire Line
 	4350 3100 4000 3100
-Wire Wire Line
-	4000 3100 4000 4050
-Wire Wire Line
-	4000 4050 4550 4050
 $Sheet
 S 9600 5200 1000 800
@@
 	1    0    0    -1
 $EndComp
+$Comp
+L Electric_Imp U7
+U 1 1 55BE7C01
+P 9500 3000
+F 0 "U7" H 9500 2575 60  0000 C CNN
+F 1 "Electric_Imp" H 9500 3425 60  0000 C CNN
+F 2 "Custom:SD_Card" H 9150 3025 60  0001 C CNN
+F 3 "" H 9150 3025 60  0000 C CNN
+	1    9500 3000
+	1    0    0    -1
+$EndComp
+$Comp
+L USB_Micro_Vertical CON1
+U 1 1 55BEE955
+P 5050 4000
+F 0 "CON1" H 5050 3725 60  0000 C CNN
+F 1 "USB_Micro_Vertical" H 5050 4275 60  0000 C CNN
+F 2 "Custom:MicroSD_Vertical" H 5050 4000 60  0001 C CNN
+F 3 "" H 5050 4000 60  0000 C CNN
+	1    5050 4000
+	1    0    0    -1
+$EndComp
+Wire Wire Line
+	4525 3850 4400 3850
+Wire Wire Line
+	4525 4150 4400 4150
+Wire Wire Line
+	4400 4150 4400 4225
+Wire Wire Line
+	5700 4225 5700 3925
+Wire Wire Line
+	5700 3925 5575 3925
+Wire Wire Line
+	5575 4000 5700 4000
+Connection ~ 5700 4000
+Wire Wire Line
+	5575 4075 5700 4075
+Connection ~ 5700 4075
+Wire Wire Line
+	4100 3925 4525 3925
+Wire Wire Line
+	4100 3200 4100 3925
+Wire Wire Line
+	4525 4000 4000 4000
+Wire Wire Line
+	4000 4000 4000 3100
 $EndSCHEMATC

Commit message: PCB work.
Parts:
- removed U7: Electric_Imp, Custom:SD_Card, symbol Electric_Imp
Changed lines of the file:
@@
-$EndComp
-$Comp
-L Electric_Imp U7
-U 1 1 55BE7C01
-P 9500 3000
-F 0 "U7" H 9500 2575 60  0000 C CNN
-F 1 "Electric_Imp" H 9500 3425 60  0000 C CNN
-F 2 "Custom:SD_Card" H 9150 3025 60  0001 C CNN
-F 3 "" H 9150 3025 60  0000 C CNN
-	1    9500 3000
-	1    0    0    -1
 $EndComp
 $Comp

Commit message: PCB work.
Parts:
- C1, C2, C3, C4, C5, C6, C7: symbol C -> C-RESCUE-7SegClock
- D1, D2: symbol LED -> LED-RESCUE-7SegClock
- R1, R2, R3, R4, R5, R6: symbol R -> R-RESCUE-7SegClock
Changed lines of the file:
@@
 EESchema Schematic File Version 2
+LIBS:7SegClock-rescue
 LIBS:power
 LIBS:device
@@
 LIBS:memory
 LIBS:xilinx
-LIBS:special
 LIBS:microcontrollers
 LIBS:dsp
@@
 NoConn ~ 5700 2000
 $Comp
-L C C1
+L C-RESCUE-7SegClock C1
 U 1 1 549F88B8
 P 6350 2100
@@
 $EndComp
 $Comp
-L R R2
+L R-RESCUE-7SegClock R2
 U 1 1 549F8BBE
 P 6750 2550
@@
 DTR
 $Comp
-L R R1
+L R-RESCUE-7SegClock R1
 U 1 1 549F93DF
 P 6750 1450
@@
 $EndComp
 $Comp
-L LED D1
+L LED-RESCUE-7SegClock D1
 U 1 1 549F9252
 P 6200 3000
@@
 $EndComp
 $Comp
-L LED D2
+L LED-RESCUE-7SegClock D2
 U 1 1 549F92C9
 P 6500 3000
@@
 $EndComp
 $Comp
-L R R3
+L R-RESCUE-7SegClock R3
 U 1 1 549F945E
 P 6350 3650
@@
 	3750 1900 3100 1900
 $Comp
-L R R6
+L R-RESCUE-7SegClock R6
 U 1 1 54A04352
 P 1200 6700
@@
 $EndComp
 $Comp
-L R R5
+L R-RESCUE-7SegClock R5
 U 1 1 54A043D7
 P 950 6700
@@
 	5050 4900 5050 5050
 $Comp
-L C C3
+L C-RESCUE-7SegClock C3
 U 1 1 54A0AA7F
 P 5600 4950
@@
 $EndComp
 $Comp
-L C C2
+L C-RESCUE-7SegClock C2
 U 1 1 54A0B1CB
 P 3550 4850
@@
 CLK_INT
 $Comp
-L R R4
+L R-RESCUE-7SegClock R4
 U 1 1 54A0C1E4
 P 6350 5050
@@
 $EndSheet
 $Comp
-L C C7
+L C-RESCUE-7SegClock C7
 U 1 1 54B5BD71
 P 2700 6750
@@
 $EndComp
 $Comp
-L C C6
+L C-RESCUE-7SegClock C6
 U 1 1 54B5BE23
 P 2450 6750
@@
 $EndComp
 $Comp
-L C C5
+L C-RESCUE-7SegClock C5
 U 1 1 54B5BE54
 P 2200 6750
@@
 $EndComp
 $Comp
-L C C4
+L C-RESCUE-7SegClock C4
 U 1 1 54B5BE86
 P 1950 6750

Commit message: Removed old directory.
Parts:
- U4: symbol 24LC256 -> 24LC256-RESCUE-7SegClock
Changed lines of the file:
@@
 SDA
 $Comp
-L 24LC256 U4
+L 24LC256-RESCUE-7SegClock U4
 U 1 1 549F6837
 P 2250 5050
@@
 BC 01 60 96 31 E6 05 00 CF E7 7F 1E 6D 7A 11 6D 4B 35 E4 B7 1B 6B 03 D8 50 55 DF E5 BD 5F 0B 59
 F0 3A 1E C0 38 64 CF D4 F2 C8 9E A9 05 CC 43 F6 BE 79 15 99 0A D7 74 00 CF 02 78 CE 18 F3 24 80
-47 91 3D 63 3D 51 4F 11 C2 FF 03 CA 62 49 C8 E1 A2 25 5C 00 00 00 00 49 45 4E 44 AE 42 60 82 00
+47 91 3D 63 3D 51 4F 11 C2 FF 03 CA 62 49 C8 E1 A2 25 5C 00 00 00 00 49 45 4E 44 AE 42 60 82
 EndData
 $EndBitmap
