File: PCB/Digit1.sch (KiCad schematic (older format))
At the start: 1 part

Commit message: Worked on PCB.
Connections:
- net labels added: D1A1, D1A2, D1A3, D1A4, D1A5, D1A6
- wire segments 0 -> 59
Other:
- moved on the sheet: D3A
Changed lines of the file:
@@
 Comment4 ""
 $EndDescr
+Text Label 3000 950  3    50   ~ 0
+D1A1
+Text Label 3300 950  3    50   ~ 0
+D1A2
+Text Label 3600 950  3    50   ~ 0
+D1A3
+Text Label 3900 950  3    50   ~ 0
+D1A4
+Text Label 4200 950  3    50   ~ 0
+D1A5
+Text Label 4500 950  3    50   ~ 0
+D1A6
+Text Label 3000 3650 3    50   ~ 0
+D1A1
+Text Label 3300 3650 3    50   ~ 0
+D1A2
+Text Label 3600 3650 3    50   ~ 0
+D1A3
+Text Label 3900 3650 3    50   ~ 0
+D1A4
+Text Label 4200 3650 3    50   ~ 0
+D1A5
+Text Label 4500 3650 3    50   ~ 0
+D1A6
+Text Label 4500 7350 1    50   ~ 0
+D1A1
+Text Label 4200 7350 1    50   ~ 0
+D1A2
+Text Label 3900 7350 1    50   ~ 0
+D1A3
+Text Label 3600 7350 1    50   ~ 0
+D1A4
+Text Label 3300 7350 1    50   ~ 0
+D1A5
+Text Label 3000 7350 1    50   ~ 0
+D1A6
 $Comp
 L LED_Array D3
 U 1 1 54BC75FA
-P 4900 4050
-F 0 "D3" H 4900 5200 50  0000 C CNN
-F 1 "LED_Array" H 4900 5300 50  0000 C CNN
-F 2 "Custom:LED-ARRAY" H 4900 4975 50  0001 C CNN
-F 3 "" H 4900 4975 50  0000 C CNN
-	1    4900 4050
+P 3750 4150
+F 0 "D3" H 3750 5300 50  0000 C CNN
+F 1 "LED_Array" H 3750 5400 50  0000 C CNN
+F 2 "Custom:LED-ARRAY" H 3750 5075 50  0001 C CNN
+F 3 "" H 3750 5075 50  0000 C CNN
+	1    3750 4150
 	1    0    0    -1
 $EndComp
+Wire Wire Line
+	3000 1150 3000 950
+Wire Wire Line
+	3300 1150 3300 950
+Wire Wire Line
+	3600 1150 3600 950
+Wire Wire Line
+	3900 1150 3900 950
+Wire Wire Line
+	4200 1150 4200 950
+Wire Wire Line
+	4500 1150 4500 950
+Wire Wire Line
+	5325 2350 5525 2350
+Wire Wire Line
+	5325 2050 5525 2050
+Wire Wire Line
+	5325 2650 5525 2650
+Wire Wire Line
+	5325 2950 5525 2950
+Wire Wire Line
+	5325 3250 5525 3250
+Wire Wire Line
+	5325 3550 5525 3550
+Wire Wire Line
+	5325 4750 5525 4750
+Wire Wire Line
+	5325 5050 5525 5050
+Wire Wire Line
+	5325 5350 5525 5350
+Wire Wire Line
+	5325 5650 5525 5650
+Wire Wire Line
+	5325 5950 5525 5950
+Wire Wire Line
+	5325 6250 5525 6250
+Wire Wire Line
+	4500 7150 4500 7350
+Wire Wire Line
+	4200 7150 4200 7350
+Wire Wire Line
+	3900 7150 3900 7350
+Wire Wire Line
+	3600 7150 3600 7350
+Wire Wire Line
+	3300 7150 3300 7350
+Wire Wire Line
+	3000 7150 3000 7350
+Wire Wire Line
+	2175 6250 1975 6250
+Wire Wire Line
+	2175 5950 1975 5950
+Wire Wire Line
+	2175 5650 1975 5650
+Wire Wire Line
+	2175 5350 1975 5350
+Wire Wire Line
+	2175 5050 1975 5050
+Wire Wire Line
+	2175 4750 1975 4750
+Wire Wire Line
+	2175 3550 1970 3550
+Wire Wire Line
+	2175 3250 1975 3250
+Wire Wire Line
+	2175 2950 1975 2950
+Wire Wire Line
+	2175 2650 1975 2650
+Wire Wire Line
+	2175 2350 1975 2350
+Wire Wire Line
+	2175 2050 1975 2050
+Wire Wire Line
+	3000 3850 3000 3650
+Wire Wire Line
+	3300 3850 3300 3650
+Wire Wire Line
+	3600 3850 3600 3650
+Wire Wire Line
+	3900 3850 3900 3650
+Wire Wire Line
+	4200 3850 4200 3650
+Wire Wire Line
+	4500 3850 4500 3650
+Wire Wire Line
+	2725 3625 2925 3625
+Wire Wire Line
+	4425 6500 4425 6600
+Wire Wire Line
+	2800 6500 4425 6500
+Wire Wire Line
+	2800 6500 2800 6825
+Wire Wire Line
+	4125 6600 4125 6500
+Connection ~ 4125 6500
+Wire Wire Line
+	3825 6600 3825 6500
+Connection ~ 3825 6500
+Wire Wire Line
+	3525 6600 3525 6500
+Connection ~ 3525 6500
+Wire Wire Line
+	3225 6600 3225 6500
+Connection ~ 3225 6500
+Wire Wire Line
+	2925 6600 2925 6500
+Connection ~ 2925 6500
+Wire Wire Line
+	4575 6600 4575 6450
+Wire Wire Line
+	4575 6450 2750 6450
+Wire Wire Line
+	2750 6450 2750 6825
+Wire Wire Line
+	4275 6600 4275 6450
+Connection ~ 4275 6450
+Wire Wire Line
+	3975 6600 3975 6450
+Connection ~ 3975 6450
+Wire Wire Line
+	3675 6600 3675 6450
+Connection ~ 3675 6450
+Wire Wire Line
+	3375 6600 3375 6450
+Connection ~ 3375 6450
+Wire Wire Line
+	3075 6600 3075 6450
+Connection ~ 3075 6450
 $EndSCHEMATC

Commit message: PCB work.
Connections:
- net labels added: D1S5G, D1S5R
- wire segments 59 -> 152

Commit message: Worked on PCB
Parts:
- added Q? (x4): FDG1024NZ, SC70-6, symbol FDG1024NZ
- added R? (x4): 10K, symbol R
Connections:
- net labels added: D1S1G, D1S1R, D1S2G, D1S2R, D1S3G, D1S3R, D1S4G, D1S4R, D1S6G, D1S6R, D1S7G, D1S7R, GND
- wire segments 152 -> 263
Other:
- moved on the sheet: D3A

Commit message: Worked on schematic.
Parts:
- added Q? (x10): FDG1024NZ, SC70-6, symbol FDG1024NZ
- added R? (x10): 10K, symbol R
Connections:
- net D1S1G: now also Q?.2 (G), Q?.6 (D), R?.1
- net D1S1R: now also Q?.2 (G), R?.1; no longer D3.11 (D1S1), D3.14 (D1S1), D3.17 (D1S1), D3.2 (D1S1), D3.5 (D1S1), D3.8 (D1S1)
- net D1S2G: now also Q?.2 (G), R?.1; no longer D3.21 (D1S2), D3.24 (D1S2), D3.27 (D1S2), D3.30 (D1S2), D3.33 (D1S2), D3.36 (D1S2)
- net D1S2R: now also Q?.2 (G), R?.1; no longer D3.20 (D1S2), D3.23 (D1S2), D3.26 (D1S2), D3.29 (D1S2), D3.32 (D1S2), D3.35 (D1S2)
- net D1S3G: now also Q?.2 (G), R?.1; no longer D3.39 (D1S2), D3.42 (D1S2), D3.45 (D1S2), D3.48 (D1S2), D3.51 (D1S2), D3.54 (D1S2)
- net D1S3R: now also Q?.2 (G), R?.1; no longer D3.38 (D1S2), D3.41 (D1S3), D3.44 (D1S3), D3.47 (D1S2), D3.50 (D1S3), D3.53 (D1S2)
- net D1S4G: now also Q?.2 (G), R?.1; no longer D3.57 (D1S4), D3.60 (D1S4), D3.63 (D1S4), D3.66 (D1S4), D3.69 (D1S4), D3.72 (D1S4)
- net D1S4R: now also Q?.2 (G), R?.1; no longer D3.56 (D1S4), D3.59 (D1S4), D3.62 (D1S4), D3.65 (D1S4), D3.68 (D1S4), D3.71 (D1S4)
- net D1S7G: now also Q?.2 (G), R?.1; no longer D3.111 (D1S7), D3.114 (D1S7), D3.117 (D1S7), D3.120 (D1S7), D3.123 (D1S7), D3.126 (D1S7)
- net D1S7R: now also Q?.2 (G), R?.1; no longer D3.110 (D1S7), D3.113 (D1S7), D3.119 (D1S7), D3.122 (D1S7), D3.125 (D1S7)
- net GND: now also Q?.1 (S), Q?.1 (S), Q?.1 (S), Q?.1 (S), Q?.1 (S), Q?.1 (S), Q?.1 (S), Q?.1 (S), Q?.1 (S), Q?.1 (S), R?.2, R?.2, R?.2, R?.2, R?.2, R?.2, R?.2, R?.2, R?.2, R?.2
- new net: D3.11 (D1S1), D3.14 (D1S1), D3.17 (D1S1), D3.2 (D1S1), D3.5 (D1S1), D3.8 (D1S1), Q?.6 (D)
- new net: D3.110 (D1S7), D3.113 (D1S7), D3.119 (D1S7), D3.122 (D1S7), D3.125 (D1S7), Q?.6 (D)
- new net: D3.111 (D1S7), D3.114 (D1S7), D3.117 (D1S7), D3.120 (D1S7), D3.123 (D1S7), D3.126 (D1S7), Q?.6 (D)
- new net: D3.20 (D1S2), D3.23 (D1S2), D3.26 (D1S2), D3.29 (D1S2), D3.32 (D1S2), D3.35 (D1S2), Q?.6 (D)
- new net: D3.21 (D1S2), D3.24 (D1S2), D3.27 (D1S2), D3.30 (D1S2), D3.33 (D1S2), D3.36 (D1S2), Q?.6 (D)
- new net: D3.38 (D1S2), D3.41 (D1S3), D3.44 (D1S3), D3.47 (D1S2), D3.50 (D1S3), D3.53 (D1S2), Q?.6 (D)
- new net: D3.39 (D1S2), D3.42 (D1S2), D3.45 (D1S2), D3.48 (D1S2), D3.51 (D1S2), D3.54 (D1S2), Q?.6 (D)
- new net: D3.56 (D1S4), D3.59 (D1S4), D3.62 (D1S4), D3.65 (D1S4), D3.68 (D1S4), D3.71 (D1S4), Q?.6 (D)
- new net: D3.57 (D1S4), D3.60 (D1S4), D3.63 (D1S4), D3.66 (D1S4), D3.69 (D1S4), D3.72 (D1S4), Q?.6 (D)

Commit message: Updated schematic.
Connections:
- net at D3.110 (D1S7), D3.113 (D1S7), D3.119 (D1S7)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: now also D3.116 (D1S7)
Changed lines of the file:
@@
 Connection ~ 3930 4550
-Wire Wire Line
-	4235 4400 4235 4550
-Connection ~ 4235 4550
 Wire Wire Line
 	4530 4400 4530 4550
@@
 	3780 1700 3780 1800
 Wire Wire Line
-	5405 1800 3780 1800
-Wire Wire Line
-	5405 675  5405 1800
+	3780 1800 5405 1800
+Wire Wire Line
+	5405 1800 5405 675
 Wire Wire Line
 	3930 1700 3930 1850
@@
 Wire Wire Line
 	5405 675  8800 675
+Wire Wire Line
+	4230 4400 4230 4550
+Connection ~ 4230 4550
 $EndSCHEMATC

Commit message: Updated schematic.
Connections:
- net D1S1G: no longer D3.12 (D1S1), D3.15 (D1S1), D3.18 (D1S1), D3.3 (D1S1), D3.6 (D1S1), D3.9 (D1S1), Q?.6 (D)
- new net: D3.12 (D1S1), D3.15 (D1S1), D3.18 (D1S1), D3.3 (D1S1), D3.6 (D1S1), D3.9 (D1S1), Q?.6 (D)
Changed lines of the file:
@@
 Text Label 2680 2050 0    50   ~ 0
 D1A6
-Text Label 5405 950  3    50   ~ 0
-D1S1G
 $Comp
 L FDG1024NZ Q?
