File: PCB/Digit1.sch (KiCad schematic (older format))
At the start: 29 parts

Commit message: Added additional mosfets.
Parts:
- added Q? (x6): DMN2041LSD-13, SO-8, symbol DMN2041LSD-13
- added R? (x6): 10K, Resistors_SMD:R_0603_HandSoldering, symbol R
- Q23, Q24, Q25, Q26, Q27, Q28, Q29: renamed from Q?; footprint SO-8 -> Power_Integrations:SO-8
- R49, R50, R51, R52, R53, R54, R55, R56, R57, R58, R59, R60, R61, R62: renamed from R?; footprint (none) -> Resistors_SMD:R_0603_HandSoldering
Connections:
- net labels added: +3V3, A1, A2, A3, A4, A5, A6
- wire segments 257 -> 287

Commit message: Added additional mosfets.
Parts:
- removed Q? (x5): DMN2041LSD-13, SO-8, symbol DMN2041LSD-13
- removed R? (x6): 10K, Resistors_SMD:R_0603_HandSoldering, symbol R
- added Q? (x5): DMN2041LSD-13, SO-8, symbol DMN2041LSD-13
- added R? (x6): 10K, Resistors_SMD:R_0603_HandSoldering, symbol R
- added R? (x6): 150, Resistors_SMD:R_0603_HandSoldering, symbol R
Connections:
- net labels added: +5V
- net labels removed: +3V3
- wire segments 287 -> 293

Commit message: Edit PCB.
Parts:
- gave numbers to parts that had none: 15

Commit message: PCB work.
Parts:
- removed Q39, Q40, Q41: DMN2041LSD-13, SO-8, symbol DMN2041LSD-13
- removed R100, R103, R104, R107, R108, R99: 10K, Resistors_SMD:R_0603_HandSoldering, symbol R
- removed R101, R102, R105, R106, R109, R110: 150, Resistors_SMD:R_0603_HandSoldering, symbol R
- renumbered Q23 to Q26, Q24 to Q27, Q25 to Q28, Q26 to Q29, Q27 to Q30, Q28 to Q31, Q29 to Q32, R49 to R61, R50 to R62, R51 to R63, R52 to R64, R53 to R65, R54 to R66, R55 to R67, R56 to R68, R57 to R69, R58 to R70, R59 to R71, R60 to R72, R61 to R73, R62 to R74
Connections:
- net labels removed: +5V
- wire segments 293 -> 257

Commit message: PCB work.
Parts:
- Q26, Q27, Q28, Q29, Q30, Q31, Q32: footprint Power_Integrations:SO-8 -> Custom:SOIC-8_3.9x4.9mm_Pitch1.27mm
- R61, R62, R63, R64, R65, R66, R67, R68, R69, R70, R71, R72, R73, R74: footprint Resistors_SMD:R_0603_HandSoldering -> Resistors_SMD:R_0402
Changed lines of the file:
@@
 F 0 "R63" V 1080 2725 40  0000 C CNN
 F 1 "10K" V 1007 2726 40  0000 C CNN
-F 2 "Resistors_SMD:R_0603_HandSoldering" V 930 2725 30  0001 C CNN
+F 2 "Resistors_SMD:R_0402" V 930 2725 30  0001 C CNN
 F 3 "" H 1000 2725 30  0000 C CNN
 	1    1000 2725
@@
 F 0 "R64" V 2080 2725 40  0000 C CNN
 F 1 "10K" V 2007 2726 40  0000 C CNN
-F 2 "Resistors_SMD:R_0603_HandSoldering" V 1930 2725 30  0001 C CNN
+F 2 "Resistors_SMD:R_0402" V 1930 2725 30  0001 C CNN
 F 3 "" H 2000 2725 30  0000 C CNN
 	1    2000 2725
@@
 F 0 "R69" V 1080 5425 40  0000 C CNN
 F 1 "10K" V 1007 5426 40  0000 C CNN
-F 2 "Resistors_SMD:R_0603_HandSoldering" V 930 5425 30  0001 C CNN
+F 2 "Resistors_SMD:R_0402" V 930 5425 30  0001 C CNN
 F 3 "" H 1000 5425 30  0000 C CNN
 	1    1000 5425
@@
 F 0 "R70" V 2080 5425 40  0000 C CNN
 F 1 "10K" V 2007 5426 40  0000 C CNN
-F 2 "Resistors_SMD:R_0603_HandSoldering" V 1930 5425 30  0001 C CNN
+F 2 "Resistors_SMD:R_0402" V 1930 5425 30  0001 C CNN
 F 3 "" H 2000 5425 30  0000 C CNN
 	1    2000 5425
@@
 F 0 "R73" V 1080 7200 40  0000 C CNN
 F 1 "10K" V 1007 7201 40  0000 C CNN
-F 2 "Resistors_SMD:R_0603_HandSoldering" V 930 7200 30  0001 C CNN
+F 2 "Resistors_SMD:R_0402" V 930 7200 30  0001 C CNN
 F 3 "" H 1000 7200 30  0000 C CNN
 	1    1000 7200
@@
 F 0 "R74" V 2080 7200 40  0000 C CNN
 F 1 "10K" V 2007 7201 40  0000 C CNN
-F 2 "Resistors_SMD:R_0603_HandSoldering" V 1930 7200 30  0001 C CNN
+F 2 "Resistors_SMD:R_0402" V 1930 7200 30  0001 C CNN
 F 3 "" H 2000 7200 30  0000 C CNN
 	1    2000 7200
@@
 F 0 "R61" V 7430 1500 40  0000 C CNN
 F 1 "10K" V 7357 1501 40  0000 C CNN
-F 2 "Resistors_SMD:R_0603_HandSoldering" V 7280 1500 30  0001 C CNN
+F 2 "Resistors_SMD:R_0402" V 7280 1500 30  0001 C CNN
 F 3 "" H 7350 1500 30  0000 C CNN
 	1    7350 1500
@@
 F 0 "R62" V 8430 1500 40  0000 C CNN
 F 1 "10K" V 8357 1501 40  0000 C CNN
-F 2 "Resistors_SMD:R_0603_HandSoldering" V 8280 1500 30  0001 C CNN
+F 2 "Resistors_SMD:R_0402" V 8280 1500 30  0001 C CNN
 F 3 "" H 8350 1500 30  0000 C CNN
 	1    8350 1500
@@
 F 0 "R65" V 7430 3000 40  0000 C CNN
 F 1 "10K" V 7357 3001 40  0000 C CNN
-F 2 "Resistors_SMD:R_0603_HandSoldering" V 7280 3000 30  0001 C CNN
+F 2 "Resistors_SMD:R_0402" V 7280 3000 30  0001 C CNN
 F 3 "" H 7350 3000 30  0000 C CNN
 	1    7350 3000
@@
 F 0 "R66" V 8430 3000 40  0000 C CNN
 F 1 "10K" V 8357 3001 40  0000 C CNN
-F 2 "Resistors_SMD:R_0603_HandSoldering" V 8280 3000 30  0001 C CNN
+F 2 "Resistors_SMD:R_0402" V 8280 3000 30  0001 C CNN
 F 3 "" H 8350 3000 30  0000 C CNN
 	1    8350 3000
@@
 F 0 "R71" V 7430 5860 40  0000 C CNN
 F 1 "10K" V 7357 5861 40  0000 C CNN
-F 2 "Resistors_SMD:R_0603_HandSoldering" V 7280 5860 30  0001 C CNN
+F 2 "Resistors_SMD:R_0402" V 7280 5860 30  0001 C CNN
 F 3 "" H 7350 5860 30  0000 C CNN
 	1    7350 5860
@@
 F 0 "R72" V 8430 5860 40  0000 C CNN
 F 1 "10K" V 8357 5861 40  0000 C CNN
-F 2 "Resistors_SMD:R_0603_HandSoldering" V 8280 5860 30  0001 C CNN
+F 2 "Resistors_SMD:R_0402" V 8280 5860 30  0001 C CNN
 F 3 "" H 8350 5860 30  0000 C CNN
 	1    8350 5860
@@
 F 0 "R67" V 7430 4385 40  0000 C CNN
 F 1 "10K" V 7357 4386 40  0000 C CNN
-F 2 "Resistors_SMD:R_0603_HandSoldering" V 7280 4385 30  0001 C CNN
+F 2 "Resistors_SMD:R_0402" V 7280 4385 30  0001 C CNN
 F 3 "" H 7350 4385 30  0000 C CNN
 	1    7350 4385
@@
 F 0 "R68" V 8430 4385 40  0000 C CNN
 F 1 "10K" V 8357 4386 40  0000 C CNN
-F 2 "Resistors_SMD:R_0603_HandSoldering" V 8280 4385 30  0001 C CNN
+F 2 "Resistors_SMD:R_0402" V 8280 4385 30  0001 C CNN
 F 3 "" H 8350 4385 30  0000 C CNN
 	1    8350 4385
@@
 F 0 "Q27" H 1350 2201 40  0000 R CNN
 F 1 "DMN2041LSD-13" H 1350 2500 40  0000 R CNN
-F 2 "Power_Integrations:SO-8" H 1220 2452 29  0001 C CNN
+F 2 "Custom:SOIC-8_3.9x4.9mm_Pitch1.27mm" H 1220 2452 29  0001 C CNN
 F 3 "" H 1350 2350 60  0000 C CNN
 	1    1350 2350
@@
 F 0 "Q27" H 2350 2201 40  0000 R CNN
 F 1 "DMN2041LSD-13" H 2350 2500 40  0000 R CNN
-F 2 "Power_Integrations:SO-8" H 2220 2452 29  0001 C CNN
+F 2 "Custom:SOIC-8_3.9x4.9mm_Pitch1.27mm" H 2220 2452 29  0001 C CNN
 F 3 "" H 2350 2350 60  0000 C CNN
 	2    2350 2350
@@
 F 0 "Q30" H 1350 4901 40  0000 R CNN
 F 1 "DMN2041LSD-13" H 1350 5200 40  0000 R CNN
-F 2 "Power_Integrations:SO-8" H 1220 5152 29  0001 C CNN
+F 2 "Custom:SOIC-8_3.9x4.9mm_Pitch1.27mm" H 1220 5152 29  0001 C CNN
 F 3 "" H 1350 5050 60  0000 C CNN
 	1    1350 5050
@@
 F 0 "Q30" H 2350 4901 40  0000 R CNN
 F 1 "DMN2041LSD-13" H 2350 5200 40  0000 R CNN
-F 2 "Power_Integrations:SO-8" H 2220 5152 29  0001 C CNN
+F 2 "Custom:SOIC-8_3.9x4.9mm_Pitch1.27mm" H 2220 5152 29  0001 C CNN
 F 3 "" H 2350 5050 60  0000 C CNN
 	2    2350 5050
@@
 F 0 "Q32" H 1350 6676 40  0000 R CNN
 F 1 "DMN2041LSD-13" H 1350 6975 40  0000 R CNN
-F 2 "Power_Integrations:SO-8" H 1220 6927 29  0001 C CNN
+F 2 "Custom:SOIC-8_3.9x4.9mm_Pitch1.27mm" H 1220 6927 29  0001 C CNN
 F 3 "" H 1350 6825 60  0000 C CNN
 	1    1350 6825
@@
 F 0 "Q32" H 2350 6676 40  0000 R CNN
 F 1 "DMN2041LSD-13" H 2350 6975 40  0000 R CNN
-F 2 "Power_Integrations:SO-8" H 2220 6927 29  0001 C CNN
+F 2 "Custom:SOIC-8_3.9x4.9mm_Pitch1.27mm" H 2220 6927 29  0001 C CNN
 F 3 "" H 2350 6825 60  0000 C CNN
 	2    2350 6825
@@
 F 0 "Q31" H 7700 5336 40  0000 R CNN
 F 1 "DMN2041LSD-13" H 7700 5635 40  0000 R CNN
-F 2 "Power_Integrations:SO-8" H 7570 5587 29  0001 C CNN
+F 2 "Custom:SOIC-8_3.9x4.9mm_Pitch1.27mm" H 7570 5587 29  0001 C CNN
 F 3 "" H 7700 5485 60  0000 C CNN
 	1    7700 5485
@@
 F 0 "Q29" H 7700 3861 40  0000 R CNN
 F 1 "DMN2041LSD-13" H 7700 4160 40  0000 R CNN
-F 2 "Power_Integrations:SO-8" H 7570 4112 29  0001 C CNN
+F 2 "Custom:SOIC-8_3.9x4.9mm_Pitch1.27mm" H 7570 4112 29  0001 C CNN
 F 3 "" H 7700 4010 60  0000 C CNN
 	1    7700 4010
@@
 F 0 "Q28" H 7700 2476 40  0000 R CNN
 F 1 "DMN2041LSD-13" H 7700 2775 40  0000 R CNN
-F 2 "Power_Integrations:SO-8" H 7570 2727 29  0001 C CNN
+F 2 "Custom:SOIC-8_3.9x4.9mm_Pitch1.27mm" H 7570 2727 29  0001 C CNN
 F 3 "" H 7700 2625 60  0000 C CNN
 	1    7700 2625
@@
 F 0 "Q26" H 7700 976 40  0000 R CNN
 F 1 "DMN2041LSD-13" H 7700 1275 40  0000 R CNN
-F 2 "Power_Integrations:SO-8" H 7570 1227 29  0001 C CNN
+F 2 "Custom:SOIC-8_3.9x4.9mm_Pitch1.27mm" H 7570 1227 29  0001 C CNN
 F 3 "" H 7700 1125 60  0000 C CNN
 	1    7700 1125
@@
 F 0 "Q26" H 8700 976 40  0000 R CNN
 F 1 "DMN2041LSD-13" H 8700 1275 40  0000 R CNN
-F 2 "Power_Integrations:SO-8" H 8570 1227 29  0001 C CNN
+F 2 "Custom:SOIC-8_3.9x4.9mm_Pitch1.27mm" H 8570 1227 29  0001 C CNN
 F 3 "" H 8700 1125 60  0000 C CNN
 	2    8700 1125
@@
 F 0 "Q28" H 8700 2476 40  0000 R CNN
 F 1 "DMN2041LSD-13" H 8700 2775 40  0000 R CNN
-F 2 "Power_Integrations:SO-8" H 8570 2727 29  0001 C CNN
+F 2 "Custom:SOIC-8_3.9x4.9mm_Pitch1.27mm" H 8570 2727 29  0001 C CNN
 F 3 "" H 8700 2625 60  0000 C CNN
 	2    8700 2625
@@
 F 0 "Q29" H 8700 3861 40  0000 R CNN
 F 1 "DMN2041LSD-13" H 8700 4160 40  0000 R CNN
-F 2 "Power_Integrations:SO-8" H 8570 4112 29  0001 C CNN
+F 2 "Custom:SOIC-8_3.9x4.9mm_Pitch1.27mm" H 8570 4112 29  0001 C CNN
 F 3 "" H 8700 4010 60  0000 C CNN
 	2    8700 4010
@@
 F 0 "Q31" H 8700 5336 40  0000 R CNN
 F 1 "DMN2041LSD-13" H 8700 5635 40  0000 R CNN
-F 2 "Power_Integrations:SO-8" H 8570 5587 29  0001 C CNN
+F 2 "Custom:SOIC-8_3.9x4.9mm_Pitch1.27mm" H 8570 5587 29  0001 C CNN
 F 3 "" H 8700 5485 60  0000 C CNN
 	2    8700 5485

Commit message: PCB work.
Parts:
- R61, R62, R63, R64, R65, R66, R67, R68, R69, R70, R71, R72, R73, R74: symbol R -> R-RESCUE-7SegClock
Changed lines of the file:
@@
 EESchema Schematic File Version 2
+LIBS:7SegClock-rescue
 LIBS:power
 LIBS:device
@@
 LIBS:memory
 LIBS:xilinx
-LIBS:special
 LIBS:microcontrollers
 LIBS:dsp
@@
 D1A6
 $Comp
-L R R63
+L R-RESCUE-7SegClock R63
 U 1 1 54C62D5E
 P 1000 2725
@@
 $EndComp
 $Comp
-L R R64
+L R-RESCUE-7SegClock R64
 U 1 1 54C62E2F
 P 2000 2725
@@
 $EndComp
 $Comp
-L R R69
+L R-RESCUE-7SegClock R69
 U 1 1 54C6512D
 P 1000 5425
@@
 $EndComp
 $Comp
-L R R70
+L R-RESCUE-7SegClock R70
 U 1 1 54C65133
 P 2000 5425
@@
 D1S5G
 $Comp
-L R R73
+L R-RESCUE-7SegClock R73
 U 1 1 54E98C02
 P 1000 7200
@@
 $EndComp
 $Comp
-L R R74
+L R-RESCUE-7SegClock R74
 U 1 1 54E98C08
 P 2000 7200
@@
 	2450 6625 2450 6500
 $Comp
-L R R61
+L R-RESCUE-7SegClock R61
 U 1 1 54E9A80E
 P 7350 1500
@@
 $EndComp
 $Comp
-L R R62
+L R-RESCUE-7SegClock R62
 U 1 1 54E9A814
 P 8350 1500
@@
 	8800 675  8800 925
 $Comp
-L R R65
+L R-RESCUE-7SegClock R65
 U 1 1 54E9ABE5
 P 7350 3000
@@
 $EndComp
 $Comp
-L R R66
+L R-RESCUE-7SegClock R66
 U 1 1 54E9ABEB
 P 8350 3000
@@
 	8800 2125 8800 2425
 $Comp
-L R R71
+L R-RESCUE-7SegClock R71
 U 1 1 54E9ADA0
 P 7350 5860
@@
 $EndComp
 $Comp
-L R R72
+L R-RESCUE-7SegClock R72
 U 1 1 54E9ADA6
 P 8350 5860
@@
 	7800 750  7800 925
 $Comp
-L R R67
+L R-RESCUE-7SegClock R67
 U 1 1 54E9E0BA
 P 7350 4385
@@
 $EndComp
 $Comp
-L R R68
+L R-RESCUE-7SegClock R68
 U 1 1 54E9E0C0
 P 8350 4385
@@
 BC 01 60 96 31 E6 05 00 CF E7 7F 1E 6D 7A 11 6D 4B 35 E4 B7 1B 6B 03 D8 50 55 DF E5 BD 5F 0B 59
 F0 3A 1E C0 38 64 CF D4 F2 C8 9E A9 05 CC 43 F6 BE 79 15 99 0A D7 74 00 CF 02 78 CE 18 F3 24 80
-47 91 3D 63 3D 51 4F 11 C2 FF 03 CA 62 49 C8 E1 A2 25 5C 00 00 00 00 49 45 4E 44 AE 42 60 82 00
+47 91 3D 63 3D 51 4F 11 C2 FF 03 CA 62 49 C8 E1 A2 25 5C 00 00 00 00 49 45 4E 44 AE 42 60 82 CC
 EndData
 $EndBitmap
