File: PCB/7SegClock.kicad_pcb (KiCad board)
At the start: 2 copper layers, 177.8 x 76.2 mm, 185 parts, among them CON1 USB-MINI-B, Q1 NPN, Q10 DMN2041LSD-13, Q11 DMN2041LSD-13, Q12 DMN2041LSD-13, Q13 DMN2041LSD-13, Q14 DMN2041LSD-13, Q15 DMN2041LSD-13, Q16 DMN2041LSD-13, Q17 DMN2041LSD-13, Q18 DMN2041LSD-13, Q19 DMN2041LSD-13, Q2 DMN2041LSD-13, Q20 DMN2041LSD-13, Q21 DMN2041LSD-13, Q22 DMN2041LSD-13, Q23 DMN2041LSD-13, Q24 DMN2041LSD-13, Q25 DMN2041LSD-13, Q26 DMN2041LSD-13, Q27 DMN2041LSD-13, Q28 DMN2041LSD-13, Q29 DMN2041LSD-13, Q3 DMN2041LSD-13, Q30 DMN2041LSD-13, Q31 DMN2041LSD-13, Q32 DMN2041LSD-13, Q33 DMN2041LSD-13, Q34 DMN2041LSD-13, Q35 DMN2041LSD-13, Q36 DMN2041LSD-13, Q37 DMN2041LSD-13, Q38 DMN2041LSD-13, Q39 DMN2041LSD-13, Q4 DMN2041LSD-13, Q40 DMN2041LSD-13, Q41 DMN2041LSD-13, Q5 DMN2041LSD-13, Q6 DMN2041LSD-13, Q7 DMN2041LSD-13, Q8 DMN2041LSD-13, Q9 DMN2041LSD-13, U1 TPS62172DSGT, U2 P8X32A, U3 FT232RL, U4 24LC256, U5 DS3231, U6 LCMX02-640UHC-4TG144C, X1 5mhz CRYSTAL

Commit message: Worked on PCB.
Parts:
- moved R41 174.7 mm to (302.1, 47.2)
- moved R46 174.7 mm to (288.5, 53.2)
- moved R35 174.7 mm to (306.5, 35.2)
- moved R36 174.7 mm to (274.9, 56.3)
- moved R37 174.7 mm to (302.2, 53.2)
- moved R38 174.7 mm to (306.6, 47.2)
- moved R39 174.7 mm to (297.6, 53.2)
- moved R40 174.7 mm to (311.1, 41.2)
- moved R42 174.7 mm to (311.1, 35.2)
- moved R43 174.7 mm to (293.1, 53.2)
- moved R44 174.7 mm to (306.5, 41.2)
- moved R45 174.7 mm to (297.5, 47.2)
- moved R47 174.7 mm to (284.0, 54.7)
- moved R48 174.7 mm to (302.0, 41.2)
- moved R63 174.7 mm to (302.0, 35.2)
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Routing:
- net /Lattice MACHXO2/Digit_1/D1A4: track 0.00 -> 87.9 mm
- net /Lattice MACHXO2/Digit_1/D1A6: track 13.8 -> 94.5 mm
- net /Lattice MACHXO2/Digit_1/D1A1: track 0.00 -> 69.6 mm
- net /Lattice MACHXO2/Digit_1/D1A5: track 29.4 -> 91.6 mm
- net /Lattice MACHXO2/Digit_1/D1A3: track 0.00 -> 56.8 mm
- net /Lattice MACHXO2/Digit_1/D1A2: track 0.00 -> 47.4 mm
- net Net-(D3-Pad74): track 0.00 -> 25.0 mm
- net Net-(D3-Pad218): track 0.00 -> 24.6 mm
- net Net-(D3-Pad20): track 0.00 -> 24.6 mm
- net Net-(D3-Pad219): track 0.00 -> 24.4 mm
- net Net-(D3-Pad75): track 0.00 -> 24.3 mm
- net Net-(D3-Pad102): track 0.00 -> 24.3 mm
- net Net-(D3-Pad21): track 0.00 -> 24.2 mm
- net Net-(D3-Pad101): track 0.00 -> 23.8 mm
- net Net-(D3-Pad11): track 0.00 -> 23.7 mm
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
Commit message: PCB work.
Parts:
- moved Q8 8.63 mm to (102.9, 127.1)
Routing:
- net /Lattice MACHXO2/Digit_1/D1A4: track 87.9 -> 256.3 mm
- net /Lattice MACHXO2/Digit_1/D1A5: track 91.6 -> 256.2 mm
- net /Lattice MACHXO2/Digit_1/D1A6: track 94.5 -> 254.8 mm
- net /Lattice MACHXO2/Digit_1/D1A3: track 56.8 -> 138.1 mm
- net /Lattice MACHXO2/Digit_1/D1A2: track 47.4 -> 113.8 mm
- net Net-(D3-Pad39): track 0.00 -> 24.6 mm
- net Net-(D3-Pad38): track 0.00 -> 24.5 mm
- net /Lattice MACHXO2/Digit_1/D1A1: track 69.6 -> 81.9 mm

Commit message: PCB work.
Parts:
- removed Q33, Q34, Q35, Q36, Q37, Q38, Q39, Q40, Q41: DMN2041LSD-13, SO-8
- removed R100, R103, R104, R107, R108, R75, R76, R79, R80, R83, R84, R87, R88, R91, R92, R95, R96, R99: 10K, Resistors_SMD:R_0603_HandSoldering
- removed R101, R102, R105, R106, R109, R110, R77, R78, R81, R82, R85, R86, R89, R90, R93, R94, R97, R98: 150, Resistors_SMD:R_0603_HandSoldering
- added REF**: SolderWirePad_single_2-5mmDrill, Wire_Pads:SolderWirePad_single_2mmDrill, F.Cu at (233.0, 52.7)
- Q10, Q11, Q12, Q13, Q14, Q15, Q16, Q17, Q18, Q19, Q2, Q20, Q21, Q22, Q23, Q24, Q25, Q26, Q27, Q28, Q29, Q3, Q30, Q31, Q32, Q4, Q5, Q6, Q7, Q8, Q9: footprint SO-8 -> Power_Integrations:SO-8
- R13, R14, R15, R16, R17, R18: value 10K -> 150
- R65, R66, R69, R70, R73, R74: value 150 -> 10K
- U5: moved to B.Cu
- moved R35 223.3 mm to (147.3, 191.7)
- moved R38 211.9 mm to (151.7, 191.7)
- moved R44 208.5 mm to (160.6, 190.1)
- moved C14 205.5 mm to (84.4, 169.5)
- moved C11 205.4 mm to (84.4, 175.4)
- moved R71 204.0 mm to (145.4, 171.2)
- moved R37 203.9 mm to (147.3, 185.8)
- moved R40 200.3 mm to (165.2, 178.3)
- moved C19 199.7 mm to (93.8, 175.4)
- moved C13 197.2 mm to (89.1, 175.4)
- moved R42 197.0 mm to (174.2, 176.8)
- moved R41 196.9 mm to (160.7, 184.2)
- moved R63 196.5 mm to (158.7, 169.6)
- moved R39 193.9 mm to (156.2, 185.8)
- moved C8 192.3 mm to (89.1, 169.5)
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Connections:
- D3 pad 1: /Lattice MACHXO2/Digit_1/D1A1 -> /Lattice MACHXO2/Digit_1/A1
- D3 pad 10: /Lattice MACHXO2/Digit_1/D1A4 -> /Lattice MACHXO2/Digit_1/A4
- D3 pad 100: /Lattice MACHXO2/Digit_1/D1A4 -> /Lattice MACHXO2/Digit_1/A4
- D3 pad 103: /Lattice MACHXO2/Digit_1/D1A5 -> /Lattice MACHXO2/Digit_1/A5
- D3 pad 106: /Lattice MACHXO2/Digit_1/D1A6 -> /Lattice MACHXO2/Digit_1/A6
- D3 pad 109: /Lattice MACHXO2/Digit_1/D1A1 -> /Lattice MACHXO2/Digit_1/A1
- D3 pad 112: /Lattice MACHXO2/Digit_1/D1A2 -> /Lattice MACHXO2/Digit_1/A2
- D3 pad 115: /Lattice MACHXO2/Digit_1/D1A3 -> /Lattice MACHXO2/Digit_1/A3
- D3 pad 118: /Lattice MACHXO2/Digit_1/D1A4 -> /Lattice MACHXO2/Digit_1/A4
- D3 pad 121: /Lattice MACHXO2/Digit_1/D1A5 -> /Lattice MACHXO2/Digit_1/A5
- D3 pad 124: /Lattice MACHXO2/Digit_1/D1A6 -> /Lattice MACHXO2/Digit_1/A6
- D3 pad 127: /Lattice MACHXO2/Digit_2/D2A1 -> /Lattice MACHXO2/Digit_1/A1
- D3 pad 13: /Lattice MACHXO2/Digit_1/D1A5 -> /Lattice MACHXO2/Digit_1/A5
- D3 pad 130: /Lattice MACHXO2/Digit_2/D2A2 -> /Lattice MACHXO2/Digit_1/A2
- D3 pad 133: /Lattice MACHXO2/Digit_2/D2A3 -> /Lattice MACHXO2/Digit_1/A3
- D3 pad 136: /Lattice MACHXO2/Digit_2/D2A4 -> /Lattice MACHXO2/Digit_1/A4
- D3 pad 139: /Lattice MACHXO2/Digit_2/D2A5 -> /Lattice MACHXO2/Digit_1/A5
- D3 pad 142: /Lattice MACHXO2/Digit_2/D2A6 -> /Lattice MACHXO2/Digit_1/A6
- D3 pad 145: /Lattice MACHXO2/Digit_2/D2A1 -> /Lattice MACHXO2/Digit_1/A1
- D3 pad 148: /Lattice MACHXO2/Digit_2/D2A2 -> /Lattice MACHXO2/Digit_1/A2
- D3 pad 151: /Lattice MACHXO2/Digit_2/D2A3 -> /Lattice MACHXO2/Digit_1/A3
- D3 pad 154: /Lattice MACHXO2/Digit_2/D2A4 -> /Lattice MACHXO2/Digit_1/A4
- D3 pad 157: /Lattice MACHXO2/Digit_2/D2A5 -> /Lattice MACHXO2/Digit_1/A5
- D3 pad 16: /Lattice MACHXO2/Digit_1/D1A6 -> /Lattice MACHXO2/Digit_1/A6
- D3 pad 160: /Lattice MACHXO2/Digit_2/D2A6 -> /Lattice MACHXO2/Digit_1/A6
- D3 pad 163: /Lattice MACHXO2/Digit_2/D2A1 -> /Lattice MACHXO2/Digit_1/A1
- D3 pad 166: /Lattice MACHXO2/Digit_2/D2A2 -> /Lattice MACHXO2/Digit_1/A2
- D3 pad 169: /Lattice MACHXO2/Digit_2/D2A3 -> /Lattice MACHXO2/Digit_1/A3
- D3 pad 172: /Lattice MACHXO2/Digit_2/D2A4 -> /Lattice MACHXO2/Digit_1/A4
- D3 pad 175: /Lattice MACHXO2/Digit_2/D2A5 -> /Lattice MACHXO2/Digit_1/A5
- D3 pad 178: /Lattice MACHXO2/Digit_2/D2A6 -> /Lattice MACHXO2/Digit_1/A6
- D3 pad 181: /Lattice MACHXO2/Digit_2/D2A1 -> /Lattice MACHXO2/Digit_1/A1
- D3 pad 184: /Lattice MACHXO2/Digit_2/D2A2 -> /Lattice MACHXO2/Digit_1/A2
- D3 pad 187: /Lattice MACHXO2/Digit_2/D2A3 -> /Lattice MACHXO2/Digit_1/A3
- D3 pad 19: /Lattice MACHXO2/Digit_1/D1A1 -> /Lattice MACHXO2/Digit_1/A1
- D3 pad 190: /Lattice MACHXO2/Digit_2/D2A4 -> /Lattice MACHXO2/Digit_1/A4
- D3 pad 193: /Lattice MACHXO2/Digit_2/D2A5 -> /Lattice MACHXO2/Digit_1/A5
- D3 pad 196: /Lattice MACHXO2/Digit_2/D2A6 -> /Lattice MACHXO2/Digit_1/A6
- D3 pad 199: /Lattice MACHXO2/Digit_2/D2A1 -> /Lattice MACHXO2/Digit_1/A1
- D3 pad 202: /Lattice MACHXO2/Digit_2/D2A2 -> /Lattice MACHXO2/Digit_1/A2
- D3 pad 205: /Lattice MACHXO2/Digit_2/D2A3 -> /Lattice MACHXO2/Digit_1/A3
- D3 pad 208: /Lattice MACHXO2/Digit_2/D2A4 -> /Lattice MACHXO2/Digit_1/A4
- D3 pad 211: /Lattice MACHXO2/Digit_2/D2A5 -> /Lattice MACHXO2/Digit_1/A5
- D3 pad 214: /Lattice MACHXO2/Digit_2/D2A6 -> /Lattice MACHXO2/Digit_1/A6
- D3 pad 217: /Lattice MACHXO2/Digit_2/D2A1 -> /Lattice MACHXO2/Digit_1/A1
- D3 pad 22: /Lattice MACHXO2/Digit_1/D1A2 -> /Lattice MACHXO2/Digit_1/A2
- D3 pad 220: /Lattice MACHXO2/Digit_2/D2A2 -> /Lattice MACHXO2/Digit_1/A2
- D3 pad 223: /Lattice MACHXO2/Digit_2/D2A3 -> /Lattice MACHXO2/Digit_1/A3
- D3 pad 226: /Lattice MACHXO2/Digit_2/D2A4 -> /Lattice MACHXO2/Digit_1/A4
- D3 pad 229: /Lattice MACHXO2/Digit_2/D2A5 -> /Lattice MACHXO2/Digit_1/A5
- D3 pad 232: /Lattice MACHXO2/Digit_2/D2A6 -> /Lattice MACHXO2/Digit_1/A6
- D3 pad 235: /Lattice MACHXO2/Digit_2/D2A1 -> /Lattice MACHXO2/Digit_1/A1
- D3 pad 238: /Lattice MACHXO2/Digit_2/D2A2 -> /Lattice MACHXO2/Digit_1/A2
- D3 pad 241: /Lattice MACHXO2/Digit_2/D2A3 -> /Lattice MACHXO2/Digit_1/A3
- D3 pad 242: Net-(D3-Pad242) -> Net-(D3-Pad236)
- D3 pad 244: /Lattice MACHXO2/Digit_2/D2A4 -> /Lattice MACHXO2/Digit_1/A4
- D3 pad 247: /Lattice MACHXO2/Digit_2/D2A5 -> /Lattice MACHXO2/Digit_1/A5
- D3 pad 25: /Lattice MACHXO2/Digit_1/D1A3 -> /Lattice MACHXO2/Digit_1/A3
- D3 pad 250: /Lattice MACHXO2/Digit_2/D2A6 -> /Lattice MACHXO2/Digit_1/A6
- D3 pad 253: /Lattice MACHXO2/Digit_3/D3A1 -> /Lattice MACHXO2/Digit_1/A1
- D3 pad 256: /Lattice MACHXO2/Digit_3/D3A2 -> /Lattice MACHXO2/Digit_1/A2
- D3 pad 259: /Lattice MACHXO2/Digit_3/D3A3 -> /Lattice MACHXO2/Digit_1/A3
- D3 pad 262: /Lattice MACHXO2/Digit_3/D3A4 -> /Lattice MACHXO2/Digit_1/A4
- D3 pad 265: /Lattice MACHXO2/Digit_3/D3A5 -> /Lattice MACHXO2/Digit_1/A5
- D3 pad 268: /Lattice MACHXO2/Digit_3/D3A6 -> /Lattice MACHXO2/Digit_1/A6
- D3 pad 271: /Lattice MACHXO2/Digit_3/D3A1 -> /Lattice MACHXO2/Digit_1/A1
- D3 pad 274: /Lattice MACHXO2/Digit_3/D3A2 -> /Lattice MACHXO2/Digit_1/A2
- D3 pad 277: /Lattice MACHXO2/Digit_3/D3A3 -> /Lattice MACHXO2/Digit_1/A3
- D3 pad 28: /Lattice MACHXO2/Digit_1/D1A4 -> /Lattice MACHXO2/Digit_1/A4
- D3 pad 280: /Lattice MACHXO2/Digit_3/D3A4 -> /Lattice MACHXO2/Digit_1/A4
- D3 pad 283: /Lattice MACHXO2/Digit_3/D3A5 -> /Lattice MACHXO2/Digit_1/A5
- D3 pad 286: /Lattice MACHXO2/Digit_3/D3A6 -> /Lattice MACHXO2/Digit_1/A6
- D3 pad 289: /Lattice MACHXO2/Digit_3/D3A1 -> /Lattice MACHXO2/Digit_1/A1
- D3 pad 292: /Lattice MACHXO2/Digit_3/D3A2 -> /Lattice MACHXO2/Digit_1/A2
- D3 pad 295: /Lattice MACHXO2/Digit_3/D3A3 -> /Lattice MACHXO2/Digit_1/A3
- D3 pad 298: /Lattice MACHXO2/Digit_3/D3A4 -> /Lattice MACHXO2/Digit_1/A4
- D3 pad 301: /Lattice MACHXO2/Digit_3/D3A5 -> /Lattice MACHXO2/Digit_1/A5
- D3 pad 304: /Lattice MACHXO2/Digit_3/D3A6 -> /Lattice MACHXO2/Digit_1/A6
- D3 pad 307: /Lattice MACHXO2/Digit_3/D3A1 -> /Lattice MACHXO2/Digit_1/A1
- D3 pad 31: /Lattice MACHXO2/Digit_1/D1A5 -> /Lattice MACHXO2/Digit_1/A5
- D3 pad 310: /Lattice MACHXO2/Digit_3/D3A2 -> /Lattice MACHXO2/Digit_1/A2
- D3 pad 313: /Lattice MACHXO2/Digit_3/D3A3 -> /Lattice MACHXO2/Digit_1/A3
- D3 pad 316: /Lattice MACHXO2/Digit_3/D3A4 -> /Lattice MACHXO2/Digit_1/A4
- D3 pad 319: /Lattice MACHXO2/Digit_3/D3A5 -> /Lattice MACHXO2/Digit_1/A5
- D3 pad 322: /Lattice MACHXO2/Digit_3/D3A6 -> /Lattice MACHXO2/Digit_1/A6
- D3 pad 325: /Lattice MACHXO2/Digit_3/D3A1 -> /Lattice MACHXO2/Digit_1/A1
- D3 pad 328: /Lattice MACHXO2/Digit_3/D3A2 -> /Lattice MACHXO2/Digit_1/A2
- D3 pad 331: /Lattice MACHXO2/Digit_3/D3A3 -> /Lattice MACHXO2/Digit_1/A3
- D3 pad 334: /Lattice MACHXO2/Digit_3/D3A4 -> /Lattice MACHXO2/Digit_1/A4
- D3 pad 337: /Lattice MACHXO2/Digit_3/D3A5 -> /Lattice MACHXO2/Digit_1/A5
- D3 pad 34: /Lattice MACHXO2/Digit_1/D1A6 -> /Lattice MACHXO2/Digit_1/A6
- D3 pad 340: /Lattice MACHXO2/Digit_3/D3A6 -> /Lattice MACHXO2/Digit_1/A6
- D3 pad 343: /Lattice MACHXO2/Digit_3/D3A1 -> /Lattice MACHXO2/Digit_1/A1
- D3 pad 346: /Lattice MACHXO2/Digit_3/D3A2 -> /Lattice MACHXO2/Digit_1/A2
- D3 pad 349: /Lattice MACHXO2/Digit_3/D3A3 -> /Lattice MACHXO2/Digit_1/A3
- D3 pad 352: /Lattice MACHXO2/Digit_3/D3A4 -> /Lattice MACHXO2/Digit_1/A4
- D3 pad 355: /Lattice MACHXO2/Digit_3/D3A5 -> /Lattice MACHXO2/Digit_1/A5
- D3 pad 358: /Lattice MACHXO2/Digit_3/D3A6 -> /Lattice MACHXO2/Digit_1/A6
- D3 pad 361: /Lattice MACHXO2/Digit_3/D3A1 -> /Lattice MACHXO2/Digit_1/A1
- D3 pad 364: /Lattice MACHXO2/Digit_3/D3A2 -> /Lattice MACHXO2/Digit_1/A2
- D3 pad 367: /Lattice MACHXO2/Digit_3/D3A3 -> /Lattice MACHXO2/Digit_1/A3
- D3 pad 368: Net-(D3-Pad368) -> Net-(D3-Pad362)
- D3 pad 37: /Lattice MACHXO2/Digit_1/D1A1 -> /Lattice MACHXO2/Digit_1/A1
- D3 pad 370: /Lattice MACHXO2/Digit_3/D3A4 -> /Lattice MACHXO2/Digit_1/A4
- D3 pad 373: /Lattice MACHXO2/Digit_3/D3A5 -> /Lattice MACHXO2/Digit_1/A5
- D3 pad 376: /Lattice MACHXO2/Digit_3/D3A6 -> /Lattice MACHXO2/Digit_1/A6
- D3 pad 379: /Lattice MACHXO2/Digit_4/D4A1 -> /Lattice MACHXO2/Digit_1/A1
- D3 pad 382: /Lattice MACHXO2/Digit_4/D4A2 -> /Lattice MACHXO2/Digit_1/A2
- D3 pad 385: /Lattice MACHXO2/Digit_4/D4A3 -> /Lattice MACHXO2/Digit_1/A3
- D3 pad 388: /Lattice MACHXO2/Digit_4/D4A4 -> /Lattice MACHXO2/Digit_1/A4
- D3 pad 391: /Lattice MACHXO2/Digit_4/D4A5 -> /Lattice MACHXO2/Digit_1/A5
- D3 pad 394: /Lattice MACHXO2/Digit_4/D4A6 -> /Lattice MACHXO2/Digit_1/A6
- D3 pad 397: /Lattice MACHXO2/Digit_4/D4A1 -> /Lattice MACHXO2/Digit_1/A1
- D3 pad 4: /Lattice MACHXO2/Digit_1/D1A2 -> /Lattice MACHXO2/Digit_1/A2
- D3 pad 40: /Lattice MACHXO2/Digit_1/D1A2 -> /Lattice MACHXO2/Digit_1/A2
- D3 pad 400: /Lattice MACHXO2/Digit_4/D4A2 -> /Lattice MACHXO2/Digit_1/A2
- D3 pad 403: /Lattice MACHXO2/Digit_4/D4A3 -> /Lattice MACHXO2/Digit_1/A3
- D3 pad 406: /Lattice MACHXO2/Digit_4/D4A4 -> /Lattice MACHXO2/Digit_1/A4
- D3 pad 409: /Lattice MACHXO2/Digit_4/D4A5 -> /Lattice MACHXO2/Digit_1/A5
- D3 pad 412: /Lattice MACHXO2/Digit_4/D4A6 -> /Lattice MACHXO2/Digit_1/A6
- D3 pad 415: /Lattice MACHXO2/Digit_4/D4A1 -> /Lattice MACHXO2/Digit_1/A1
- D3 pad 418: /Lattice MACHXO2/Digit_4/D4A2 -> /Lattice MACHXO2/Digit_1/A2
- D3 pad 421: /Lattice MACHXO2/Digit_4/D4A3 -> /Lattice MACHXO2/Digit_1/A3
- D3 pad 424: /Lattice MACHXO2/Digit_4/D4A4 -> /Lattice MACHXO2/Digit_1/A4
- D3 pad 427: /Lattice MACHXO2/Digit_4/D4A5 -> /Lattice MACHXO2/Digit_1/A5
- D3 pad 43: /Lattice MACHXO2/Digit_1/D1A3 -> /Lattice MACHXO2/Digit_1/A3
- D3 pad 430: /Lattice MACHXO2/Digit_4/D4A6 -> /Lattice MACHXO2/Digit_1/A6
- D3 pad 433: /Lattice MACHXO2/Digit_4/D4A1 -> /Lattice MACHXO2/Digit_1/A1
- D3 pad 436: /Lattice MACHXO2/Digit_4/D4A2 -> /Lattice MACHXO2/Digit_1/A2
- D3 pad 439: /Lattice MACHXO2/Digit_4/D4A3 -> /Lattice MACHXO2/Digit_1/A3
- D3 pad 442: /Lattice MACHXO2/Digit_4/D4A4 -> /Lattice MACHXO2/Digit_1/A4
- D3 pad 445: /Lattice MACHXO2/Digit_4/D4A5 -> /Lattice MACHXO2/Digit_1/A5
- D3 pad 448: /Lattice MACHXO2/Digit_4/D4A6 -> /Lattice MACHXO2/Digit_1/A6
- D3 pad 451: /Lattice MACHXO2/Digit_4/D4A1 -> /Lattice MACHXO2/Digit_1/A1
- D3 pad 454: /Lattice MACHXO2/Digit_4/D4A2 -> /Lattice MACHXO2/Digit_1/A2
- D3 pad 457: /Lattice MACHXO2/Digit_4/D4A3 -> /Lattice MACHXO2/Digit_1/A3
- D3 pad 46: /Lattice MACHXO2/Digit_1/D1A4 -> /Lattice MACHXO2/Digit_1/A4
- D3 pad 460: /Lattice MACHXO2/Digit_4/D4A4 -> /Lattice MACHXO2/Digit_1/A4
- D3 pad 463: /Lattice MACHXO2/Digit_4/D4A5 -> /Lattice MACHXO2/Digit_1/A5
- D3 pad 466: /Lattice MACHXO2/Digit_4/D4A6 -> /Lattice MACHXO2/Digit_1/A6
- D3 pad 469: /Lattice MACHXO2/Digit_4/D4A1 -> /Lattice MACHXO2/Digit_1/A1
- D3 pad 472: /Lattice MACHXO2/Digit_4/D4A2 -> /Lattice MACHXO2/Digit_1/A2
- D3 pad 475: /Lattice MACHXO2/Digit_4/D4A3 -> /Lattice MACHXO2/Digit_1/A3
- D3 pad 478: /Lattice MACHXO2/Digit_4/D4A4 -> /Lattice MACHXO2/Digit_1/A4
- D3 pad 481: /Lattice MACHXO2/Digit_4/D4A5 -> /Lattice MACHXO2/Digit_1/A5
- D3 pad 484: /Lattice MACHXO2/Digit_4/D4A6 -> /Lattice MACHXO2/Digit_1/A6
- D3 pad 487: /Lattice MACHXO2/Digit_4/D4A1 -> /Lattice MACHXO2/Digit_1/A1
- D3 pad 49: /Lattice MACHXO2/Digit_1/D1A5 -> /Lattice MACHXO2/Digit_1/A5
- D3 pad 490: /Lattice MACHXO2/Digit_4/D4A2 -> /Lattice MACHXO2/Digit_1/A2
- D3 pad 493: /Lattice MACHXO2/Digit_4/D4A3 -> /Lattice MACHXO2/Digit_1/A3
- D3 pad 496: /Lattice MACHXO2/Digit_4/D4A4 -> /Lattice MACHXO2/Digit_1/A4
- D3 pad 499: /Lattice MACHXO2/Digit_4/D4A5 -> /Lattice MACHXO2/Digit_1/A5
- D3 pad 502: /Lattice MACHXO2/Digit_4/D4A6 -> /Lattice MACHXO2/Digit_1/A6
- D3 pad 52: /Lattice MACHXO2/Digit_1/D1A6 -> /Lattice MACHXO2/Digit_1/A6
- D3 pad 55: /Lattice MACHXO2/Digit_1/D1A1 -> /Lattice MACHXO2/Digit_1/A1
- D3 pad 58: /Lattice MACHXO2/Digit_1/D1A2 -> /Lattice MACHXO2/Digit_1/A2
- D3 pad 61: /Lattice MACHXO2/Digit_1/D1A3 -> /Lattice MACHXO2/Digit_1/A3
- D3 pad 64: /Lattice MACHXO2/Digit_1/D1A4 -> /Lattice MACHXO2/Digit_1/A4
- D3 pad 67: /Lattice MACHXO2/Digit_1/D1A5 -> /Lattice MACHXO2/Digit_1/A5
- D3 pad 7: /Lattice MACHXO2/Digit_1/D1A3 -> /Lattice MACHXO2/Digit_1/A3
- D3 pad 70: /Lattice MACHXO2/Digit_1/D1A6 -> /Lattice MACHXO2/Digit_1/A6
- D3 pad 73: /Lattice MACHXO2/Digit_1/D1A1 -> /Lattice MACHXO2/Digit_1/A1
- D3 pad 76: /Lattice MACHXO2/Digit_1/D1A2 -> /Lattice MACHXO2/Digit_1/A2
- D3 pad 79: /Lattice MACHXO2/Digit_1/D1A3 -> /Lattice MACHXO2/Digit_1/A3
- D3 pad 82: /Lattice MACHXO2/Digit_1/D1A4 -> /Lattice MACHXO2/Digit_1/A4
- D3 pad 85: /Lattice MACHXO2/Digit_1/D1A5 -> /Lattice MACHXO2/Digit_1/A5
- D3 pad 88: /Lattice MACHXO2/Digit_1/D1A6 -> /Lattice MACHXO2/Digit_1/A6
- D3 pad 91: /Lattice MACHXO2/Digit_1/D1A1 -> /Lattice MACHXO2/Digit_1/A1
- D3 pad 94: /Lattice MACHXO2/Digit_1/D1A2 -> /Lattice MACHXO2/Digit_1/A2
- D3 pad 97: /Lattice MACHXO2/Digit_1/D1A3 -> /Lattice MACHXO2/Digit_1/A3
- Q10 pad 2: /Lattice MACHXO2/Digit_3/D3S6R -> /Lattice MACHXO2/Digit_4/D4S3R
- Q10 pad 4: /Lattice MACHXO2/Digit_3/D3S6G -> /Lattice MACHXO2/Digit_4/D4S3G
- Q10 pad 5: Net-(D3-Pad345) -> Net-(D3-Pad417)
- Q10 pad 8: Net-(D3-Pad344) -> Net-(D3-Pad416)
- Q11 pad 2: /Lattice MACHXO2/Digit_3/D3S2R -> /Lattice MACHXO2/Digit_4/D4S4R
- Q11 pad 4: /Lattice MACHXO2/Digit_3/D3S2G -> /Lattice MACHXO2/Digit_4/D4S4G
- Q11 pad 5: Net-(D3-Pad273) -> Net-(D3-Pad435)
- Q11 pad 8: Net-(D3-Pad272) -> Net-(D3-Pad434)
- Q12 pad 2: /Lattice MACHXO2/Digit_3/D3S7R -> /Lattice MACHXO2/Digit_2/D2S1R
- Q12 pad 4: /Lattice MACHXO2/Digit_3/D3S7G -> /Lattice MACHXO2/Digit_2/D2S1G
- Q12 pad 5: Net-(D3-Pad363) -> Net-(D3-Pad129)
- Q12 pad 8: Net-(D3-Pad362) -> Net-(D3-Pad128)
- Q13 pad 2: /Lattice MACHXO2/Digit_3/D3S5R -> /Lattice MACHXO2/Digit_2/D2S6R
- Q13 pad 4: /Lattice MACHXO2/Digit_3/D3S5G -> /Lattice MACHXO2/Digit_2/D2S6G
- Q13 pad 5: Net-(D3-Pad327) -> Net-(D3-Pad219)
- Q13 pad 8: Net-(D3-Pad326) -> Net-(D3-Pad218)
- Q14 pad 2: /Lattice MACHXO2/Digit_3/D3S3R -> /Lattice MACHXO2/Digit_2/D2S2R
- Q14 pad 4: /Lattice MACHXO2/Digit_3/D3S3G -> /Lattice MACHXO2/Digit_2/D2S2G
- Q14 pad 5: Net-(D3-Pad291) -> Net-(D3-Pad147)
- Q14 pad 8: Net-(D3-Pad290) -> Net-(D3-Pad146)
- Q15 pad 2: /Lattice MACHXO2/Digit_3/D3S4R -> /Lattice MACHXO2/Digit_2/D2S7R
- Q15 pad 4: /Lattice MACHXO2/Digit_3/D3S4G -> /Lattice MACHXO2/Digit_2/D2S7G
- Q15 pad 5: Net-(D3-Pad309) -> Net-(D3-Pad237)
- Q15 pad 8: Net-(D3-Pad308) -> Net-(D3-Pad236)
- Q16 pad 2: /Lattice MACHXO2/Digit_4/D4S1R -> /Lattice MACHXO2/Digit_2/D2S5R
- Q16 pad 4: /Lattice MACHXO2/Digit_4/D4S1G -> /Lattice MACHXO2/Digit_2/D2S5G
- Q16 pad 5: Net-(D3-Pad381) -> Net-(D3-Pad201)
- Q16 pad 8: Net-(D3-Pad380) -> Net-(D3-Pad200)
- Q17 pad 2: /Lattice MACHXO2/Digit_4/D4S6R -> /Lattice MACHXO2/Digit_2/D2S3R
- Q17 pad 4: /Lattice MACHXO2/Digit_4/D4S6G -> /Lattice MACHXO2/Digit_2/D2S3G
- Q17 pad 5: Net-(D3-Pad471) -> Net-(D3-Pad165)
- Q17 pad 8: Net-(D3-Pad470) -> Net-(D3-Pad164)
- Q18 pad 2: /Lattice MACHXO2/Digit_4/D4S2R -> /Lattice MACHXO2/Digit_2/D2S4R
- Q18 pad 4: /Lattice MACHXO2/Digit_4/D4S2G -> /Lattice MACHXO2/Digit_2/D2S4G
- Q18 pad 5: Net-(D3-Pad399) -> Net-(D3-Pad183)
- Q18 pad 8: Net-(D3-Pad398) -> Net-(D3-Pad182)
- Q19 pad 2: /Lattice MACHXO2/Digit_4/D4S7R -> /Lattice MACHXO2/Digit_3/D3S1R
- Q19 pad 4: /Lattice MACHXO2/Digit_4/D4S7G -> /Lattice MACHXO2/Digit_3/D3S1G
- Q19 pad 5: Net-(D3-Pad489) -> Net-(D3-Pad255)
- Q19 pad 8: Net-(D3-Pad488) -> Net-(D3-Pad254)
- Q2 pad 1: GND -> Net-(Q2-Pad1)
- Q2 pad 2: /Lattice MACHXO2/Digit_2/D2S1R -> Net-(Q2-Pad2)
- Q2 pad 3: GND -> Net-(Q2-Pad3)
- Q2 pad 4: /Lattice MACHXO2/Digit_2/D2S1G -> Net-(Q2-Pad4)
- Q2 pad 5: Net-(D3-Pad129) -> +5V
- Q2 pad 8: Net-(D3-Pad128) -> +5V
- Q20 pad 2: /Lattice MACHXO2/Digit_4/D4S5R -> /Lattice MACHXO2/Digit_3/D3S6R
- Q20 pad 4: /Lattice MACHXO2/Digit_4/D4S5G -> /Lattice MACHXO2/Digit_3/D3S6G
- Q20 pad 5: Net-(D3-Pad453) -> Net-(D3-Pad345)
- Q20 pad 8: Net-(D3-Pad452) -> Net-(D3-Pad344)
- Q21 pad 2: /Lattice MACHXO2/Digit_4/D4S3R -> /Lattice MACHXO2/Digit_3/D3S2R
- Q21 pad 4: /Lattice MACHXO2/Digit_4/D4S3G -> /Lattice MACHXO2/Digit_3/D3S2G
- Q21 pad 5: Net-(D3-Pad417) -> Net-(D3-Pad273)
- Q21 pad 8: Net-(D3-Pad416) -> Net-(D3-Pad272)
- Q22 pad 2: /Lattice MACHXO2/Digit_4/D4S4R -> /Lattice MACHXO2/Digit_3/D3S7R
- Q22 pad 4: /Lattice MACHXO2/Digit_4/D4S4G -> /Lattice MACHXO2/Digit_3/D3S7G
- Q22 pad 5: Net-(D3-Pad435) -> Net-(D3-Pad363)
- Q22 pad 8: Net-(D3-Pad434) -> Net-(D3-Pad362)
- Q23 pad 2: /Lattice MACHXO2/Digit_1/D1S1R -> /Lattice MACHXO2/Digit_3/D3S5R
- Q23 pad 4: /Lattice MACHXO2/Digit_1/D1S1G -> /Lattice MACHXO2/Digit_3/D3S5G
- Q23 pad 5: Net-(D3-Pad12) -> Net-(D3-Pad327)
- Q23 pad 8: Net-(D3-Pad11) -> Net-(D3-Pad326)
- Q24 pad 2: /Lattice MACHXO2/Digit_1/D1S6R -> /Lattice MACHXO2/Digit_3/D3S3R
- Q24 pad 4: /Lattice MACHXO2/Digit_1/D1S6G -> /Lattice MACHXO2/Digit_3/D3S3G
- Q24 pad 5: Net-(D3-Pad102) -> Net-(D3-Pad291)
- Q24 pad 8: Net-(D3-Pad101) -> Net-(D3-Pad290)
- Q25 pad 2: /Lattice MACHXO2/Digit_1/D1S2R -> /Lattice MACHXO2/Digit_3/D3S4R
- Q25 pad 4: /Lattice MACHXO2/Digit_1/D1S2G -> /Lattice MACHXO2/Digit_3/D3S4G
- Q25 pad 5: Net-(D3-Pad21) -> Net-(D3-Pad309)
- Q25 pad 8: Net-(D3-Pad20) -> Net-(D3-Pad308)
- Q26 pad 2: /Lattice MACHXO2/Digit_1/D1S7R -> /Lattice MACHXO2/Digit_1/D1S1R
- Q26 pad 4: /Lattice MACHXO2/Digit_1/D1S7G -> /Lattice MACHXO2/Digit_1/D1S1G
- Q26 pad 5: Net-(D3-Pad111) -> Net-(D3-Pad12)
- Q26 pad 8: Net-(D3-Pad110) -> Net-(D3-Pad11)
- Q27 pad 2: /Lattice MACHXO2/Digit_1/D1S5R -> /Lattice MACHXO2/Digit_1/D1S6R
- Q27 pad 4: /Lattice MACHXO2/Digit_1/D1S5G -> /Lattice MACHXO2/Digit_1/D1S6G
- Q27 pad 5: Net-(D3-Pad75) -> Net-(D3-Pad102)
- Q27 pad 8: Net-(D3-Pad74) -> Net-(D3-Pad101)
- Q28 pad 2: /Lattice MACHXO2/Digit_1/D1S3R -> /Lattice MACHXO2/Digit_1/D1S2R
- Q28 pad 4: /Lattice MACHXO2/Digit_1/D1S3G -> /Lattice MACHXO2/Digit_1/D1S2G
- Q28 pad 5: Net-(D3-Pad39) -> Net-(D3-Pad21)
- Q28 pad 8: Net-(D3-Pad38) -> Net-(D3-Pad20)
- Q29 pad 2: /Lattice MACHXO2/Digit_1/D1S4R -> /Lattice MACHXO2/Digit_1/D1S7R
- Q29 pad 4: /Lattice MACHXO2/Digit_1/D1S4G -> /Lattice MACHXO2/Digit_1/D1S7G
- Q29 pad 5: Net-(D3-Pad57) -> Net-(D3-Pad111)
- Q29 pad 8: Net-(D3-Pad56) -> Net-(D3-Pad110)
- Q3 pad 1: GND -> Net-(Q3-Pad1)
- Q3 pad 2: /Lattice MACHXO2/Digit_2/D2S6R -> Net-(Q3-Pad2)
- Q3 pad 3: GND -> Net-(Q3-Pad3)
- Q3 pad 4: /Lattice MACHXO2/Digit_2/D2S6G -> Net-(Q3-Pad4)
- Q3 pad 5: Net-(D3-Pad219) -> +5V
- Q3 pad 8: Net-(D3-Pad218) -> +5V
- Q30 pad 1: Net-(Q30-Pad1) -> GND
- Q30 pad 2: /Lattice MACHXO2/Digit_4/A1 -> /Lattice MACHXO2/Digit_1/D1S5R
- Q30 pad 3: Net-(Q30-Pad3) -> GND
- Q30 pad 4: /Lattice MACHXO2/Digit_4/A2 -> /Lattice MACHXO2/Digit_1/D1S5G
- Q30 pad 5: +5V -> Net-(D3-Pad75)
- Q30 pad 8: +5V -> Net-(D3-Pad74)
- Q31 pad 1: Net-(Q31-Pad1) -> GND
- Q31 pad 2: /Lattice MACHXO2/Digit_4/A3 -> /Lattice MACHXO2/Digit_1/D1S3R
- Q31 pad 3: Net-(Q31-Pad3) -> GND
- Q31 pad 4: /Lattice MACHXO2/Digit_4/A4 -> /Lattice MACHXO2/Digit_1/D1S3G
- Q31 pad 5: +5V -> Net-(D3-Pad39)
- Q31 pad 8: +5V -> Net-(D3-Pad38)
- Q32 pad 1: Net-(Q32-Pad1) -> GND
- Q32 pad 2: /Lattice MACHXO2/Digit_4/A5 -> /Lattice MACHXO2/Digit_1/D1S4R
- Q32 pad 3: Net-(Q32-Pad3) -> GND
- Q32 pad 4: /Lattice MACHXO2/Digit_4/A6 -> /Lattice MACHXO2/Digit_1/D1S4G
- Q32 pad 5: +5V -> Net-(D3-Pad57)
- Q32 pad 8: +5V -> Net-(D3-Pad56)
- Q4 pad 1: GND -> Net-(Q4-Pad1)
- Q4 pad 2: /Lattice MACHXO2/Digit_2/D2S2R -> Net-(Q4-Pad2)
- Q4 pad 3: GND -> Net-(Q4-Pad3)
- Q4 pad 4: /Lattice MACHXO2/Digit_2/D2S2G -> Net-(Q4-Pad4)
- Q4 pad 5: Net-(D3-Pad147) -> +5V
- Q4 pad 8: Net-(D3-Pad146) -> +5V
- Q5 pad 2: /Lattice MACHXO2/Digit_2/D2S7R -> /Lattice MACHXO2/Digit_4/D4S1R
- Q5 pad 4: /Lattice MACHXO2/Digit_2/D2S7G -> /Lattice MACHXO2/Digit_4/D4S1G
- Q5 pad 5: Net-(D3-Pad237) -> Net-(D3-Pad381)
- Q5 pad 8: Net-(D3-Pad236) -> Net-(D3-Pad380)
- Q6 pad 2: /Lattice MACHXO2/Digit_2/D2S5R -> /Lattice MACHXO2/Digit_4/D4S6R
- Q6 pad 4: /Lattice MACHXO2/Digit_2/D2S5G -> /Lattice MACHXO2/Digit_4/D4S6G
- Q6 pad 5: Net-(D3-Pad201) -> Net-(D3-Pad471)
- Q6 pad 8: Net-(D3-Pad200) -> Net-(D3-Pad470)
- Q7 pad 2: /Lattice MACHXO2/Digit_2/D2S3R -> /Lattice MACHXO2/Digit_4/D4S2R
- Q7 pad 4: /Lattice MACHXO2/Digit_2/D2S3G -> /Lattice MACHXO2/Digit_4/D4S2G
- Q7 pad 5: Net-(D3-Pad165) -> Net-(D3-Pad399)
- Q7 pad 8: Net-(D3-Pad164) -> Net-(D3-Pad398)
- Q8 pad 2: /Lattice MACHXO2/Digit_2/D2S4R -> /Lattice MACHXO2/Digit_4/D4S7R
- Q8 pad 4: /Lattice MACHXO2/Digit_2/D2S4G -> /Lattice MACHXO2/Digit_4/D4S7G
- Q8 pad 5: Net-(D3-Pad183) -> Net-(D3-Pad489)
- Q8 pad 8: Net-(D3-Pad182) -> Net-(D3-Pad488)
- Q9 pad 2: /Lattice MACHXO2/Digit_3/D3S1R -> /Lattice MACHXO2/Digit_4/D4S5R
- Q9 pad 4: /Lattice MACHXO2/Digit_3/D3S1G -> /Lattice MACHXO2/Digit_4/D4S5G
- Q9 pad 5: Net-(D3-Pad255) -> Net-(D3-Pad453)
- Q9 pad 8: Net-(D3-Pad254) -> Net-(D3-Pad452)
- R10 pad 1: /Lattice MACHXO2/Digit_2/D2S6G -> Net-(Q3-Pad4)
- R11 pad 1: /Lattice MACHXO2/Digit_2/D2S2R -> Net-(Q4-Pad2)
- R12 pad 1: /Lattice MACHXO2/Digit_2/D2S2G -> Net-(Q4-Pad4)
- R13 pad 1: /Lattice MACHXO2/Digit_2/D2S7R -> Net-(Q2-Pad1)
- R13 pad 2: GND -> /Lattice MACHXO2/Digit_1/A1
- R14 pad 1: /Lattice MACHXO2/Digit_2/D2S7G -> Net-(Q2-Pad3)
- R14 pad 2: GND -> /Lattice MACHXO2/Digit_1/A2
- R15 pad 1: /Lattice MACHXO2/Digit_2/D2S5R -> Net-(Q3-Pad1)
- R15 pad 2: GND -> /Lattice MACHXO2/Digit_1/A3
- R16 pad 1: /Lattice MACHXO2/Digit_2/D2S5G -> Net-(Q3-Pad3)
- R16 pad 2: GND -> /Lattice MACHXO2/Digit_1/A4
- R17 pad 1: /Lattice MACHXO2/Digit_2/D2S3R -> Net-(Q4-Pad1)
- R17 pad 2: GND -> /Lattice MACHXO2/Digit_1/A5
- R18 pad 1: /Lattice MACHXO2/Digit_2/D2S3G -> Net-(Q4-Pad3)
- R18 pad 2: GND -> /Lattice MACHXO2/Digit_1/A6
- R19 pad 1: /Lattice MACHXO2/Digit_2/D2S4R -> /Lattice MACHXO2/Digit_4/D4S1R
- R20 pad 1: /Lattice MACHXO2/Digit_2/D2S4G -> /Lattice MACHXO2/Digit_4/D4S1G
- R21 pad 1: /Lattice MACHXO2/Digit_3/D3S1R -> /Lattice MACHXO2/Digit_4/D4S6R
- R22 pad 1: /Lattice MACHXO2/Digit_3/D3S1G -> /Lattice MACHXO2/Digit_4/D4S6G
- R23 pad 1: /Lattice MACHXO2/Digit_3/D3S6R -> /Lattice MACHXO2/Digit_4/D4S2R
- R24 pad 1: /Lattice MACHXO2/Digit_3/D3S6G -> /Lattice MACHXO2/Digit_4/D4S2G
- R25 pad 1: /Lattice MACHXO2/Digit_3/D3S2R -> /Lattice MACHXO2/Digit_4/D4S7R
- R26 pad 1: /Lattice MACHXO2/Digit_3/D3S2G -> /Lattice MACHXO2/Digit_4/D4S7G
- R27 pad 1: /Lattice MACHXO2/Digit_3/D3S7R -> /Lattice MACHXO2/Digit_4/D4S5R
- R28 pad 1: /Lattice MACHXO2/Digit_3/D3S7G -> /Lattice MACHXO2/Digit_4/D4S5G
- R29 pad 1: /Lattice MACHXO2/Digit_3/D3S5R -> /Lattice MACHXO2/Digit_4/D4S3R
- R30 pad 1: /Lattice MACHXO2/Digit_3/D3S5G -> /Lattice MACHXO2/Digit_4/D4S3G
- R31 pad 1: /Lattice MACHXO2/Digit_3/D3S3R -> /Lattice MACHXO2/Digit_4/D4S4R
- R32 pad 1: /Lattice MACHXO2/Digit_3/D3S3G -> /Lattice MACHXO2/Digit_4/D4S4G
- R33 pad 1: /Lattice MACHXO2/Digit_3/D3S4R -> /Lattice MACHXO2/Digit_2/D2S1R
- R34 pad 1: /Lattice MACHXO2/Digit_3/D3S4G -> /Lattice MACHXO2/Digit_2/D2S1G
- R35 pad 1: /Lattice MACHXO2/Digit_4/D4S1R -> /Lattice MACHXO2/Digit_2/D2S6R
- R36 pad 1: /Lattice MACHXO2/Digit_4/D4S1G -> /Lattice MACHXO2/Digit_2/D2S6G
- R37 pad 1: /Lattice MACHXO2/Digit_4/D4S6R -> /Lattice MACHXO2/Digit_2/D2S2R
- R38 pad 1: /Lattice MACHXO2/Digit_4/D4S6G -> /Lattice MACHXO2/Digit_2/D2S2G
- R39 pad 1: /Lattice MACHXO2/Digit_4/D4S2R -> /Lattice MACHXO2/Digit_2/D2S7R
- R40 pad 1: /Lattice MACHXO2/Digit_4/D4S2G -> /Lattice MACHXO2/Digit_2/D2S7G
- R41 pad 1: /Lattice MACHXO2/Digit_4/D4S7R -> /Lattice MACHXO2/Digit_2/D2S5R
- R42 pad 1: /Lattice MACHXO2/Digit_4/D4S7G -> /Lattice MACHXO2/Digit_2/D2S5G
- R43 pad 1: /Lattice MACHXO2/Digit_4/D4S5R -> /Lattice MACHXO2/Digit_2/D2S3R
- R44 pad 1: /Lattice MACHXO2/Digit_4/D4S5G -> /Lattice MACHXO2/Digit_2/D2S3G
- R45 pad 1: /Lattice MACHXO2/Digit_4/D4S3R -> /Lattice MACHXO2/Digit_2/D2S4R
- R46 pad 1: /Lattice MACHXO2/Digit_4/D4S3G -> /Lattice MACHXO2/Digit_2/D2S4G
- R47 pad 1: /Lattice MACHXO2/Digit_4/D4S4R -> /Lattice MACHXO2/Digit_3/D3S1R
- R48 pad 1: /Lattice MACHXO2/Digit_4/D4S4G -> /Lattice MACHXO2/Digit_3/D3S1G
- R49 pad 1: /Lattice MACHXO2/Digit_1/D1S1R -> /Lattice MACHXO2/Digit_3/D3S6R
- R50 pad 1: /Lattice MACHXO2/Digit_1/D1S1G -> /Lattice MACHXO2/Digit_3/D3S6G
- R51 pad 1: /Lattice MACHXO2/Digit_1/D1S6R -> /Lattice MACHXO2/Digit_3/D3S2R
- R52 pad 1: /Lattice MACHXO2/Digit_1/D1S6G -> /Lattice MACHXO2/Digit_3/D3S2G
- R53 pad 1: /Lattice MACHXO2/Digit_1/D1S2R -> /Lattice MACHXO2/Digit_3/D3S7R
- R54 pad 1: /Lattice MACHXO2/Digit_1/D1S2G -> /Lattice MACHXO2/Digit_3/D3S7G
- R55 pad 1: /Lattice MACHXO2/Digit_1/D1S7R -> /Lattice MACHXO2/Digit_3/D3S5R
- R56 pad 1: /Lattice MACHXO2/Digit_1/D1S7G -> /Lattice MACHXO2/Digit_3/D3S5G
- R57 pad 1: /Lattice MACHXO2/Digit_1/D1S5R -> /Lattice MACHXO2/Digit_3/D3S3R
- R58 pad 1: /Lattice MACHXO2/Digit_1/D1S5G -> /Lattice MACHXO2/Digit_3/D3S3G
- R59 pad 1: /Lattice MACHXO2/Digit_1/D1S3R -> /Lattice MACHXO2/Digit_3/D3S4R
- R60 pad 1: /Lattice MACHXO2/Digit_1/D1S3G -> /Lattice MACHXO2/Digit_3/D3S4G
- R61 pad 1: /Lattice MACHXO2/Digit_1/D1S4R -> /Lattice MACHXO2/Digit_1/D1S1R
- R62 pad 1: /Lattice MACHXO2/Digit_1/D1S4G -> /Lattice MACHXO2/Digit_1/D1S1G
- R63 pad 1: /Lattice MACHXO2/Digit_4/A1 -> /Lattice MACHXO2/Digit_1/D1S6R
- R64 pad 1: /Lattice MACHXO2/Digit_4/A2 -> /Lattice MACHXO2/Digit_1/D1S6G
- R65 pad 1: Net-(Q30-Pad1) -> /Lattice MACHXO2/Digit_1/D1S2R
- R65 pad 2: /Lattice MACHXO2/Digit_4/D4A1 -> GND
- R66 pad 1: Net-(Q30-Pad3) -> /Lattice MACHXO2/Digit_1/D1S2G
- R66 pad 2: /Lattice MACHXO2/Digit_4/D4A2 -> GND
- R67 pad 1: /Lattice MACHXO2/Digit_4/A3 -> /Lattice MACHXO2/Digit_1/D1S7R
- R68 pad 1: /Lattice MACHXO2/Digit_4/A4 -> /Lattice MACHXO2/Digit_1/D1S7G
- R69 pad 1: Net-(Q31-Pad1) -> /Lattice MACHXO2/Digit_1/D1S5R
- R69 pad 2: /Lattice MACHXO2/Digit_4/D4A3 -> GND
- R7 pad 1: /Lattice MACHXO2/Digit_2/D2S1R -> Net-(Q2-Pad2)
- R70 pad 1: Net-(Q31-Pad3) -> /Lattice MACHXO2/Digit_1/D1S5G
- R70 pad 2: /Lattice MACHXO2/Digit_4/D4A4 -> GND
- R71 pad 1: /Lattice MACHXO2/Digit_4/A5 -> /Lattice MACHXO2/Digit_1/D1S3R
- R72 pad 1: /Lattice MACHXO2/Digit_4/A6 -> /Lattice MACHXO2/Digit_1/D1S3G
- R73 pad 1: Net-(Q32-Pad1) -> /Lattice MACHXO2/Digit_1/D1S4R
- R73 pad 2: /Lattice MACHXO2/Digit_4/D4A5 -> GND
- R74 pad 1: Net-(Q32-Pad3) -> /Lattice MACHXO2/Digit_1/D1S4G
- R74 pad 2: /Lattice MACHXO2/Digit_4/D4A6 -> GND
- R8 pad 1: /Lattice MACHXO2/Digit_2/D2S1G -> Net-(Q2-Pad4)
- R9 pad 1: /Lattice MACHXO2/Digit_2/D2S6R -> Net-(Q3-Pad2)
Routing:
- net /Lattice MACHXO2/Digit_1/A3: track 0.00 -> 1075.4 mm
- net /Lattice MACHXO2/Digit_1/A2: track 0.00 -> 1041.9 mm
- net /Lattice MACHXO2/Digit_1/A4: track 0.00 -> 985.1 mm
- net /Lattice MACHXO2/Digit_1/A5: track 0.00 -> 925.1 mm
- net /Lattice MACHXO2/Digit_1/A1: track 0.00 -> 810.6 mm
- net /Lattice MACHXO2/Digit_1/A6: track 0.00 -> 696.5 mm
- net /Lattice MACHXO2/Digit_1/D1A4: track 256.3 -> 0.00 mm
- net /Lattice MACHXO2/Digit_1/D1A5: track 256.2 -> 0.00 mm
- net /Lattice MACHXO2/Digit_1/D1A6: track 254.8 -> 0.00 mm
- net /Lattice MACHXO2/Digit_1/D1A3: track 138.1 -> 0.00 mm
- net /Lattice MACHXO2/Digit_1/D1A2: track 113.8 -> 0.00 mm
- net /Lattice MACHXO2/Digit_1/D1A1: track 81.9 -> 0.00 mm
- net Net-(D3-Pad470): track 0.00 -> 23.7 mm
- net Net-(D3-Pad471): track 0.00 -> 23.7 mm
- net Net-(D3-Pad201): track 0.00 -> 23.7 mm
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
Commit message: PCB work.
Routing:
- net /Lattice MACHXO2/Digit_1/A2: track 1041.9 -> 566.6 mm
- net /Lattice MACHXO2/Digit_1/A3: track 1075.4 -> 605.6 mm
- net /Lattice MACHXO2/Digit_1/A1: track 810.6 -> 409.8 mm
- net /Lattice MACHXO2/Digit_1/A4: track 985.1 -> 596.2 mm
- net /Lattice MACHXO2/Digit_1/A5: track 925.1 -> 577.8 mm
- net /Lattice MACHXO2/Digit_1/A6: track 696.5 -> 438.0 mm
- net Net-(D3-Pad146): track 0.00 -> 23.6 mm
- net Net-(D3-Pad164): track 0.00 -> 23.5 mm
- net Net-(D3-Pad147): track 0.00 -> 23.2 mm
- net Net-(D3-Pad165): track 0.00 -> 23.1 mm
Other:
- net class OSHPARK added: clearance 0.1524, trace_width 0.1524, via_dia 0.889, via_drill 0.635

Commit message: PCB work.
Parts:
- added D4: Indicators, Custom:SingleLED, F.Cu at (148.6, 86.4)
- moved C11 192.9 mm to (241.6, 63.6)
- moved C13 192.9 mm to (246.3, 63.6)
- moved C19 192.9 mm to (251.0, 63.6)
- moved C14 192.9 mm to (241.6, 57.7)
- moved C15 192.9 mm to (259.8, 50.2)
- moved C18 192.9 mm to (255.7, 56.1)
- moved C22 192.9 mm to (255.7, 62.0)
- moved C23 192.9 mm to (251.0, 57.7)
- moved C8 192.9 mm to (246.3, 57.7)
- moved C9 192.9 mm to (255.1, 50.2)
- moved R16 131.3 mm to (123.4, 46.9)
- moved R13 126.2 mm to (117.6, 40.9)
- moved R40 126.0 mm to (260.3, 95.7)
- moved R43 126.0 mm to (260.3, 101.6)
- moved R33 126.0 mm to (255.8, 95.7)
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Routing:
- net /Lattice MACHXO2/Digit_1/A4: track 596.2 -> 847.4 mm
- net /Lattice MACHXO2/Digit_1/A5: track 577.8 -> 828.7 mm
- net /Lattice MACHXO2/Digit_1/A6: track 438.0 -> 660.3 mm
- net /Lattice MACHXO2/Digit_1/A3: track 605.6 -> 779.4 mm
- net /Lattice MACHXO2/Digit_1/A2: track 566.6 -> 724.2 mm
- net /Lattice MACHXO2/Digit_1/A1: track 409.8 -> 519.9 mm
- net Net-(D3-Pad327): track 0.00 -> 23.6 mm
- net Net-(D3-Pad326): track 0.00 -> 23.2 mm

Commit message: PCB work.
Routing:
- net /Lattice MACHXO2/Digit_1/A4: track 847.4 -> 1430.7 mm
- net /Lattice MACHXO2/Digit_1/A5: track 828.7 -> 1399.4 mm
- net /Lattice MACHXO2/Digit_1/A3: track 779.4 -> 1293.8 mm
- net /Lattice MACHXO2/Digit_1/A2: track 724.2 -> 1197.2 mm
- net /Lattice MACHXO2/Digit_1/A6: track 660.3 -> 1122.6 mm
- net /Lattice MACHXO2/Digit_1/A1: track 519.9 -> 848.7 mm
- net Net-(D3-Pad453): track 0.00 -> 24.6 mm
- net Net-(D3-Pad290): track 0.00 -> 24.2 mm
- net Net-(D3-Pad272): track 0.00 -> 24.2 mm
- net Net-(D3-Pad345): track 0.00 -> 24.1 mm
- net Net-(D3-Pad273): track 0.00 -> 24.1 mm
- net Net-(D3-Pad291): track 0.00 -> 24.1 mm
- net Net-(D3-Pad344): track 0.00 -> 24.0 mm
- net Net-(D3-Pad452): track 0.00 -> 23.9 mm
- net Net-(D3-Pad110): track 23.7 -> 0.00 mm
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
Commit message: PCB work.
Parts:
- removed REF**: SolderWirePad_single_2-5mmDrill, Wire_Pads:SolderWirePad_single_2mmDrill
- added BT1: BATTERY, Custom:SuperCap_604-1020-1-ND, B.Cu at (172.7, 97.2)
- added F1: FUSE, Fuse_Holders_and_Fuses:Fuse_SMD1206_HandSoldering, F.Cu at (229.4, 128.3)
- added U7: Electric_Imp, Custom:SD_Card, B.Cu at (83.8, 78.1)
- CON1: value USB-MINI-B -> USB_Micro_Vertical; footprint Connect:USB_Mini-B -> Custom:MicroSD_Vertical
- Q10, Q11, Q12, Q13, Q14, Q15, Q16, Q17, Q18, Q19, Q2, Q20, Q21, Q22, Q23, Q24, Q25, Q26, Q27, Q28, Q29, Q3, Q30, Q31, Q32, Q4, Q5, Q6, Q7, Q8, Q9: footprint Power_Integrations:SO-8 -> Custom:SOIC-8_3.9x4.9mm_Pitch1.27mm
- R1, R10, R11, R12, R13, R14, R15, R16, R17, R18, R19, R2, R20, R21, R22, R23, R24, R25, R26, R27, R28, R29, R3, R30, R31, R32, R33, R34, R35, R36, R37, R38, R39, R4, R40, R41, R42, R43, R44, R45, R46, R47, R48, R49, R5, R50, R51, R52, R53, R54, R55, R56, R57, R58, R59, R6, R60, R61, R62, R63, R64, R65, R66, R67, R68, R69, R7, R70, R71, R72, R73, R74, R8, R9: footprint Resistors_SMD:R_0603_HandSoldering -> Resistors_SMD:R_0402
- U1: footprint SMD_Packages:TQFP-44 -> Custom:WSON-8-1EP
- U2: footprint SMD_Packages:SOIC-8-N -> Custom:TQFP-44
- U4: footprint SMD_Packages:SO-16-W -> SMD_Packages:SOIC-8-N
- U5: footprint SMD_Packages:WSON-8-1EP -> SMD_Packages:SO-16-L
- moved U3 114.3 mm to (212.7, 104.8)
- moved U1 58.4 mm to (156.8, 118.7)
- moved R13 55.9 mm to (173.4, 44.5)
- moved R15 55.0 mm to (178.4, 44.5)
- moved R17 53.6 mm to (183.5, 44.5)
- moved U2 46.2 mm to (148.6, 106.7), turned to 180 degrees
- moved Q4 44.3 mm to (152.4, 43.8), turned to 0 degrees
- moved Q3 41.8 mm to (142.2, 43.8), turned to 0 degrees
- moved U4 31.3 mm to (124.5, 93.3)
- moved U5 24.8 mm to (124.5, 103.5), turned to 270 degrees
- moved X1 14.0 mm to (172.1, 69.8)
- moved Q2 12.7 mm to (105.4, 43.8)
- moved U6 2.54 mm to (148.6, 83.8)
- moved R18 1.91 mm to (128.3, 45.7)
- moved R14 1.25 mm to (118.1, 45.7)
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Routing:
- net /Lattice MACHXO2/Digit_1/A3: track 1293.8 -> 1505.5 mm, vias 0 -> 4
- net /Lattice MACHXO2/Digit_1/A2: track 1197.2 -> 1406.9 mm, vias 0 -> 4
- net /Lattice MACHXO2/Digit_1/A1: track 848.7 -> 1056.2 mm, vias 0 -> 4
- net /Lattice MACHXO2/Digit_1/A4: track 1430.7 -> 1590.1 mm, vias 0 -> 4
- net /Lattice MACHXO2/Digit_1/A5: track 1399.4 -> 1552.5 mm, vias 0 -> 4
- net /Lattice MACHXO2/Digit_1/A6: track 1122.6 -> 1269.0 mm, vias 0 -> 4
- net Net-(D3-Pad237): track 0.00 -> 24.3 mm
- net Net-(D3-Pad111): track 0.00 -> 24.3 mm
- net Net-(D3-Pad363): track 0.00 -> 24.3 mm
- net Net-(D3-Pad489): track 0.00 -> 24.2 mm
- net Net-(D3-Pad236): track 0.00 -> 24.1 mm
- net Net-(D3-Pad362): track 0.00 -> 24.0 mm
- net Net-(D3-Pad110): track 0.00 -> 23.9 mm
- net Net-(D3-Pad488): track 0.00 -> 23.9 mm
Other:
- net class OSHPARK: via_dia 0.889 -> 0.6858; via_drill 0.635 -> 0.3302
- rule via_min_drill: 0.508 -> 0.3302
- rule via_min_size: 0.889 -> 0.6858

Commit message: PCB work.
Routing:
- net Net-(D3-Pad56): track 23.1 -> 24.4 mm
