File: PCB/7SegClock.kicad_pcb (KiCad board)
At the start: 2 copper layers, 177.8 x 76.2 mm, 144 parts, among them CON1 USB_Micro_Vertical, Q1 NPN, Q10 DMN2041LSD-13, Q11 DMN2041LSD-13, Q12 DMN2041LSD-13, Q13 DMN2041LSD-13, Q14 DMN2041LSD-13, Q15 DMN2041LSD-13, Q16 DMN2041LSD-13, Q17 DMN2041LSD-13, Q18 DMN2041LSD-13, Q19 DMN2041LSD-13, Q2 DMN2041LSD-13, Q20 DMN2041LSD-13, Q21 DMN2041LSD-13, Q22 DMN2041LSD-13, Q23 DMN2041LSD-13, Q24 DMN2041LSD-13, Q25 DMN2041LSD-13, Q26 DMN2041LSD-13, Q27 DMN2041LSD-13, Q28 DMN2041LSD-13, Q29 DMN2041LSD-13, Q3 DMN2041LSD-13, Q30 DMN2041LSD-13, Q31 DMN2041LSD-13, Q32 DMN2041LSD-13, Q4 DMN2041LSD-13, Q5 DMN2041LSD-13, Q6 DMN2041LSD-13, Q7 DMN2041LSD-13, Q8 DMN2041LSD-13, Q9 DMN2041LSD-13, U1 TPS62172DSGT, U2 P8X32A, U3 FT232RL, U4 24LC256, U5 DS3231, U6 LCMX02-640UHC-4TG144C, U7 Electric_Imp, X1 5mhz CRYSTAL

Commit message: PCB work.
Parts:
- moved R12 138.8 mm to (189.4, 54.5)
- moved R11 132.0 mm to (189.5, 50.9)
- moved R10 116.1 mm to (152.7, 57.1), turned to 270 degrees
- moved R7 114.3 mm to (101.6, 51.6), turned to 90 degrees
- moved R8 106.4 mm to (101.6, 54.2), turned to 90 degrees
- moved R9 103.8 mm to (150.6, 50.3), turned to 180 degrees
- moved R69 91.7 mm to (237.1, 143.1)
- moved R71 91.7 mm to (232.6, 143.1)
- moved R72 91.7 mm to (237.1, 137.2)
- moved R74 91.7 mm to (232.6, 137.2)
- moved R18 68.0 mm to (195.3, 56.9)
- moved R13 63.4 mm to (111.3, 57.1)
- moved R64 55.3 mm to (216.9, 150.2)
- moved R67 55.3 mm to (216.9, 144.3)
- moved R70 55.3 mm to (225.0, 148.5)
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Routing:
- net /Lattice MACHXO2/Digit_1/A2: track 1406.9 -> 1422.7 mm, vias 4 -> 5
- net /Lattice MACHXO2/Digit_1/A4: track 1590.1 -> 1604.5 mm, vias 4 -> 5
- net Net-(Q2-Pad1): track 0.00 -> 10.3 mm
- net Net-(Q3-Pad1): track 0.00 -> 10.2 mm
- net /Lattice MACHXO2/Digit_1/A1: track 1056.2 -> 1066.4 mm, vias 4 -> 5
- net /Lattice MACHXO2/Digit_1/A3: track 1505.5 -> 1514.6 mm, vias 4 -> 5
- net Net-(Q3-Pad3): track 0.00 -> 5.24 mm
- net Net-(Q2-Pad3): track 0.00 -> 5.17 mm
- net Net-(Q2-Pad4): track 0.00 -> 4.31 mm
- net Net-(Q2-Pad2): track 0.00 -> 4.31 mm
- net Net-(Q3-Pad2): track 0.00 -> 3.05 mm
- net Net-(Q3-Pad4): track 0.00 -> 2.39 mm

Commit message: PCB work.
Parts:
- moved C2 169.0 mm to (88.7, 128.4)
- moved C6 169.0 mm to (84.0, 128.4)
- moved R65 166.4 mm to (77.2, 67.9)
- moved R62 164.9 mm to (77.2, 64.3)
- moved R69 164.1 mm to (77.5, 104.8)
- moved C1 162.5 mm to (103.1, 132.6)
- moved C7 162.5 mm to (98.7, 132.6)
- moved C3 162.2 mm to (108.0, 132.7)
- moved R71 161.3 mm to (77.5, 99.1)
- moved R45 160.7 mm to (106.7, 125.1)
- moved R74 160.6 mm to (72.4, 126.4)
- moved C5 157.7 mm to (116.8, 135.9)
- moved R72 157.0 mm to (83.8, 102.9)
- moved R64 157.0 mm to (77.2, 78.5)
- moved R66 156.5 mm to (77.2, 71.4)
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
Commit message: PCB work.
Parts:
- moved R38 6.93 mm to (117.6, 70.9)
- moved R34 6.92 mm to (117.6, 63.8)
- moved R22 6.84 mm to (206.4, 80.0)
- moved R24 6.84 mm to (206.4, 72.4)
- moved R20 6.63 mm to (206.4, 64.8)
- moved R40 6.56 mm to (119.4, 95.0)
- moved R44 6.48 mm to (119.4, 102.2)
- moved R58 6.48 mm to (166.4, 102.9)
- moved R28 6.45 mm to (207.6, 110.4)
- moved R42 6.43 mm to (119.4, 110.9)
- moved R26 6.43 mm to (207.6, 95.0)
- moved R30 6.41 mm to (207.6, 102.5)
- moved R68 6.41 mm to (77.5, 96.1)
- moved R48 6.38 mm to (165.1, 64.1)
- moved R72 6.36 mm to (77.5, 103.3)
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Routing:
- net Net-(D3-Pad101): track 24.1 -> 49.8 mm
- net Net-(D3-Pad102): track 24.0 -> 42.5 mm
- net Net-(D3-Pad12): track 24.0 -> 34.9 mm
- net /Lattice MACHXO2/Digit_1/A4: track 1604.5 -> 1612.6 mm
- net Net-(D3-Pad11): track 24.2 -> 29.7 mm
- net /Lattice MACHXO2/Digit_1/A5: track 1552.5 -> 1556.5 mm
- net /Lattice MACHXO2/Digit_1/A1: track 1066.4 -> 1064.5 mm
- net /Lattice MACHXO2/Digit_1/A2: track 1422.7 -> 1420.9 mm
- net /Lattice MACHXO2/Digit_1/A3: track 1514.6 -> 1512.8 mm
- net /Lattice MACHXO2/Digit_1/A6: track 1269.0 -> 1269.5 mm

Commit message: PCB work.
Parts:
- C1, C10, C11, C12, C13, C14, C15, C16, C17, C18, C19, C2, C20, C21, C22, C23, C3, C4, C5, C6, C7, C8, C9, D1, D2, F1, Q1, R1, R2, R3, R4, R5, R6: moved to B.Cu
- moved C23 94.8 mm to (214.0, 41.9)
- moved C8 94.7 mm to (207.6, 41.9)
- moved C14 94.6 mm to (201.3, 41.9)
- moved C22 94.4 mm to (175.9, 41.9)
- moved C18 90.4 mm to (182.2, 41.9)
- moved C15 87.7 mm to (188.6, 41.9)
- moved C9 86.5 mm to (194.9, 41.9)
- moved R32 42.1 mm to (191.1, 122.0)
- moved R31 38.8 mm to (191.0, 116.7)
- moved CON1 38.8 mm to (232.3, 115.4), turned to 270 degrees
- moved Q11 35.8 mm to (197.2, 118.1)
- moved R73 23.1 mm to (81.3, 108.0), turned to 90 degrees
- moved Q32 23.0 mm to (87.6, 109.2)
- moved Q30 20.7 mm to (67.1, 118.1)
- moved R69 18.8 mm to (61.6, 116.8), turned to 90 degrees
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Routing:
- net GND: track 0.00 -> 50.9 mm
- net Net-(D3-Pad110): track 23.9 -> 49.4 mm
- net Net-(D3-Pad111): track 24.3 -> 42.6 mm
- net /Lattice MACHXO2/Digit_1/A5: track 1556.5 -> 1569.0 mm
- net /Lattice MACHXO2/Digit_1/A4: track 1612.6 -> 1625.0 mm
- net Net-(D3-Pad75): track 24.3 -> 35.5 mm
- net /Lattice MACHXO2/Digit_1/A2: track 1420.9 -> 1431.7 mm
- net /Lattice MACHXO2/Digit_1/A3: track 1512.8 -> 1523.5 mm
- net Net-(D3-Pad56): track 24.4 -> 34.7 mm
- net /Lattice MACHXO2/Digit_1/A6: track 1269.5 -> 1279.1 mm
- net Net-(D3-Pad38): track 24.5 -> 30.7 mm
- net Net-(D3-Pad39): track 24.6 -> 30.4 mm
- net Net-(D3-Pad57): track 24.1 -> 29.0 mm
- net Net-(D3-Pad74): track 25.0 -> 29.8 mm
- net /Lattice MACHXO2/Digit_1/D1S7G: track 0.00 -> 3.73 mm
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
Commit message: PCB work.
Parts:
- moved R45 23.1 mm to (122.6, 108.0)
- moved Q16 22.6 mm to (108.1, 118.1)
- moved Q18 22.4 mm to (128.9, 109.2)
- moved R46 21.1 mm to (122.6, 110.5)
- moved R41 20.1 mm to (101.7, 116.8), turned to 90 degrees
- moved R42 19.6 mm to (101.7, 119.4), turned to 90 degrees
- moved R39 9.92 mm to (122.6, 101.0), turned to 90 degrees
- moved R40 9.08 mm to (122.6, 103.5), turned to 90 degrees
- moved Q15 6.98 mm to (128.9, 102.2)
- moved Q17 6.98 mm to (128.9, 95.2)
- moved R44 6.54 mm to (122.6, 96.5), turned to 90 degrees
- moved R43 5.67 mm to (122.6, 94.0), turned to 90 degrees
- moved R37 3.41 mm to (120.7, 68.6), turned to 90 degrees
- moved R33 3.26 mm to (120.7, 61.6), turned to 90 degrees
- moved R35 3.26 mm to (120.7, 75.6), turned to 90 degrees
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Routing:
- net GND: track 50.9 -> 103.1 mm
- net Net-(D3-Pad218): track 24.6 -> 50.3 mm
- net /Lattice MACHXO2/Digit_1/A4: track 1625.0 -> 1644.8 mm
- net Net-(D3-Pad219): track 24.4 -> 42.7 mm
- net /Lattice MACHXO2/Digit_1/A5: track 1569.0 -> 1584.8 mm
- net Net-(D3-Pad201): track 23.9 -> 35.5 mm
- net Net-(D3-Pad129): track 24.2 -> 35.6 mm
- net Net-(D3-Pad182): track 24.1 -> 34.5 mm
- net /Lattice MACHXO2/Digit_1/A6: track 1279.1 -> 1289.2 mm
- net Net-(D3-Pad128): track 23.5 -> 29.1 mm
- net Net-(D3-Pad200): track 24.0 -> 28.8 mm
- net Net-(D3-Pad183): track 24.2 -> 29.0 mm
- net /Lattice MACHXO2/Digit_2/D2S7G: track 0.00 -> 3.73 mm
- net /Lattice MACHXO2/Digit_2/D2S6R: track 0.00 -> 3.73 mm
- net /Lattice MACHXO2/Digit_2/D2S5G: track 0.00 -> 3.73 mm
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
Commit message: PCB work.
Parts:
- moved R59 32.0 mm to (170.2, 108.0), turned to 90 degrees
- moved R60 27.3 mm to (170.2, 110.5), turned to 90 degrees
- moved R55 24.8 mm to (144.4, 118.1), turned to 90 degrees
- moved R56 24.6 mm to (144.7, 121.9), turned to 90 degrees
- moved R32 23.4 mm to (211.5, 110.5), turned to 90 degrees
- moved Q23 22.7 mm to (156.0, 118.1)
- moved Q9 22.7 mm to (197.2, 118.1)
- moved Q11 22.4 mm to (217.8, 109.2)
- moved Q25 22.4 mm to (176.5, 109.2)
- moved R31 22.2 mm to (211.5, 108.0), turned to 90 degrees
- moved R27 19.2 mm to (191.4, 117.0), turned to 90 degrees
- moved R28 18.6 mm to (191.4, 119.4), turned to 90 degrees
- moved R25 10.1 mm to (211.5, 101.0), turned to 90 degrees
- moved R53 9.67 mm to (170.2, 101.0), turned to 90 degrees
- moved R26 9.32 mm to (211.5, 103.5), turned to 90 degrees
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Routing:
- net GND: track 103.1 -> 192.5 mm
- net /Lattice MACHXO2/Digit_1/A2: track 1429.2 -> 1460.6 mm
- net /Lattice MACHXO2/Digit_1/A3: track 1520.9 -> 1552.4 mm
- net Net-(D3-Pad236): track 23.5 -> 48.2 mm
- net Net-(D3-Pad237): track 24.3 -> 42.5 mm
- net Net-(D3-Pad308): track 24.2 -> 34.4 mm
- net Net-(D3-Pad165): track 24.0 -> 30.1 mm
- net Net-(D3-Pad164): track 24.2 -> 30.1 mm
- net /Lattice MACHXO2/Digit_1/A1: track 1068.4 -> 1074.2 mm
- net Net-(D3-Pad290): track 24.2 -> 29.9 mm
- net Net-(D3-Pad416): track 24.1 -> 29.8 mm
- net Net-(D3-Pad291): track 24.1 -> 29.7 mm
- net Net-(D3-Pad417): track 24.2 -> 29.6 mm
- net Net-(D3-Pad309): track 24.3 -> 28.9 mm
- net /Lattice MACHXO2/Digit_3/D3S7G: track 0.00 -> 3.73 mm
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
Commit message: PCB work.
Routing:
- net Net-(D3-Pad344): track 24.0 -> 49.7 mm
- net Net-(D3-Pad470): track 23.8 -> 49.5 mm
- net Net-(D3-Pad488): track 23.3 -> 47.7 mm
- net Net-(D3-Pad362): track 23.4 -> 47.7 mm
- net Net-(D3-Pad471): track 24.5 -> 43.4 mm
- net Net-(D3-Pad345): track 24.1 -> 42.9 mm
- net Net-(D3-Pad363): track 24.3 -> 42.5 mm
- net Net-(D3-Pad489): track 24.2 -> 42.3 mm
- net /Lattice MACHXO2/Digit_1/A4: track 1644.8 -> 1661.4 mm
- net Net-(D3-Pad255): track 24.0 -> 35.4 mm
- net Net-(D3-Pad381): track 24.1 -> 35.4 mm
- net Net-(D3-Pad434): track 24.2 -> 34.5 mm
- net /Lattice MACHXO2/Digit_1/A5: track 1584.8 -> 1593.4 mm
- net Net-(D3-Pad435): track 23.5 -> 28.8 mm
- net Net-(D3-Pad380): track 24.1 -> 29.1 mm
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
Commit message: PCB work.
Parts:
- moved R11 0.64 mm to (189.1, 51.4), turned to 90 degrees
- moved R12 0.57 mm to (189.1, 54.0), turned to 90 degrees
Routing:
- net /Lattice MACHXO2/Digit_1/A6: track 1291.0 -> 1312.8 mm, vias 4 -> 5
- net /Lattice MACHXO2/Digit_1/A5: track 1593.4 -> 1612.7 mm, vias 4 -> 5
- net /Lattice MACHXO2/Digit_1/A4: track 1661.4 -> 1673.3 mm
- net Net-(Q4-Pad1): track 0.00 -> 10.1 mm
- net Net-(Q4-Pad3): track 0.00 -> 4.91 mm
- net Net-(Q4-Pad4): track 0.00 -> 4.31 mm
- net Net-(Q4-Pad2): track 0.00 -> 4.31 mm
