File: PCB/Digit2.sch (KiCad schematic (older format))
At the start: 37 parts, among them Q2 DMN2041LSD-13, Q3 DMN2041LSD-13, Q33 DMN2041LSD-13, Q34 DMN2041LSD-13, Q35 DMN2041LSD-13, Q4 DMN2041LSD-13, Q5 DMN2041LSD-13, Q6 DMN2041LSD-13, Q7 DMN2041LSD-13, Q8 DMN2041LSD-13

Commit message: PCB work.
Parts:
- removed Q33, Q34, Q35: DMN2041LSD-13, SO-8, symbol DMN2041LSD-13
- removed R75, R76, R79, R80, R83, R84: 10K, Resistors_SMD:R_0603_HandSoldering, symbol R
- removed R77, R78, R81, R82, R85, R86: 150, Resistors_SMD:R_0603_HandSoldering, symbol R
- renumbered Q2 to Q12, Q3 to Q13, Q4 to Q14, Q5 to Q15, Q6 to Q16, Q7 to Q17, Q8 to Q18, R7 to R33, R8 to R34, R9 to R35, R10 to R36, R11 to R37, R12 to R38, R13 to R39, R14 to R40, R15 to R41, R16 to R42, R17 to R43, R18 to R44, R19 to R45, R20 to R46
Connections:
- net labels removed: +5V
- wire segments 293 -> 257

Commit message: PCB work.
Parts:
- Q12, Q13, Q14, Q15, Q16, Q17, Q18: footprint Power_Integrations:SO-8 -> Custom:SOIC-8_3.9x4.9mm_Pitch1.27mm
- R33, R34, R35, R36, R37, R38, R39, R40, R41, R42, R43, R44, R45, R46: footprint Resistors_SMD:R_0603_HandSoldering -> Resistors_SMD:R_0402
Changed lines of the file:
@@
 F 0 "R35" V 1080 2725 40  0000 C CNN
 F 1 "10K" V 1007 2726 40  0000 C CNN
-F 2 "Resistors_SMD:R_0603_HandSoldering" V 930 2725 30  0001 C CNN
+F 2 "Resistors_SMD:R_0402" V 930 2725 30  0001 C CNN
 F 3 "" H 1000 2725 30  0000 C CNN
 	1    1000 2725
@@
 F 0 "R36" V 2080 2725 40  0000 C CNN
 F 1 "10K" V 2007 2726 40  0000 C CNN
-F 2 "Resistors_SMD:R_0603_HandSoldering" V 1930 2725 30  0001 C CNN
+F 2 "Resistors_SMD:R_0402" V 1930 2725 30  0001 C CNN
 F 3 "" H 2000 2725 30  0000 C CNN
 	1    2000 2725
@@
 F 0 "R41" V 1080 5425 40  0000 C CNN
 F 1 "10K" V 1007 5426 40  0000 C CNN
-F 2 "Resistors_SMD:R_0603_HandSoldering" V 930 5425 30  0001 C CNN
+F 2 "Resistors_SMD:R_0402" V 930 5425 30  0001 C CNN
 F 3 "" H 1000 5425 30  0000 C CNN
 	1    1000 5425
@@
 F 0 "R42" V 2080 5425 40  0000 C CNN
 F 1 "10K" V 2007 5426 40  0000 C CNN
-F 2 "Resistors_SMD:R_0603_HandSoldering" V 1930 5425 30  0001 C CNN
+F 2 "Resistors_SMD:R_0402" V 1930 5425 30  0001 C CNN
 F 3 "" H 2000 5425 30  0000 C CNN
 	1    2000 5425
@@
 F 0 "R45" V 1080 7200 40  0000 C CNN
 F 1 "10K" V 1007 7201 40  0000 C CNN
-F 2 "Resistors_SMD:R_0603_HandSoldering" V 930 7200 30  0001 C CNN
+F 2 "Resistors_SMD:R_0402" V 930 7200 30  0001 C CNN
 F 3 "" H 1000 7200 30  0000 C CNN
 	1    1000 7200
@@
 F 0 "R46" V 2080 7200 40  0000 C CNN
 F 1 "10K" V 2007 7201 40  0000 C CNN
-F 2 "Resistors_SMD:R_0603_HandSoldering" V 1930 7200 30  0001 C CNN
+F 2 "Resistors_SMD:R_0402" V 1930 7200 30  0001 C CNN
 F 3 "" H 2000 7200 30  0000 C CNN
 	1    2000 7200
@@
 F 0 "R33" V 7430 1500 40  0000 C CNN
 F 1 "10K" V 7357 1501 40  0000 C CNN
-F 2 "Resistors_SMD:R_0603_HandSoldering" V 7280 1500 30  0001 C CNN
+F 2 "Resistors_SMD:R_0402" V 7280 1500 30  0001 C CNN
 F 3 "" H 7350 1500 30  0000 C CNN
 	1    7350 1500
@@
 F 0 "R34" V 8430 1500 40  0000 C CNN
 F 1 "10K" V 8357 1501 40  0000 C CNN
-F 2 "Resistors_SMD:R_0603_HandSoldering" V 8280 1500 30  0001 C CNN
+F 2 "Resistors_SMD:R_0402" V 8280 1500 30  0001 C CNN
 F 3 "" H 8350 1500 30  0000 C CNN
 	1    8350 1500
@@
 F 0 "R37" V 7430 3000 40  0000 C CNN
 F 1 "10K" V 7357 3001 40  0000 C CNN
-F 2 "Resistors_SMD:R_0603_HandSoldering" V 7280 3000 30  0001 C CNN
+F 2 "Resistors_SMD:R_0402" V 7280 3000 30  0001 C CNN
 F 3 "" H 7350 3000 30  0000 C CNN
 	1    7350 3000
@@
 F 0 "R38" V 8430 3000 40  0000 C CNN
 F 1 "10K" V 8357 3001 40  0000 C CNN
-F 2 "Resistors_SMD:R_0603_HandSoldering" V 8280 3000 30  0001 C CNN
+F 2 "Resistors_SMD:R_0402" V 8280 3000 30  0001 C CNN
 F 3 "" H 8350 3000 30  0000 C CNN
 	1    8350 3000
@@
 F 0 "R43" V 7430 5860 40  0000 C CNN
 F 1 "10K" V 7357 5861 40  0000 C CNN
-F 2 "Resistors_SMD:R_0603_HandSoldering" V 7280 5860 30  0001 C CNN
+F 2 "Resistors_SMD:R_0402" V 7280 5860 30  0001 C CNN
 F 3 "" H 7350 5860 30  0000 C CNN
 	1    7350 5860
@@
 F 0 "R44" V 8430 5860 40  0000 C CNN
 F 1 "10K" V 8357 5861 40  0000 C CNN
-F 2 "Resistors_SMD:R_0603_HandSoldering" V 8280 5860 30  0001 C CNN
+F 2 "Resistors_SMD:R_0402" V 8280 5860 30  0001 C CNN
 F 3 "" H 8350 5860 30  0000 C CNN
 	1    8350 5860
@@
 F 0 "R39" V 7430 4385 40  0000 C CNN
 F 1 "10K" V 7357 4386 40  0000 C CNN
-F 2 "Resistors_SMD:R_0603_HandSoldering" V 7280 4385 30  0001 C CNN
+F 2 "Resistors_SMD:R_0402" V 7280 4385 30  0001 C CNN
 F 3 "" H 7350 4385 30  0000 C CNN
 	1    7350 4385
@@
 F 0 "R40" V 8430 4385 40  0000 C CNN
 F 1 "10K" V 8357 4386 40  0000 C CNN
-F 2 "Resistors_SMD:R_0603_HandSoldering" V 8280 4385 30  0001 C CNN
+F 2 "Resistors_SMD:R_0402" V 8280 4385 30  0001 C CNN
 F 3 "" H 8350 4385 30  0000 C CNN
 	1    8350 4385
@@
 F 0 "Q13" H 1350 2201 40  0000 R CNN
 F 1 "DMN2041LSD-13" H 1350 2500 40  0000 R CNN
-F 2 "Power_Integrations:SO-8" H 1220 2452 29  0001 C CNN
+F 2 "Custom:SOIC-8_3.9x4.9mm_Pitch1.27mm" H 1220 2452 29  0001 C CNN
 F 3 "" H 1350 2350 60  0000 C CNN
 	1    1350 2350
@@
 F 0 "Q13" H 2350 2201 40  0000 R CNN
 F 1 "DMN2041LSD-13" H 2350 2500 40  0000 R CNN
-F 2 "Power_Integrations:SO-8" H 2220 2452 29  0001 C CNN
+F 2 "Custom:SOIC-8_3.9x4.9mm_Pitch1.27mm" H 2220 2452 29  0001 C CNN
 F 3 "" H 2350 2350 60  0000 C CNN
 	2    2350 2350
@@
 F 0 "Q16" H 1350 4901 40  0000 R CNN
 F 1 "DMN2041LSD-13" H 1350 5200 40  0000 R CNN
-F 2 "Power_Integrations:SO-8" H 1220 5152 29  0001 C CNN
+F 2 "Custom:SOIC-8_3.9x4.9mm_Pitch1.27mm" H 1220 5152 29  0001 C CNN
 F 3 "" H 1350 5050 60  0000 C CNN
 	1    1350 5050
@@
 F 0 "Q16" H 2350 4901 40  0000 R CNN
 F 1 "DMN2041LSD-13" H 2350 5200 40  0000 R CNN
-F 2 "Power_Integrations:SO-8" H 2220 5152 29  0001 C CNN
+F 2 "Custom:SOIC-8_3.9x4.9mm_Pitch1.27mm" H 2220 5152 29  0001 C CNN
 F 3 "" H 2350 5050 60  0000 C CNN
 	2    2350 5050
@@
 F 0 "Q18" H 1350 6676 40  0000 R CNN
 F 1 "DMN2041LSD-13" H 1350 6975 40  0000 R CNN
-F 2 "Power_Integrations:SO-8" H 1220 6927 29  0001 C CNN
+F 2 "Custom:SOIC-8_3.9x4.9mm_Pitch1.27mm" H 1220 6927 29  0001 C CNN
 F 3 "" H 1350 6825 60  0000 C CNN
 	1    1350 6825
@@
 F 0 "Q18" H 2350 6676 40  0000 R CNN
 F 1 "DMN2041LSD-13" H 2350 6975 40  0000 R CNN
-F 2 "Power_Integrations:SO-8" H 2220 6927 29  0001 C CNN
+F 2 "Custom:SOIC-8_3.9x4.9mm_Pitch1.27mm" H 2220 6927 29  0001 C CNN
 F 3 "" H 2350 6825 60  0000 C CNN
 	2    2350 6825
@@
 F 0 "Q17" H 7700 5336 40  0000 R CNN
 F 1 "DMN2041LSD-13" H 7700 5635 40  0000 R CNN
-F 2 "Power_Integrations:SO-8" H 7570 5587 29  0001 C CNN
+F 2 "Custom:SOIC-8_3.9x4.9mm_Pitch1.27mm" H 7570 5587 29  0001 C CNN
 F 3 "" H 7700 5485 60  0000 C CNN
 	1    7700 5485
@@
 F 0 "Q17" H 8700 5336 40  0000 R CNN
 F 1 "DMN2041LSD-13" H 8700 5635 40  0000 R CNN
-F 2 "Power_Integrations:SO-8" H 8570 5587 29  0001 C CNN
+F 2 "Custom:SOIC-8_3.9x4.9mm_Pitch1.27mm" H 8570 5587 29  0001 C CNN
 F 3 "" H 8700 5485 60  0000 C CNN
 	2    8700 5485
@@
 F 0 "Q15" H 7700 3861 40  0000 R CNN
 F 1 "DMN2041LSD-13" H 7700 4160 40  0000 R CNN
-F 2 "Power_Integrations:SO-8" H 7570 4112 29  0001 C CNN
+F 2 "Custom:SOIC-8_3.9x4.9mm_Pitch1.27mm" H 7570 4112 29  0001 C CNN
 F 3 "" H 7700 4010 60  0000 C CNN
 	1    7700 4010
@@
 F 0 "Q15" H 8700 3861 40  0000 R CNN
 F 1 "DMN2041LSD-13" H 8700 4160 40  0000 R CNN
-F 2 "Power_Integrations:SO-8" H 8570 4112 29  0001 C CNN
+F 2 "Custom:SOIC-8_3.9x4.9mm_Pitch1.27mm" H 8570 4112 29  0001 C CNN
 F 3 "" H 8700 4010 60  0000 C CNN
 	2    8700 4010
@@
 F 0 "Q14" H 7700 2476 40  0000 R CNN
 F 1 "DMN2041LSD-13" H 7700 2775 40  0000 R CNN
-F 2 "Power_Integrations:SO-8" H 7570 2727 29  0001 C CNN
+F 2 "Custom:SOIC-8_3.9x4.9mm_Pitch1.27mm" H 7570 2727 29  0001 C CNN
 F 3 "" H 7700 2625 60  0000 C CNN
 	1    7700 2625
@@
 F 0 "Q14" H 8700 2476 40  0000 R CNN
 F 1 "DMN2041LSD-13" H 8700 2775 40  0000 R CNN
-F 2 "Power_Integrations:SO-8" H 8570 2727 29  0001 C CNN
+F 2 "Custom:SOIC-8_3.9x4.9mm_Pitch1.27mm" H 8570 2727 29  0001 C CNN
 F 3 "" H 8700 2625 60  0000 C CNN
 	2    8700 2625
@@
 F 0 "Q12" H 7700 976 40  0000 R CNN
 F 1 "DMN2041LSD-13" H 7700 1275 40  0000 R CNN
-F 2 "Power_Integrations:SO-8" H 7570 1227 29  0001 C CNN
+F 2 "Custom:SOIC-8_3.9x4.9mm_Pitch1.27mm" H 7570 1227 29  0001 C CNN
 F 3 "" H 7700 1125 60  0000 C CNN
 	1    7700 1125
@@
 F 0 "Q12" H 8700 976 40  0000 R CNN
 F 1 "DMN2041LSD-13" H 8700 1275 40  0000 R CNN
-F 2 "Power_Integrations:SO-8" H 8570 1227 29  0001 C CNN
+F 2 "Custom:SOIC-8_3.9x4.9mm_Pitch1.27mm" H 8570 1227 29  0001 C CNN
 F 3 "" H 8700 1125 60  0000 C CNN
 	2    8700 1125

Commit message: PCB work.
Parts:
- R33, R34, R35, R36, R37, R38, R39, R40, R41, R42, R43, R44, R45, R46: symbol R -> R-RESCUE-7SegClock
Changed lines of the file:
@@
 EESchema Schematic File Version 2
+LIBS:7SegClock-rescue
 LIBS:power
 LIBS:device
@@
 LIBS:memory
 LIBS:xilinx
-LIBS:special
 LIBS:microcontrollers
 LIBS:dsp
@@
 D2A6
 $Comp
-L R R35
+L R-RESCUE-7SegClock R35
 U 1 1 54E99F27
 P 1000 2725
@@
 $EndComp
 $Comp
-L R R36
+L R-RESCUE-7SegClock R36
 U 1 1 54E99F2E
 P 2000 2725
@@
 $EndComp
 $Comp
-L R R41
+L R-RESCUE-7SegClock R41
 U 1 1 54E99F48
 P 1000 5425
@@
 $EndComp
 $Comp
-L R R42
+L R-RESCUE-7SegClock R42
 U 1 1 54E99F4F
 P 2000 5425
@@
 D2S5G
 $Comp
-L R R45
+L R-RESCUE-7SegClock R45
 U 1 1 54E99F74
 P 1000 7200
@@
 $EndComp
 $Comp
-L R R46
+L R-RESCUE-7SegClock R46
 U 1 1 54E99F7B
 P 2000 7200
@@
 	2450 6625 2450 6500
 $Comp
-L R R33
+L R-RESCUE-7SegClock R33
 U 1 1 54E9A0B9
 P 7350 1500
@@
 $EndComp
 $Comp
-L R R34
+L R-RESCUE-7SegClock R34
 U 1 1 54E9A0C0
 P 8350 1500
@@
 	8800 675  8800 925
 $Comp
-L R R37
+L R-RESCUE-7SegClock R37
 U 1 1 54E9A0F2
 P 7350 3000
@@
 $EndComp
 $Comp
-L R R38
+L R-RESCUE-7SegClock R38
 U 1 1 54E9A0F9
 P 8350 3000
@@
 	8800 2125 8800 2425
 $Comp
-L R R43
+L R-RESCUE-7SegClock R43
 U 1 1 54E9A12C
 P 7350 5860
@@
 $EndComp
 $Comp
-L R R44
+L R-RESCUE-7SegClock R44
 U 1 1 54E9A133
 P 8350 5860
@@
 	7800 750  7800 925
 $Comp
-L R R39
+L R-RESCUE-7SegClock R39
 U 1 1 54E9A167
 P 7350 4385
@@
 $EndComp
 $Comp
-L R R40
+L R-RESCUE-7SegClock R40
 U 1 1 54E9A16E
 P 8350 4385
