File: PCB/Digit3.sch (KiCad schematic (older format))
At the start: 22 parts, among them Q19 DMN2041LSD-13, Q20 DMN2041LSD-13, Q21 DMN2041LSD-13, Q22 DMN2041LSD-13, Q23 DMN2041LSD-13, Q24 DMN2041LSD-13, Q25 DMN2041LSD-13

Commit message: PCB work.
Parts:
- Q19, Q20, Q21, Q22, Q23, Q24, Q25: footprint Power_Integrations:SO-8 -> Custom:SOIC-8_3.9x4.9mm_Pitch1.27mm
- R47, R48, R49, R50, R51, R52, R53, R54, R55, R56, R57, R58, R59, R60: footprint Resistors_SMD:R_0603_HandSoldering -> Resistors_SMD:R_0402
Changed lines of the file:
@@
 F 0 "R49" V 1080 2725 40  0000 C CNN
 F 1 "10K" V 1007 2726 40  0000 C CNN
-F 2 "Resistors_SMD:R_0603_HandSoldering" V 930 2725 30  0001 C CNN
+F 2 "Resistors_SMD:R_0402" V 930 2725 30  0001 C CNN
 F 3 "" H 1000 2725 30  0000 C CNN
 	1    1000 2725
@@
 F 0 "R50" V 2080 2725 40  0000 C CNN
 F 1 "10K" V 2007 2726 40  0000 C CNN
-F 2 "Resistors_SMD:R_0603_HandSoldering" V 1930 2725 30  0001 C CNN
+F 2 "Resistors_SMD:R_0402" V 1930 2725 30  0001 C CNN
 F 3 "" H 2000 2725 30  0000 C CNN
 	1    2000 2725
@@
 F 0 "R55" V 1080 5425 40  0000 C CNN
 F 1 "10K" V 1007 5426 40  0000 C CNN
-F 2 "Resistors_SMD:R_0603_HandSoldering" V 930 5425 30  0001 C CNN
+F 2 "Resistors_SMD:R_0402" V 930 5425 30  0001 C CNN
 F 3 "" H 1000 5425 30  0000 C CNN
 	1    1000 5425
@@
 F 0 "R56" V 2080 5425 40  0000 C CNN
 F 1 "10K" V 2007 5426 40  0000 C CNN
-F 2 "Resistors_SMD:R_0603_HandSoldering" V 1930 5425 30  0001 C CNN
+F 2 "Resistors_SMD:R_0402" V 1930 5425 30  0001 C CNN
 F 3 "" H 2000 5425 30  0000 C CNN
 	1    2000 5425
@@
 F 0 "R59" V 1080 7200 40  0000 C CNN
 F 1 "10K" V 1007 7201 40  0000 C CNN
-F 2 "Resistors_SMD:R_0603_HandSoldering" V 930 7200 30  0001 C CNN
+F 2 "Resistors_SMD:R_0402" V 930 7200 30  0001 C CNN
 F 3 "" H 1000 7200 30  0000 C CNN
 	1    1000 7200
@@
 F 0 "R60" V 2080 7200 40  0000 C CNN
 F 1 "10K" V 2007 7201 40  0000 C CNN
-F 2 "Resistors_SMD:R_0603_HandSoldering" V 1930 7200 30  0001 C CNN
+F 2 "Resistors_SMD:R_0402" V 1930 7200 30  0001 C CNN
 F 3 "" H 2000 7200 30  0000 C CNN
 	1    2000 7200
@@
 F 0 "R47" V 7430 1500 40  0000 C CNN
 F 1 "10K" V 7357 1501 40  0000 C CNN
-F 2 "Resistors_SMD:R_0603_HandSoldering" V 7280 1500 30  0001 C CNN
+F 2 "Resistors_SMD:R_0402" V 7280 1500 30  0001 C CNN
 F 3 "" H 7350 1500 30  0000 C CNN
 	1    7350 1500
@@
 F 0 "R48" V 8430 1500 40  0000 C CNN
 F 1 "10K" V 8357 1501 40  0000 C CNN
-F 2 "Resistors_SMD:R_0603_HandSoldering" V 8280 1500 30  0001 C CNN
+F 2 "Resistors_SMD:R_0402" V 8280 1500 30  0001 C CNN
 F 3 "" H 8350 1500 30  0000 C CNN
 	1    8350 1500
@@
 F 0 "R51" V 7430 3000 40  0000 C CNN
 F 1 "10K" V 7357 3001 40  0000 C CNN
-F 2 "Resistors_SMD:R_0603_HandSoldering" V 7280 3000 30  0001 C CNN
+F 2 "Resistors_SMD:R_0402" V 7280 3000 30  0001 C CNN
 F 3 "" H 7350 3000 30  0000 C CNN
 	1    7350 3000
@@
 F 0 "R52" V 8430 3000 40  0000 C CNN
 F 1 "10K" V 8357 3001 40  0000 C CNN
-F 2 "Resistors_SMD:R_0603_HandSoldering" V 8280 3000 30  0001 C CNN
+F 2 "Resistors_SMD:R_0402" V 8280 3000 30  0001 C CNN
 F 3 "" H 8350 3000 30  0000 C CNN
 	1    8350 3000
@@
 F 0 "R57" V 7430 5860 40  0000 C CNN
 F 1 "10K" V 7357 5861 40  0000 C CNN
-F 2 "Resistors_SMD:R_0603_HandSoldering" V 7280 5860 30  0001 C CNN
+F 2 "Resistors_SMD:R_0402" V 7280 5860 30  0001 C CNN
 F 3 "" H 7350 5860 30  0000 C CNN
 	1    7350 5860
@@
 F 0 "R58" V 8430 5860 40  0000 C CNN
 F 1 "10K" V 8357 5861 40  0000 C CNN
-F 2 "Resistors_SMD:R_0603_HandSoldering" V 8280 5860 30  0001 C CNN
+F 2 "Resistors_SMD:R_0402" V 8280 5860 30  0001 C CNN
 F 3 "" H 8350 5860 30  0000 C CNN
 	1    8350 5860
@@
 F 0 "R53" V 7430 4385 40  0000 C CNN
 F 1 "10K" V 7357 4386 40  0000 C CNN
-F 2 "Resistors_SMD:R_0603_HandSoldering" V 7280 4385 30  0001 C CNN
+F 2 "Resistors_SMD:R_0402" V 7280 4385 30  0001 C CNN
 F 3 "" H 7350 4385 30  0000 C CNN
 	1    7350 4385
@@
 F 0 "R54" V 8430 4385 40  0000 C CNN
 F 1 "10K" V 8357 4386 40  0000 C CNN
-F 2 "Resistors_SMD:R_0603_HandSoldering" V 8280 4385 30  0001 C CNN
+F 2 "Resistors_SMD:R_0402" V 8280 4385 30  0001 C CNN
 F 3 "" H 8350 4385 30  0000 C CNN
 	1    8350 4385
@@
 F 0 "Q20" H 1350 2201 40  0000 R CNN
 F 1 "DMN2041LSD-13" H 1350 2500 40  0000 R CNN
-F 2 "Power_Integrations:SO-8" H 1220 2452 29  0001 C CNN
+F 2 "Custom:SOIC-8_3.9x4.9mm_Pitch1.27mm" H 1220 2452 29  0001 C CNN
 F 3 "" H 1350 2350 60  0000 C CNN
 	1    1350 2350
@@
 F 0 "Q20" H 2350 2201 40  0000 R CNN
 F 1 "DMN2041LSD-13" H 2350 2500 40  0000 R CNN
-F 2 "Power_Integrations:SO-8" H 2220 2452 29  0001 C CNN
+F 2 "Custom:SOIC-8_3.9x4.9mm_Pitch1.27mm" H 2220 2452 29  0001 C CNN
 F 3 "" H 2350 2350 60  0000 C CNN
 	2    2350 2350
@@
 F 0 "Q23" H 1350 4901 40  0000 R CNN
 F 1 "DMN2041LSD-13" H 1350 5200 40  0000 R CNN
-F 2 "Power_Integrations:SO-8" H 1220 5152 29  0001 C CNN
+F 2 "Custom:SOIC-8_3.9x4.9mm_Pitch1.27mm" H 1220 5152 29  0001 C CNN
 F 3 "" H 1350 5050 60  0000 C CNN
 	1    1350 5050
@@
 F 0 "Q23" H 2350 4901 40  0000 R CNN
 F 1 "DMN2041LSD-13" H 2350 5200 40  0000 R CNN
-F 2 "Power_Integrations:SO-8" H 2220 5152 29  0001 C CNN
+F 2 "Custom:SOIC-8_3.9x4.9mm_Pitch1.27mm" H 2220 5152 29  0001 C CNN
 F 3 "" H 2350 5050 60  0000 C CNN
 	2    2350 5050
@@
 F 0 "Q25" H 1350 6676 40  0000 R CNN
 F 1 "DMN2041LSD-13" H 1350 6975 40  0000 R CNN
-F 2 "Power_Integrations:SO-8" H 1220 6927 29  0001 C CNN
+F 2 "Custom:SOIC-8_3.9x4.9mm_Pitch1.27mm" H 1220 6927 29  0001 C CNN
 F 3 "" H 1350 6825 60  0000 C CNN
 	1    1350 6825
@@
 F 0 "Q25" H 2350 6676 40  0000 R CNN
 F 1 "DMN2041LSD-13" H 2350 6975 40  0000 R CNN
-F 2 "Power_Integrations:SO-8" H 2220 6927 29  0001 C CNN
+F 2 "Custom:SOIC-8_3.9x4.9mm_Pitch1.27mm" H 2220 6927 29  0001 C CNN
 F 3 "" H 2350 6825 60  0000 C CNN
 	2    2350 6825
@@
 F 0 "Q24" H 7700 5336 40  0000 R CNN
 F 1 "DMN2041LSD-13" H 7700 5635 40  0000 R CNN
-F 2 "Power_Integrations:SO-8" H 7570 5587 29  0001 C CNN
+F 2 "Custom:SOIC-8_3.9x4.9mm_Pitch1.27mm" H 7570 5587 29  0001 C CNN
 F 3 "" H 7700 5485 60  0000 C CNN
 	1    7700 5485
@@
 F 0 "Q24" H 8700 5336 40  0000 R CNN
 F 1 "DMN2041LSD-13" H 8700 5635 40  0000 R CNN
-F 2 "Power_Integrations:SO-8" H 8570 5587 29  0001 C CNN
+F 2 "Custom:SOIC-8_3.9x4.9mm_Pitch1.27mm" H 8570 5587 29  0001 C CNN
 F 3 "" H 8700 5485 60  0000 C CNN
 	2    8700 5485
@@
 F 0 "Q22" H 7700 3861 40  0000 R CNN
 F 1 "DMN2041LSD-13" H 7700 4160 40  0000 R CNN
-F 2 "Power_Integrations:SO-8" H 7570 4112 29  0001 C CNN
+F 2 "Custom:SOIC-8_3.9x4.9mm_Pitch1.27mm" H 7570 4112 29  0001 C CNN
 F 3 "" H 7700 4010 60  0000 C CNN
 	1    7700 4010
@@
 F 0 "Q22" H 8700 3861 40  0000 R CNN
 F 1 "DMN2041LSD-13" H 8700 4160 40  0000 R CNN
-F 2 "Power_Integrations:SO-8" H 8570 4112 29  0001 C CNN
+F 2 "Custom:SOIC-8_3.9x4.9mm_Pitch1.27mm" H 8570 4112 29  0001 C CNN
 F 3 "" H 8700 4010 60  0000 C CNN
 	2    8700 4010
@@
 F 0 "Q21" H 7700 2476 40  0000 R CNN
 F 1 "DMN2041LSD-13" H 7700 2775 40  0000 R CNN
-F 2 "Power_Integrations:SO-8" H 7570 2727 29  0001 C CNN
+F 2 "Custom:SOIC-8_3.9x4.9mm_Pitch1.27mm" H 7570 2727 29  0001 C CNN
 F 3 "" H 7700 2625 60  0000 C CNN
 	1    7700 2625
@@
 F 0 "Q21" H 8700 2476 40  0000 R CNN
 F 1 "DMN2041LSD-13" H 8700 2775 40  0000 R CNN
-F 2 "Power_Integrations:SO-8" H 8570 2727 29  0001 C CNN
+F 2 "Custom:SOIC-8_3.9x4.9mm_Pitch1.27mm" H 8570 2727 29  0001 C CNN
 F 3 "" H 8700 2625 60  0000 C CNN
 	2    8700 2625
@@
 F 0 "Q19" H 7700 976 40  0000 R CNN
 F 1 "DMN2041LSD-13" H 7700 1275 40  0000 R CNN
-F 2 "Power_Integrations:SO-8" H 7570 1227 29  0001 C CNN
+F 2 "Custom:SOIC-8_3.9x4.9mm_Pitch1.27mm" H 7570 1227 29  0001 C CNN
 F 3 "" H 7700 1125 60  0000 C CNN
 	1    7700 1125
@@
 F 0 "Q19" H 8700 976 40  0000 R CNN
 F 1 "DMN2041LSD-13" H 8700 1275 40  0000 R CNN
-F 2 "Power_Integrations:SO-8" H 8570 1227 29  0001 C CNN
+F 2 "Custom:SOIC-8_3.9x4.9mm_Pitch1.27mm" H 8570 1227 29  0001 C CNN
 F 3 "" H 8700 1125 60  0000 C CNN
 	2    8700 1125

Commit message: PCB work.
Parts:
- R47, R48, R49, R50, R51, R52, R53, R54, R55, R56, R57, R58, R59, R60: symbol R -> R-RESCUE-7SegClock
Changed lines of the file:
@@
 EESchema Schematic File Version 2
+LIBS:7SegClock-rescue
 LIBS:power
 LIBS:device
@@
 LIBS:memory
 LIBS:xilinx
-LIBS:special
 LIBS:microcontrollers
 LIBS:dsp
@@
 D3A6
 $Comp
-L R R49
+L R-RESCUE-7SegClock R49
 U 1 1 54EB2DD9
 P 1000 2725
@@
 $EndComp
 $Comp
-L R R50
+L R-RESCUE-7SegClock R50
 U 1 1 54EB2DE0
 P 2000 2725
@@
 $EndComp
 $Comp
-L R R55
+L R-RESCUE-7SegClock R55
 U 1 1 54EB2DFA
 P 1000 5425
@@
 $EndComp
 $Comp
-L R R56
+L R-RESCUE-7SegClock R56
 U 1 1 54EB2E01
 P 2000 5425
@@
 D3S5G
 $Comp
-L R R59
+L R-RESCUE-7SegClock R59
 U 1 1 54EB2E26
 P 1000 7200
@@
 $EndComp
 $Comp
-L R R60
+L R-RESCUE-7SegClock R60
 U 1 1 54EB2E2D
 P 2000 7200
@@
 	2450 6625 2450 6500
 $Comp
-L R R47
+L R-RESCUE-7SegClock R47
 U 1 1 54EB2F64
 P 7350 1500
@@
 $EndComp
 $Comp
-L R R48
+L R-RESCUE-7SegClock R48
 U 1 1 54EB2F6B
 P 8350 1500
@@
 	8800 675  8800 925
 $Comp
-L R R51
+L R-RESCUE-7SegClock R51
 U 1 1 54EB2F9D
 P 7350 3000
@@
 $EndComp
 $Comp
-L R R52
+L R-RESCUE-7SegClock R52
 U 1 1 54EB2FA4
 P 8350 3000
@@
 	8800 2125 8800 2425
 $Comp
-L R R57
+L R-RESCUE-7SegClock R57
 U 1 1 54EB2FD7
 P 7350 5860
@@
 $EndComp
 $Comp
-L R R58
+L R-RESCUE-7SegClock R58
 U 1 1 54EB2FDE
 P 8350 5860
@@
 	7800 750  7800 925
 $Comp
-L R R53
+L R-RESCUE-7SegClock R53
 U 1 1 54EB3012
 P 7350 4385
@@
 $EndComp
 $Comp
-L R R54
+L R-RESCUE-7SegClock R54
 U 1 1 54EB3019
 P 8350 4385
