File: PCB/Digit4.sch (KiCad schematic (older format))
At the start: 22 parts, among them Q10 DMN2041LSD-13, Q11 DMN2041LSD-13, Q5 DMN2041LSD-13, Q6 DMN2041LSD-13, Q7 DMN2041LSD-13, Q8 DMN2041LSD-13, Q9 DMN2041LSD-13

Commit message: PCB work.
Parts:
- Q10, Q11, Q5, Q6, Q7, Q8, Q9: footprint Power_Integrations:SO-8 -> Custom:SOIC-8_3.9x4.9mm_Pitch1.27mm
- R19, R20, R21, R22, R23, R24, R25, R26, R27, R28, R29, R30, R31, R32: footprint Resistors_SMD:R_0603_HandSoldering -> Resistors_SMD:R_0402
Changed lines of the file:
@@
 F 0 "R21" V 1080 2725 40  0000 C CNN
 F 1 "10K" V 1007 2726 40  0000 C CNN
-F 2 "Resistors_SMD:R_0603_HandSoldering" V 930 2725 30  0001 C CNN
+F 2 "Resistors_SMD:R_0402" V 930 2725 30  0001 C CNN
 F 3 "" H 1000 2725 30  0000 C CNN
 	1    1000 2725
@@
 F 0 "R22" V 2080 2725 40  0000 C CNN
 F 1 "10K" V 2007 2726 40  0000 C CNN
-F 2 "Resistors_SMD:R_0603_HandSoldering" V 1930 2725 30  0001 C CNN
+F 2 "Resistors_SMD:R_0402" V 1930 2725 30  0001 C CNN
 F 3 "" H 2000 2725 30  0000 C CNN
 	1    2000 2725
@@
 F 0 "R27" V 1080 5425 40  0000 C CNN
 F 1 "10K" V 1007 5426 40  0000 C CNN
-F 2 "Resistors_SMD:R_0603_HandSoldering" V 930 5425 30  0001 C CNN
+F 2 "Resistors_SMD:R_0402" V 930 5425 30  0001 C CNN
 F 3 "" H 1000 5425 30  0000 C CNN
 	1    1000 5425
@@
 F 0 "R28" V 2080 5425 40  0000 C CNN
 F 1 "10K" V 2007 5426 40  0000 C CNN
-F 2 "Resistors_SMD:R_0603_HandSoldering" V 1930 5425 30  0001 C CNN
+F 2 "Resistors_SMD:R_0402" V 1930 5425 30  0001 C CNN
 F 3 "" H 2000 5425 30  0000 C CNN
 	1    2000 5425
@@
 F 0 "R31" V 1080 7200 40  0000 C CNN
 F 1 "10K" V 1007 7201 40  0000 C CNN
-F 2 "Resistors_SMD:R_0603_HandSoldering" V 930 7200 30  0001 C CNN
+F 2 "Resistors_SMD:R_0402" V 930 7200 30  0001 C CNN
 F 3 "" H 1000 7200 30  0000 C CNN
 	1    1000 7200
@@
 F 0 "R32" V 2080 7200 40  0000 C CNN
 F 1 "10K" V 2007 7201 40  0000 C CNN
-F 2 "Resistors_SMD:R_0603_HandSoldering" V 1930 7200 30  0001 C CNN
+F 2 "Resistors_SMD:R_0402" V 1930 7200 30  0001 C CNN
 F 3 "" H 2000 7200 30  0000 C CNN
 	1    2000 7200
@@
 F 0 "R19" V 7430 1500 40  0000 C CNN
 F 1 "10K" V 7357 1501 40  0000 C CNN
-F 2 "Resistors_SMD:R_0603_HandSoldering" V 7280 1500 30  0001 C CNN
+F 2 "Resistors_SMD:R_0402" V 7280 1500 30  0001 C CNN
 F 3 "" H 7350 1500 30  0000 C CNN
 	1    7350 1500
@@
 F 0 "R20" V 8430 1500 40  0000 C CNN
 F 1 "10K" V 8357 1501 40  0000 C CNN
-F 2 "Resistors_SMD:R_0603_HandSoldering" V 8280 1500 30  0001 C CNN
+F 2 "Resistors_SMD:R_0402" V 8280 1500 30  0001 C CNN
 F 3 "" H 8350 1500 30  0000 C CNN
 	1    8350 1500
@@
 F 0 "R23" V 7430 3000 40  0000 C CNN
 F 1 "10K" V 7357 3001 40  0000 C CNN
-F 2 "Resistors_SMD:R_0603_HandSoldering" V 7280 3000 30  0001 C CNN
+F 2 "Resistors_SMD:R_0402" V 7280 3000 30  0001 C CNN
 F 3 "" H 7350 3000 30  0000 C CNN
 	1    7350 3000
@@
 F 0 "R24" V 8430 3000 40  0000 C CNN
 F 1 "10K" V 8357 3001 40  0000 C CNN
-F 2 "Resistors_SMD:R_0603_HandSoldering" V 8280 3000 30  0001 C CNN
+F 2 "Resistors_SMD:R_0402" V 8280 3000 30  0001 C CNN
 F 3 "" H 8350 3000 30  0000 C CNN
 	1    8350 3000
@@
 F 0 "R29" V 7430 5860 40  0000 C CNN
 F 1 "10K" V 7357 5861 40  0000 C CNN
-F 2 "Resistors_SMD:R_0603_HandSoldering" V 7280 5860 30  0001 C CNN
+F 2 "Resistors_SMD:R_0402" V 7280 5860 30  0001 C CNN
 F 3 "" H 7350 5860 30  0000 C CNN
 	1    7350 5860
@@
 F 0 "R30" V 8430 5860 40  0000 C CNN
 F 1 "10K" V 8357 5861 40  0000 C CNN
-F 2 "Resistors_SMD:R_0603_HandSoldering" V 8280 5860 30  0001 C CNN
+F 2 "Resistors_SMD:R_0402" V 8280 5860 30  0001 C CNN
 F 3 "" H 8350 5860 30  0000 C CNN
 	1    8350 5860
@@
 F 0 "R25" V 7430 4385 40  0000 C CNN
 F 1 "10K" V 7357 4386 40  0000 C CNN
-F 2 "Resistors_SMD:R_0603_HandSoldering" V 7280 4385 30  0001 C CNN
+F 2 "Resistors_SMD:R_0402" V 7280 4385 30  0001 C CNN
 F 3 "" H 7350 4385 30  0000 C CNN
 	1    7350 4385
@@
 F 0 "R26" V 8430 4385 40  0000 C CNN
 F 1 "10K" V 8357 4386 40  0000 C CNN
-F 2 "Resistors_SMD:R_0603_HandSoldering" V 8280 4385 30  0001 C CNN
+F 2 "Resistors_SMD:R_0402" V 8280 4385 30  0001 C CNN
 F 3 "" H 8350 4385 30  0000 C CNN
 	1    8350 4385
@@
 F 0 "Q6" H 1350 2201 40  0000 R CNN
 F 1 "DMN2041LSD-13" H 1350 2500 40  0000 R CNN
-F 2 "Power_Integrations:SO-8" H 1220 2452 29  0001 C CNN
+F 2 "Custom:SOIC-8_3.9x4.9mm_Pitch1.27mm" H 1220 2452 29  0001 C CNN
 F 3 "" H 1350 2350 60  0000 C CNN
 	1    1350 2350
@@
 F 0 "Q6" H 2350 2201 40  0000 R CNN
 F 1 "DMN2041LSD-13" H 2350 2500 40  0000 R CNN
-F 2 "Power_Integrations:SO-8" H 2220 2452 29  0001 C CNN
+F 2 "Custom:SOIC-8_3.9x4.9mm_Pitch1.27mm" H 2220 2452 29  0001 C CNN
 F 3 "" H 2350 2350 60  0000 C CNN
 	2    2350 2350
@@
 F 0 "Q9" H 1350 4901 40  0000 R CNN
 F 1 "DMN2041LSD-13" H 1350 5200 40  0000 R CNN
-F 2 "Power_Integrations:SO-8" H 1220 5152 29  0001 C CNN
+F 2 "Custom:SOIC-8_3.9x4.9mm_Pitch1.27mm" H 1220 5152 29  0001 C CNN
 F 3 "" H 1350 5050 60  0000 C CNN
 	1    1350 5050
@@
 F 0 "Q9" H 2350 4901 40  0000 R CNN
 F 1 "DMN2041LSD-13" H 2350 5200 40  0000 R CNN
-F 2 "Power_Integrations:SO-8" H 2220 5152 29  0001 C CNN
+F 2 "Custom:SOIC-8_3.9x4.9mm_Pitch1.27mm" H 2220 5152 29  0001 C CNN
 F 3 "" H 2350 5050 60  0000 C CNN
 	2    2350 5050
@@
 F 0 "Q11" H 1350 6676 40  0000 R CNN
 F 1 "DMN2041LSD-13" H 1350 6975 40  0000 R CNN
-F 2 "Power_Integrations:SO-8" H 1220 6927 29  0001 C CNN
+F 2 "Custom:SOIC-8_3.9x4.9mm_Pitch1.27mm" H 1220 6927 29  0001 C CNN
 F 3 "" H 1350 6825 60  0000 C CNN
 	1    1350 6825
@@
 F 0 "Q11" H 2350 6676 40  0000 R CNN
 F 1 "DMN2041LSD-13" H 2350 6975 40  0000 R CNN
-F 2 "Power_Integrations:SO-8" H 2220 6927 29  0001 C CNN
+F 2 "Custom:SOIC-8_3.9x4.9mm_Pitch1.27mm" H 2220 6927 29  0001 C CNN
 F 3 "" H 2350 6825 60  0000 C CNN
 	2    2350 6825
@@
 F 0 "Q10" H 7700 5336 40  0000 R CNN
 F 1 "DMN2041LSD-13" H 7700 5635 40  0000 R CNN
-F 2 "Power_Integrations:SO-8" H 7570 5587 29  0001 C CNN
+F 2 "Custom:SOIC-8_3.9x4.9mm_Pitch1.27mm" H 7570 5587 29  0001 C CNN
 F 3 "" H 7700 5485 60  0000 C CNN
 	1    7700 5485
@@
 F 0 "Q10" H 8700 5336 40  0000 R CNN
 F 1 "DMN2041LSD-13" H 8700 5635 40  0000 R CNN
-F 2 "Power_Integrations:SO-8" H 8570 5587 29  0001 C CNN
+F 2 "Custom:SOIC-8_3.9x4.9mm_Pitch1.27mm" H 8570 5587 29  0001 C CNN
 F 3 "" H 8700 5485 60  0000 C CNN
 	2    8700 5485
@@
 F 0 "Q8" H 7700 3861 40  0000 R CNN
 F 1 "DMN2041LSD-13" H 7700 4160 40  0000 R CNN
-F 2 "Power_Integrations:SO-8" H 7570 4112 29  0001 C CNN
+F 2 "Custom:SOIC-8_3.9x4.9mm_Pitch1.27mm" H 7570 4112 29  0001 C CNN
 F 3 "" H 7700 4010 60  0000 C CNN
 	1    7700 4010
@@
 F 0 "Q8" H 8700 3861 40  0000 R CNN
 F 1 "DMN2041LSD-13" H 8700 4160 40  0000 R CNN
-F 2 "Power_Integrations:SO-8" H 8570 4112 29  0001 C CNN
+F 2 "Custom:SOIC-8_3.9x4.9mm_Pitch1.27mm" H 8570 4112 29  0001 C CNN
 F 3 "" H 8700 4010 60  0000 C CNN
 	2    8700 4010
@@
 F 0 "Q7" H 7700 2476 40  0000 R CNN
 F 1 "DMN2041LSD-13" H 7700 2775 40  0000 R CNN
-F 2 "Power_Integrations:SO-8" H 7570 2727 29  0001 C CNN
+F 2 "Custom:SOIC-8_3.9x4.9mm_Pitch1.27mm" H 7570 2727 29  0001 C CNN
 F 3 "" H 7700 2625 60  0000 C CNN
 	1    7700 2625
@@
 F 0 "Q7" H 8700 2476 40  0000 R CNN
 F 1 "DMN2041LSD-13" H 8700 2775 40  0000 R CNN
-F 2 "Power_Integrations:SO-8" H 8570 2727 29  0001 C CNN
+F 2 "Custom:SOIC-8_3.9x4.9mm_Pitch1.27mm" H 8570 2727 29  0001 C CNN
 F 3 "" H 8700 2625 60  0000 C CNN
 	2    8700 2625
@@
 F 0 "Q5" H 7700 976 40  0000 R CNN
 F 1 "DMN2041LSD-13" H 7700 1275 40  0000 R CNN
-F 2 "Power_Integrations:SO-8" H 7570 1227 29  0001 C CNN
+F 2 "Custom:SOIC-8_3.9x4.9mm_Pitch1.27mm" H 7570 1227 29  0001 C CNN
 F 3 "" H 7700 1125 60  0000 C CNN
 	1    7700 1125
@@
 F 0 "Q5" H 8700 976 40  0000 R CNN
 F 1 "DMN2041LSD-13" H 8700 1275 40  0000 R CNN
-F 2 "Power_Integrations:SO-8" H 8570 1227 29  0001 C CNN
+F 2 "Custom:SOIC-8_3.9x4.9mm_Pitch1.27mm" H 8570 1227 29  0001 C CNN
 F 3 "" H 8700 1125 60  0000 C CNN
 	2    8700 1125

Commit message: PCB work.
Parts:
- R19, R20, R21, R22, R23, R24, R25, R26, R27, R28, R29, R30, R31, R32: symbol R -> R-RESCUE-7SegClock
Changed lines of the file:
@@
 EESchema Schematic File Version 2
+LIBS:7SegClock-rescue
 LIBS:power
 LIBS:device
@@
 LIBS:memory
 LIBS:xilinx
-LIBS:special
 LIBS:microcontrollers
 LIBS:dsp
@@
 D4A6
 $Comp
-L R R21
+L R-RESCUE-7SegClock R21
 U 1 1 54EADD8C
 P 1000 2725
@@
 $EndComp
 $Comp
-L R R22
+L R-RESCUE-7SegClock R22
 U 1 1 54EADD93
 P 2000 2725
@@
 $EndComp
 $Comp
-L R R27
+L R-RESCUE-7SegClock R27
 U 1 1 54EADDAD
 P 1000 5425
@@
 $EndComp
 $Comp
-L R R28
+L R-RESCUE-7SegClock R28
 U 1 1 54EADDB4
 P 2000 5425
@@
 D4S5G
 $Comp
-L R R31
+L R-RESCUE-7SegClock R31
 U 1 1 54EADDD9
 P 1000 7200
@@
 $EndComp
 $Comp
-L R R32
+L R-RESCUE-7SegClock R32
 U 1 1 54EADDE0
 P 2000 7200
@@
 	2450 6625 2450 6500
 $Comp
-L R R19
+L R-RESCUE-7SegClock R19
 U 1 1 54EADF1C
 P 7350 1500
@@
 $EndComp
 $Comp
-L R R20
+L R-RESCUE-7SegClock R20
 U 1 1 54EADF23
 P 8350 1500
@@
 	8800 675  8800 925
 $Comp
-L R R23
+L R-RESCUE-7SegClock R23
 U 1 1 54EADF55
 P 7350 3000
@@
 $EndComp
 $Comp
-L R R24
+L R-RESCUE-7SegClock R24
 U 1 1 54EADF5C
 P 8350 3000
@@
 	8800 2125 8800 2425
 $Comp
-L R R29
+L R-RESCUE-7SegClock R29
 U 1 1 54EADF8F
 P 7350 5860
@@
 $EndComp
 $Comp
-L R R30
+L R-RESCUE-7SegClock R30
 U 1 1 54EADF96
 P 8350 5860
@@
 	7800 750  7800 925
 $Comp
-L R R25
+L R-RESCUE-7SegClock R25
 U 1 1 54EADFCA
 P 7350 4385
@@
 $EndComp
 $Comp
-L R R26
+L R-RESCUE-7SegClock R26
 U 1 1 54EADFD1
 P 8350 4385
@@
 BC 01 60 96 31 E6 05 00 CF E7 7F 1E 6D 7A 11 6D 4B 35 E4 B7 1B 6B 03 D8 50 55 DF E5 BD 5F 0B 59
 F0 3A 1E C0 38 64 CF D4 F2 C8 9E A9 05 CC 43 F6 BE 79 15 99 0A D7 74 00 CF 02 78 CE 18 F3 24 80
-47 91 3D 63 3D 51 4F 11 C2 FF 03 CA 62 49 C8 E1 A2 25 5C 00 00 00 00 49 45 4E 44 AE 42 60 82 00
+47 91 3D 63 3D 51 4F 11 C2 FF 03 CA 62 49 C8 E1 A2 25 5C 00 00 00 00 49 45 4E 44 AE 42 60 82 FF
 EndData
 $EndBitmap
