File: PCB_1.1/Digit1.sch (KiCad schematic (older format))
At the start: 37 parts, among them Q23 DMN2041LSD-13, Q24 DMN2041LSD-13, Q25 DMN2041LSD-13, Q26 DMN2041LSD-13, Q27 DMN2041LSD-13, Q28 DMN2041LSD-13, Q29 DMN2041LSD-13, Q39 DMN2041LSD-13, Q40 DMN2041LSD-13, Q41 DMN2041LSD-13

Commit message: PCB work.
Parts:
- removed Q23, Q24, Q25, Q26, Q27, Q28, Q29: DMN2041LSD-13, Power_Integrations:SO-8, symbol DMN2041LSD-13
- removed Q39, Q40, Q41: DMN2041LSD-13, SO-8, symbol DMN2041LSD-13
- removed R100, R103, R104, R107, R108, R49, R50, R51, R52, R53, R54, R55, R56, R57, R58, R59, R60, R61, R62, R99: 10K, Resistors_SMD:R_0603_HandSoldering, symbol R
- removed R101, R102, R105, R106, R109, R110: 150, Resistors_SMD:R_0603_HandSoldering, symbol R
Connections:
- net labels removed: +5V, A1, A2, A3, A4, A5, A6, D1S1G, D1S1R, D1S2G, D1S2R, D1S3G, D1S3R, D1S4G, D1S4R, D1S5G, D1S5R, D1S6G, D1S6R, D1S7G, D1S7R, GND
- wire segments 293 -> 157

Commit message: PCB work.
Connections:
- net labels added: D1S1G, D1S1R, D1S2G, D1S2R, D1S3G, D1S3R, D1S4G, D1S4R, D1S5G, D1S5R, D1S6G, D1S6R, D1S7G, D1S7R
- wire segments 157 -> 158
Changed lines of the file:
@@
 	5130 6500 5130 6600
-Wire Wire Line
-	2450 6500 5130 6500
 Wire Wire Line
 	4830 6600 4830 6500
@@
 	5280 6450 5280 6600
 Wire Wire Line
-	1450 6450 5280 6450
-Wire Wire Line
 	4980 6600 4980 6450
 Connection ~ 4980 6450
@@
 	5380 4825 5380 6450
 Wire Wire Line
-	5380 6450 6550 6450
-Wire Wire Line
 	5480 4675 5330 4675
 Wire Wire Line
-	5330 4675 5330 6525
-Wire Wire Line
-	5330 6525 6625 6525
+	5330 4675 5330 6600
 Wire Wire Line
 	5480 6325 5380 6325
@@
 	3530 4550 3530 6175
 Wire Wire Line
-	2450 4550 3530 4550
-Wire Wire Line
 	3580 6325 3430 6325
 Wire Wire Line
-	3580 4475 3580 6325
-Wire Wire Line
-	1450 4475 3580 4475
+	3580 4400 3580 6325
 Wire Wire Line
 	3430 6025 3580 6025
@@
 	3630 4400 3630 4550
 Wire Wire Line
-	3630 4550 5505 4550
-Wire Wire Line
-	5505 4550 5505 4200
-Wire Wire Line
 	3780 4400 3780 4500
-Wire Wire Line
-	3780 4500 5430 4500
-Wire Wire Line
-	5430 4500 5430 4125
 Wire Wire Line
 	3930 4400 3930 4550
@@
 Connection ~ 5280 4500
 Wire Wire Line
-	5480 1975 5330 1975
-Wire Wire Line
-	5330 1975 5330 3825
-Wire Wire Line
-	5330 3825 6525 3825
-Wire Wire Line
 	5480 2125 5380 2125
 Wire Wire Line
 	5380 2125 5380 3750
-Wire Wire Line
-	5380 3750 6450 3750
-Wire Wire Line
-	5480 2275 5330 2275
-Wire Wire Line
-	5330 2275 5330 2270
-Connection ~ 5330 2270
 Wire Wire Line
 	5480 2425 5380 2425
@@
 	3530 1850 3530 3475
 Wire Wire Line
-	2450 1850 3530 1850
-Wire Wire Line
 	3580 3625 3430 3625
 Wire Wire Line
-	3580 1775 3580 3625
+	3580 1700 3580 3625
 Wire Wire Line
 	3430 3325 3580 3325
@@
 	3630 1700 3630 1850
 Wire Wire Line
-	3630 1850 5480 1850
+	3630 1850 5555 1850
 Wire Wire Line
 	3780 1700 3780 1800
 Wire Wire Line
 	3780 1800 5405 1800
-Wire Wire Line
-	5405 1800 5405 675
 Wire Wire Line
 	3930 1700 3930 1850
@@
 	5280 1700 5280 1800
 Connection ~ 5280 1800
-Wire Wire Line
-	5480 1850 5480 750
 Wire Wire Line
 	4230 4400 4230 4550
@@
 EndData
 $EndBitmap
-Wire Wire Line
-	2450 2150 2450 1850
+Text HLabel 6230 4750 2    50   Input ~ 0
+D1A1
+Text HLabel 6230 5050 2    50   Input ~ 0
+D1A2
+Text HLabel 6230 5350 2    50   Input ~ 0
+D1A3
+Text HLabel 6230 5650 2    50   Input ~ 0
+D1A4
+Text HLabel 6230 5950 2    50   Input ~ 0
+D1A5
+Text HLabel 6230 6250 2    50   Input ~ 0
+D1A6
+Wire Wire Line
+	5330 1975 5330 3900
+Wire Wire Line
+	5480 2275 5330 2275
+Connection ~ 5330 2275
+Wire Wire Line
+	5480 1975 5330 1975
+Wire Wire Line
+	5130 6500 3505 6500
+Wire Wire Line
+	5280 6450 3355 6450
+Wire Wire Line
+	3780 4500 5405 4500
+Wire Wire Line
+	3630 4550 5555 4550
+Wire Wire Line
+	3505 6500 3505 7450
+Wire Wire Line
+	3355 6450 3355 7450
+Wire Wire Line
+	5380 6450 6330 6450
+Wire Wire Line
+	5330 6600 6330 6600
+Wire Wire Line
+	5380 3750 6330 3750
+Wire Wire Line
+	5330 3900 6330 3900
+Wire Wire Line
+	3580 1700 2580 1700
+Wire Wire Line
+	3530 1850 2580 1850
+Wire Wire Line
+	3580 4400 2580 4400
+Wire Wire Line
+	3530 4550 2580 4550
+Wire Wire Line
+	5555 1850 5555 850
+Wire Wire Line
+	5405 1800 5405 850
+Text HLabel 5405 850  1    50   Input ~ 0
+D1S1G
+Text HLabel 5555 850  1    50   Input ~ 0
+D1S1R
+Text HLabel 6330 3750 2    50   Input ~ 0
+D1S2G
+Text HLabel 6330 3900 2    50   Input ~ 0
+D1S2R
+Text HLabel 6330 6450 2    50   Input ~ 0
+D1S3G
+Text HLabel 6330 6600 2    50   Input ~ 0
+D1S3R
+Text HLabel 3505 7450 3    50   Input ~ 0
+D1S4G
+Text HLabel 3355 7450 3    50   Input ~ 0
+D1S4R
+Wire Wire Line
+	5555 4550 5555 4300
+Wire Wire Line
+	5405 4500 5405 4300
+Text HLabel 5405 4300 1    50   Input ~ 0
+D1S7G
+Text HLabel 5555 4300 1    50   Input ~ 0
+D1S7R
+Text HLabel 2580 4550 0    50   Input ~ 0
+D1S5G
+Text HLabel 2580 4400 0    50   Input ~ 0
+D1S5R
+Text HLabel 2580 1700 0    50   Input ~ 0
+D1S6R
+Text HLabel 2580 1850 0    50   Input ~ 0
+D1S6G
 $EndSCHEMATC
