File: PCB_1.1/DigitDrivers.sch (KiCad schematic (older format))
At the start: 18 parts, among them P1 CONN_01X05, U6 LCMX02-640UHC-4TG144C

Commit message: PCB work.
Parts:
- removed C10, C11, C12, C13, C14, C15, C16, C17, C18, C19, C20, C21, C22, C23, C8, C9: 0.1uF, Capacitors_SMD:C_0603_HandSoldering, symbol C
- removed P1: CONN_01X05, symbol CONN_01X05
- removed U6: LCMX02-640UHC-4TG144C, Housings_QFP:TQFP-144_20x20mm_Pitch0.5mm, symbol LCMX02-640UHC-4TG144C
- added Q? (x20): DMN2041LSD-13, SO-8, symbol DMN2041LSD-13
- added R? (x20): 10K, Resistors_SMD:R_0603_HandSoldering, symbol R
- added R? (x6): 150, Resistors_SMD:R_0603_HandSoldering, symbol R
Connections:
- net labels added: +5V, A1, A2, A3, A4, A5, A6, D1A1, D1A2, D1A3, D1A4, D1A5, D1A6, S1G, S1R, S2G, S2R, S3G, S3R, S4G, S4R, S5G, S5R, S6G, S6R, S7G, S7R
- net labels removed: +3V3, CLK, CS_Clock, CS_Encoder, CS_PWM, DataIN, DataOUT, SCL, SDA, TCK, TDI, TDO, TMS, VCC, VCCIO0, VCCIO1, VCCIO2, VCCIO3
- wire segments 90 -> 120

Commit message: PCB work.
Parts:
- gave numbers to parts that had none: 36
Connections:
- net labels added: AN1, AN2, AN3, AN4, AN5, AN6, SEG1G, SEG1R, SEG2G, SEG2R, SEG3G, SEG3R, SEG4G, SEG4R, SEG5G, SEG5R, SEG6G, SEG6R, SEG7G, SEG7R
- net labels removed: D1A1, D1A2, D1A3, D1A4, D1A5, D1A6
- wire segments 120 -> 200
