File: PCB_1.1/7SegClock.kicad_pcb (KiCad board)
At the start: 2 copper layers, 177.8 x 76.2 mm, 185 parts, among them CON1 USB-MINI-B, Q1 NPN, Q10 DMN2041LSD-13, Q11 DMN2041LSD-13, Q12 DMN2041LSD-13, Q13 DMN2041LSD-13, Q14 DMN2041LSD-13, Q15 DMN2041LSD-13, Q16 DMN2041LSD-13, Q17 DMN2041LSD-13, Q18 DMN2041LSD-13, Q19 DMN2041LSD-13, Q2 DMN2041LSD-13, Q20 DMN2041LSD-13, Q21 DMN2041LSD-13, Q22 DMN2041LSD-13, Q23 DMN2041LSD-13, Q24 DMN2041LSD-13, Q25 DMN2041LSD-13, Q26 DMN2041LSD-13, Q27 DMN2041LSD-13, Q28 DMN2041LSD-13, Q29 DMN2041LSD-13, Q3 DMN2041LSD-13, Q30 DMN2041LSD-13, Q31 DMN2041LSD-13, Q32 DMN2041LSD-13, Q33 DMN2041LSD-13, Q34 DMN2041LSD-13, Q35 DMN2041LSD-13, Q36 DMN2041LSD-13, Q37 DMN2041LSD-13, Q38 DMN2041LSD-13, Q39 DMN2041LSD-13, Q4 DMN2041LSD-13, Q40 DMN2041LSD-13, Q41 DMN2041LSD-13, Q5 DMN2041LSD-13, Q6 DMN2041LSD-13, Q7 DMN2041LSD-13, Q8 DMN2041LSD-13, Q9 DMN2041LSD-13, U1 TPS62172DSGT, U2 P8X32A, U3 FT232RL, U4 24LC256, U5 DS3231, U6 LCMX02-640UHC-4TG144C, X1 5mhz CRYSTAL

Commit message: PCB work.
Parts:
- removed Q12, Q13, Q14, Q15, Q16, Q17, Q18, Q19, Q20, Q21, Q22, Q23, Q24, Q25, Q26, Q27, Q28, Q29, Q30, Q31, Q32, Q33, Q34, Q35, Q36, Q37, Q38, Q39, Q40, Q41: DMN2041LSD-13, SO-8
- removed R100, R103, R104, R107, R108, R33, R34, R35, R36, R37, R38, R39, R40, R41, R42, R43, R44, R45, R46, R47, R48, R49, R50, R51, R52, R53, R54, R55, R56, R57, R58, R59, R60, R61, R62, R63, R64, R67, R68, R71, R72, R75, R76, R79, R80, R83, R84, R87, R88, R91, R92, R95, R96, R99: 10K, Resistors_SMD:R_0603_HandSoldering
- removed R101, R102, R105, R106, R109, R110, R65, R66, R69, R70, R73, R74, R77, R78, R81, R82, R85, R86, R89, R90, R93, R94, R97, R98: 150, Resistors_SMD:R_0603_HandSoldering
- Q10, Q11, Q2, Q3, Q4, Q5, Q6, Q7, Q8, Q9: footprint SO-8 -> Power_Integrations:SO-8
- R13, R14, R21, R22, R29, R30: value 10K -> 150
- U5: moved to B.Cu
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Connections:
- net /Lattice MACHXO2/Digit_2/D2S2G renamed /Lattice MACHXO2/Digit Drivers/A2
- net /Lattice MACHXO2/Digit_2/D2S2R renamed /Lattice MACHXO2/Digit Drivers/A1
- D3 pad 1: /Lattice MACHXO2/Digit_1/D1A1 -> /Lattice MACHXO2/Digit Drivers/Digit 1/D1A1
- D3 pad 10: /Lattice MACHXO2/Digit_1/D1A4 -> /Lattice MACHXO2/Digit Drivers/Digit 1/D1A4
- D3 pad 100: /Lattice MACHXO2/Digit_1/D1A4 -> /Lattice MACHXO2/Digit Drivers/Digit 1/D1A4
- D3 pad 101: Net-(D3-Pad101) -> /Lattice MACHXO2/Digit Drivers/S6R
- D3 pad 102: Net-(D3-Pad102) -> /Lattice MACHXO2/Digit Drivers/S6G
- D3 pad 103: /Lattice MACHXO2/Digit_1/D1A5 -> /Lattice MACHXO2/Digit Drivers/Digit 1/D1A5
- D3 pad 104: Net-(D3-Pad101) -> /Lattice MACHXO2/Digit Drivers/S6R
- D3 pad 105: Net-(D3-Pad102) -> /Lattice MACHXO2/Digit Drivers/S6G
- D3 pad 106: /Lattice MACHXO2/Digit_1/D1A6 -> /Lattice MACHXO2/Digit Drivers/Digit 1/D1A6
- D3 pad 107: Net-(D3-Pad101) -> /Lattice MACHXO2/Digit Drivers/S6R
- D3 pad 108: Net-(D3-Pad102) -> /Lattice MACHXO2/Digit Drivers/S6G
- D3 pad 109: /Lattice MACHXO2/Digit_1/D1A1 -> /Lattice MACHXO2/Digit Drivers/Digit 1/D1A1
- D3 pad 11: Net-(D3-Pad11) -> /Lattice MACHXO2/Digit Drivers/S1R
- D3 pad 110: Net-(D3-Pad110) -> /Lattice MACHXO2/Digit Drivers/S7R
- D3 pad 111: Net-(D3-Pad111) -> /Lattice MACHXO2/Digit Drivers/S7G
- D3 pad 112: /Lattice MACHXO2/Digit_1/D1A2 -> /Lattice MACHXO2/Digit Drivers/Digit 1/D1A2
- D3 pad 113: Net-(D3-Pad110) -> /Lattice MACHXO2/Digit Drivers/S7R
- D3 pad 114: Net-(D3-Pad111) -> /Lattice MACHXO2/Digit Drivers/S7G
- D3 pad 115: /Lattice MACHXO2/Digit_1/D1A3 -> /Lattice MACHXO2/Digit Drivers/Digit 1/D1A3
- D3 pad 116: Net-(D3-Pad110) -> /Lattice MACHXO2/Digit Drivers/S7R
- D3 pad 117: Net-(D3-Pad111) -> /Lattice MACHXO2/Digit Drivers/S7G
- D3 pad 118: /Lattice MACHXO2/Digit_1/D1A4 -> /Lattice MACHXO2/Digit Drivers/Digit 1/D1A4
- D3 pad 119: Net-(D3-Pad110) -> /Lattice MACHXO2/Digit Drivers/S7R
- D3 pad 12: Net-(D3-Pad12) -> /Lattice MACHXO2/Digit Drivers/S1G
- D3 pad 120: Net-(D3-Pad111) -> /Lattice MACHXO2/Digit Drivers/S7G
- D3 pad 121: /Lattice MACHXO2/Digit_1/D1A5 -> /Lattice MACHXO2/Digit Drivers/Digit 1/D1A5
- D3 pad 122: Net-(D3-Pad110) -> /Lattice MACHXO2/Digit Drivers/S7R
- D3 pad 123: Net-(D3-Pad111) -> /Lattice MACHXO2/Digit Drivers/S7G
- D3 pad 124: /Lattice MACHXO2/Digit_1/D1A6 -> /Lattice MACHXO2/Digit Drivers/Digit 1/D1A6
- D3 pad 125: Net-(D3-Pad110) -> /Lattice MACHXO2/Digit Drivers/S7R
- D3 pad 126: Net-(D3-Pad111) -> /Lattice MACHXO2/Digit Drivers/S7G
- D3 pad 127: /Lattice MACHXO2/Digit_2/D2A1 -> /Lattice MACHXO2/Digit Drivers/Digit 1/D1A1
- D3 pad 128: Net-(D3-Pad128) -> /Lattice MACHXO2/Digit Drivers/S1R
- D3 pad 129: Net-(D3-Pad129) -> /Lattice MACHXO2/Digit Drivers/S1G
- D3 pad 13: /Lattice MACHXO2/Digit_1/D1A5 -> /Lattice MACHXO2/Digit Drivers/Digit 1/D1A5
- D3 pad 130: /Lattice MACHXO2/Digit_2/D2A2 -> /Lattice MACHXO2/Digit Drivers/Digit 1/D1A2
- D3 pad 131: Net-(D3-Pad128) -> /Lattice MACHXO2/Digit Drivers/S1R
- D3 pad 132: Net-(D3-Pad129) -> /Lattice MACHXO2/Digit Drivers/S1G
- D3 pad 133: /Lattice MACHXO2/Digit_2/D2A3 -> /Lattice MACHXO2/Digit Drivers/Digit 1/D1A3
- D3 pad 134: Net-(D3-Pad128) -> /Lattice MACHXO2/Digit Drivers/S1R
- D3 pad 135: Net-(D3-Pad129) -> /Lattice MACHXO2/Digit Drivers/S1G
- D3 pad 136: /Lattice MACHXO2/Digit_2/D2A4 -> /Lattice MACHXO2/Digit Drivers/Digit 1/D1A4
- D3 pad 137: Net-(D3-Pad128) -> /Lattice MACHXO2/Digit Drivers/S1R
- D3 pad 138: Net-(D3-Pad129) -> /Lattice MACHXO2/Digit Drivers/S1G
- D3 pad 139: /Lattice MACHXO2/Digit_2/D2A5 -> /Lattice MACHXO2/Digit Drivers/Digit 1/D1A5
- D3 pad 14: Net-(D3-Pad11) -> /Lattice MACHXO2/Digit Drivers/S1R
- D3 pad 140: Net-(D3-Pad128) -> /Lattice MACHXO2/Digit Drivers/S1R
- D3 pad 141: Net-(D3-Pad129) -> /Lattice MACHXO2/Digit Drivers/S1G
- D3 pad 142: /Lattice MACHXO2/Digit_2/D2A6 -> /Lattice MACHXO2/Digit Drivers/Digit 1/D1A6
- D3 pad 143: Net-(D3-Pad128) -> /Lattice MACHXO2/Digit Drivers/S1R
- D3 pad 144: Net-(D3-Pad129) -> /Lattice MACHXO2/Digit Drivers/S1G
- D3 pad 145: /Lattice MACHXO2/Digit_2/D2A1 -> /Lattice MACHXO2/Digit Drivers/Digit 1/D1A1
- D3 pad 146: Net-(D3-Pad146) -> /Lattice MACHXO2/Digit Drivers/S2R
- D3 pad 147: Net-(D3-Pad147) -> /Lattice MACHXO2/Digit Drivers/S2G
- D3 pad 148: /Lattice MACHXO2/Digit_2/D2A2 -> /Lattice MACHXO2/Digit Drivers/Digit 1/D1A2
- D3 pad 149: Net-(D3-Pad146) -> /Lattice MACHXO2/Digit Drivers/S2R
- D3 pad 15: Net-(D3-Pad12) -> /Lattice MACHXO2/Digit Drivers/S1G
- D3 pad 150: Net-(D3-Pad147) -> /Lattice MACHXO2/Digit Drivers/S2G
- D3 pad 151: /Lattice MACHXO2/Digit_2/D2A3 -> /Lattice MACHXO2/Digit Drivers/Digit 1/D1A3
- D3 pad 152: Net-(D3-Pad146) -> /Lattice MACHXO2/Digit Drivers/S2R
- D3 pad 153: Net-(D3-Pad147) -> /Lattice MACHXO2/Digit Drivers/S2G
- D3 pad 154: /Lattice MACHXO2/Digit_2/D2A4 -> /Lattice MACHXO2/Digit Drivers/Digit 1/D1A4
- D3 pad 155: Net-(D3-Pad146) -> /Lattice MACHXO2/Digit Drivers/S2R
- D3 pad 156: Net-(D3-Pad147) -> /Lattice MACHXO2/Digit Drivers/S2G
- D3 pad 157: /Lattice MACHXO2/Digit_2/D2A5 -> /Lattice MACHXO2/Digit Drivers/Digit 1/D1A5
- D3 pad 158: Net-(D3-Pad146) -> /Lattice MACHXO2/Digit Drivers/S2R
- D3 pad 159: Net-(D3-Pad147) -> /Lattice MACHXO2/Digit Drivers/S2G
- D3 pad 16: /Lattice MACHXO2/Digit_1/D1A6 -> /Lattice MACHXO2/Digit Drivers/Digit 1/D1A6
- D3 pad 160: /Lattice MACHXO2/Digit_2/D2A6 -> /Lattice MACHXO2/Digit Drivers/Digit 1/D1A6
- D3 pad 161: Net-(D3-Pad146) -> /Lattice MACHXO2/Digit Drivers/S2R
- D3 pad 162: Net-(D3-Pad147) -> /Lattice MACHXO2/Digit Drivers/S2G
- D3 pad 163: /Lattice MACHXO2/Digit_2/D2A1 -> /Lattice MACHXO2/Digit Drivers/Digit 1/D1A1
- D3 pad 164: Net-(D3-Pad164) -> /Lattice MACHXO2/Digit Drivers/S3R
- D3 pad 165: Net-(D3-Pad165) -> /Lattice MACHXO2/Digit Drivers/S3G
- D3 pad 166: /Lattice MACHXO2/Digit_2/D2A2 -> /Lattice MACHXO2/Digit Drivers/Digit 1/D1A2
- D3 pad 167: Net-(D3-Pad164) -> /Lattice MACHXO2/Digit Drivers/S3R
- D3 pad 168: Net-(D3-Pad165) -> /Lattice MACHXO2/Digit Drivers/S3G
- D3 pad 169: /Lattice MACHXO2/Digit_2/D2A3 -> /Lattice MACHXO2/Digit Drivers/Digit 1/D1A3
- D3 pad 17: Net-(D3-Pad11) -> /Lattice MACHXO2/Digit Drivers/S1R
- D3 pad 170: Net-(D3-Pad164) -> /Lattice MACHXO2/Digit Drivers/S3R
- D3 pad 171: Net-(D3-Pad165) -> /Lattice MACHXO2/Digit Drivers/S3G
- D3 pad 172: /Lattice MACHXO2/Digit_2/D2A4 -> /Lattice MACHXO2/Digit Drivers/Digit 1/D1A4
- D3 pad 173: Net-(D3-Pad164) -> /Lattice MACHXO2/Digit Drivers/S3R
- D3 pad 174: Net-(D3-Pad165) -> /Lattice MACHXO2/Digit Drivers/S3G
- D3 pad 175: /Lattice MACHXO2/Digit_2/D2A5 -> /Lattice MACHXO2/Digit Drivers/Digit 1/D1A5
- D3 pad 176: Net-(D3-Pad164) -> /Lattice MACHXO2/Digit Drivers/S3R
- D3 pad 177: Net-(D3-Pad165) -> /Lattice MACHXO2/Digit Drivers/S3G
- D3 pad 178: /Lattice MACHXO2/Digit_2/D2A6 -> /Lattice MACHXO2/Digit Drivers/Digit 1/D1A6
- D3 pad 179: Net-(D3-Pad164) -> /Lattice MACHXO2/Digit Drivers/S3R
- D3 pad 18: Net-(D3-Pad12) -> /Lattice MACHXO2/Digit Drivers/S1G
- D3 pad 180: Net-(D3-Pad165) -> /Lattice MACHXO2/Digit Drivers/S3G
- D3 pad 181: /Lattice MACHXO2/Digit_2/D2A1 -> /Lattice MACHXO2/Digit Drivers/Digit 1/D1A1
- D3 pad 182: Net-(D3-Pad182) -> /Lattice MACHXO2/Digit Drivers/S4R
- D3 pad 183: Net-(D3-Pad183) -> /Lattice MACHXO2/Digit Drivers/S4G
- D3 pad 184: /Lattice MACHXO2/Digit_2/D2A2 -> /Lattice MACHXO2/Digit Drivers/Digit 1/D1A2
- D3 pad 185: Net-(D3-Pad182) -> /Lattice MACHXO2/Digit Drivers/S4R
- D3 pad 186: Net-(D3-Pad183) -> /Lattice MACHXO2/Digit Drivers/S4G
- D3 pad 187: /Lattice MACHXO2/Digit_2/D2A3 -> /Lattice MACHXO2/Digit Drivers/Digit 1/D1A3
- D3 pad 188: Net-(D3-Pad182) -> /Lattice MACHXO2/Digit Drivers/S4R
- D3 pad 189: Net-(D3-Pad183) -> /Lattice MACHXO2/Digit Drivers/S4G
- D3 pad 19: /Lattice MACHXO2/Digit_1/D1A1 -> /Lattice MACHXO2/Digit Drivers/Digit 1/D1A1
- D3 pad 190: /Lattice MACHXO2/Digit_2/D2A4 -> /Lattice MACHXO2/Digit Drivers/Digit 1/D1A4
- D3 pad 191: Net-(D3-Pad182) -> /Lattice MACHXO2/Digit Drivers/S4R
- D3 pad 192: Net-(D3-Pad183) -> /Lattice MACHXO2/Digit Drivers/S4G
- D3 pad 193: /Lattice MACHXO2/Digit_2/D2A5 -> /Lattice MACHXO2/Digit Drivers/Digit 1/D1A5
- D3 pad 194: Net-(D3-Pad182) -> /Lattice MACHXO2/Digit Drivers/S4R
- D3 pad 195: Net-(D3-Pad183) -> /Lattice MACHXO2/Digit Drivers/S4G
- D3 pad 196: /Lattice MACHXO2/Digit_2/D2A6 -> /Lattice MACHXO2/Digit Drivers/Digit 1/D1A6
- D3 pad 197: Net-(D3-Pad182) -> /Lattice MACHXO2/Digit Drivers/S4R
- D3 pad 198: Net-(D3-Pad183) -> /Lattice MACHXO2/Digit Drivers/S4G
- D3 pad 199: /Lattice MACHXO2/Digit_2/D2A1 -> /Lattice MACHXO2/Digit Drivers/Digit 1/D1A1
- D3 pad 2: Net-(D3-Pad11) -> /Lattice MACHXO2/Digit Drivers/S1R
- D3 pad 20: Net-(D3-Pad20) -> /Lattice MACHXO2/Digit Drivers/S2R
- D3 pad 200: Net-(D3-Pad200) -> /Lattice MACHXO2/Digit Drivers/S5R
- D3 pad 201: Net-(D3-Pad201) -> /Lattice MACHXO2/Digit Drivers/S5G
- D3 pad 202: /Lattice MACHXO2/Digit_2/D2A2 -> /Lattice MACHXO2/Digit Drivers/Digit 1/D1A2
- D3 pad 203: Net-(D3-Pad200) -> /Lattice MACHXO2/Digit Drivers/S5R
- D3 pad 204: Net-(D3-Pad201) -> /Lattice MACHXO2/Digit Drivers/S5G
- D3 pad 205: /Lattice MACHXO2/Digit_2/D2A3 -> /Lattice MACHXO2/Digit Drivers/Digit 1/D1A3
- D3 pad 206: Net-(D3-Pad200) -> /Lattice MACHXO2/Digit Drivers/S5R
- D3 pad 207: Net-(D3-Pad201) -> /Lattice MACHXO2/Digit Drivers/S5G
- D3 pad 208: /Lattice MACHXO2/Digit_2/D2A4 -> /Lattice MACHXO2/Digit Drivers/Digit 1/D1A4
- D3 pad 209: Net-(D3-Pad200) -> /Lattice MACHXO2/Digit Drivers/S5R
- D3 pad 21: Net-(D3-Pad21) -> /Lattice MACHXO2/Digit Drivers/S2G
- D3 pad 210: Net-(D3-Pad201) -> /Lattice MACHXO2/Digit Drivers/S5G
- D3 pad 211: /Lattice MACHXO2/Digit_2/D2A5 -> /Lattice MACHXO2/Digit Drivers/Digit 1/D1A5
- D3 pad 212: Net-(D3-Pad200) -> /Lattice MACHXO2/Digit Drivers/S5R
- D3 pad 213: Net-(D3-Pad201) -> /Lattice MACHXO2/Digit Drivers/S5G
- D3 pad 214: /Lattice MACHXO2/Digit_2/D2A6 -> /Lattice MACHXO2/Digit Drivers/Digit 1/D1A6
- D3 pad 215: Net-(D3-Pad200) -> /Lattice MACHXO2/Digit Drivers/S5R
- D3 pad 216: Net-(D3-Pad201) -> /Lattice MACHXO2/Digit Drivers/S5G
- D3 pad 217: /Lattice MACHXO2/Digit_2/D2A1 -> /Lattice MACHXO2/Digit Drivers/Digit 1/D1A1
- D3 pad 218: Net-(D3-Pad218) -> /Lattice MACHXO2/Digit Drivers/S6R
- D3 pad 219: Net-(D3-Pad219) -> /Lattice MACHXO2/Digit Drivers/S6G
- D3 pad 22: /Lattice MACHXO2/Digit_1/D1A2 -> /Lattice MACHXO2/Digit Drivers/Digit 1/D1A2
- D3 pad 220: /Lattice MACHXO2/Digit_2/D2A2 -> /Lattice MACHXO2/Digit Drivers/Digit 1/D1A2
- D3 pad 221: Net-(D3-Pad218) -> /Lattice MACHXO2/Digit Drivers/S6R
- D3 pad 222: Net-(D3-Pad219) -> /Lattice MACHXO2/Digit Drivers/S6G
- D3 pad 223: /Lattice MACHXO2/Digit_2/D2A3 -> /Lattice MACHXO2/Digit Drivers/Digit 1/D1A3
- D3 pad 224: Net-(D3-Pad218) -> /Lattice MACHXO2/Digit Drivers/S6R
- D3 pad 225: Net-(D3-Pad219) -> /Lattice MACHXO2/Digit Drivers/S6G
- D3 pad 226: /Lattice MACHXO2/Digit_2/D2A4 -> /Lattice MACHXO2/Digit Drivers/Digit 1/D1A4
- D3 pad 227: Net-(D3-Pad218) -> /Lattice MACHXO2/Digit Drivers/S6R
- D3 pad 228: Net-(D3-Pad219) -> /Lattice MACHXO2/Digit Drivers/S6G
- D3 pad 229: /Lattice MACHXO2/Digit_2/D2A5 -> /Lattice MACHXO2/Digit Drivers/Digit 1/D1A5
- D3 pad 23: Net-(D3-Pad20) -> /Lattice MACHXO2/Digit Drivers/S2R
- D3 pad 230: Net-(D3-Pad218) -> /Lattice MACHXO2/Digit Drivers/S6R
- D3 pad 231: Net-(D3-Pad219) -> /Lattice MACHXO2/Digit Drivers/S6G
- D3 pad 232: /Lattice MACHXO2/Digit_2/D2A6 -> /Lattice MACHXO2/Digit Drivers/Digit 1/D1A6
- D3 pad 233: Net-(D3-Pad218) -> /Lattice MACHXO2/Digit Drivers/S6R
- D3 pad 234: Net-(D3-Pad219) -> /Lattice MACHXO2/Digit Drivers/S6G
- D3 pad 235: /Lattice MACHXO2/Digit_2/D2A1 -> /Lattice MACHXO2/Digit Drivers/Digit 1/D1A1
- D3 pad 236: Net-(D3-Pad236) -> /Lattice MACHXO2/Digit Drivers/S7R
- D3 pad 237: Net-(D3-Pad237) -> /Lattice MACHXO2/Digit Drivers/S7G
- D3 pad 238: /Lattice MACHXO2/Digit_2/D2A2 -> /Lattice MACHXO2/Digit Drivers/Digit 1/D1A2
- D3 pad 239: Net-(D3-Pad236) -> /Lattice MACHXO2/Digit Drivers/S7R
- D3 pad 24: Net-(D3-Pad21) -> /Lattice MACHXO2/Digit Drivers/S2G
- D3 pad 240: Net-(D3-Pad237) -> /Lattice MACHXO2/Digit Drivers/S7G
- D3 pad 241: /Lattice MACHXO2/Digit_2/D2A3 -> /Lattice MACHXO2/Digit Drivers/Digit 1/D1A3
- D3 pad 242: Net-(D3-Pad242) -> /Lattice MACHXO2/Digit Drivers/S7R
- D3 pad 243: Net-(D3-Pad237) -> /Lattice MACHXO2/Digit Drivers/S7G
- D3 pad 244: /Lattice MACHXO2/Digit_2/D2A4 -> /Lattice MACHXO2/Digit Drivers/Digit 1/D1A4
- D3 pad 245: Net-(D3-Pad236) -> /Lattice MACHXO2/Digit Drivers/S7R
- D3 pad 246: Net-(D3-Pad237) -> /Lattice MACHXO2/Digit Drivers/S7G
- D3 pad 247: /Lattice MACHXO2/Digit_2/D2A5 -> /Lattice MACHXO2/Digit Drivers/Digit 1/D1A5
- D3 pad 248: Net-(D3-Pad236) -> /Lattice MACHXO2/Digit Drivers/S7R
- D3 pad 249: Net-(D3-Pad237) -> /Lattice MACHXO2/Digit Drivers/S7G
- D3 pad 25: /Lattice MACHXO2/Digit_1/D1A3 -> /Lattice MACHXO2/Digit Drivers/Digit 1/D1A3
- D3 pad 250: /Lattice MACHXO2/Digit_2/D2A6 -> /Lattice MACHXO2/Digit Drivers/Digit 1/D1A6
- D3 pad 251: Net-(D3-Pad236) -> /Lattice MACHXO2/Digit Drivers/S7R
- D3 pad 252: Net-(D3-Pad237) -> /Lattice MACHXO2/Digit Drivers/S7G
- D3 pad 253: /Lattice MACHXO2/Digit_3/D3A1 -> /Lattice MACHXO2/Digit Drivers/Digit 1/D1A1
- D3 pad 254: Net-(D3-Pad254) -> /Lattice MACHXO2/Digit Drivers/S1R
- D3 pad 255: Net-(D3-Pad255) -> /Lattice MACHXO2/Digit Drivers/S1G
- D3 pad 256: /Lattice MACHXO2/Digit_3/D3A2 -> /Lattice MACHXO2/Digit Drivers/Digit 1/D1A2
- D3 pad 257: Net-(D3-Pad254) -> /Lattice MACHXO2/Digit Drivers/S1R
- D3 pad 258: Net-(D3-Pad255) -> /Lattice MACHXO2/Digit Drivers/S1G
- D3 pad 259: /Lattice MACHXO2/Digit_3/D3A3 -> /Lattice MACHXO2/Digit Drivers/Digit 1/D1A3
- D3 pad 26: Net-(D3-Pad20) -> /Lattice MACHXO2/Digit Drivers/S2R
- D3 pad 260: Net-(D3-Pad254) -> /Lattice MACHXO2/Digit Drivers/S1R
- D3 pad 261: Net-(D3-Pad255) -> /Lattice MACHXO2/Digit Drivers/S1G
- D3 pad 262: /Lattice MACHXO2/Digit_3/D3A4 -> /Lattice MACHXO2/Digit Drivers/Digit 1/D1A4
- D3 pad 263: Net-(D3-Pad254) -> /Lattice MACHXO2/Digit Drivers/S1R
- D3 pad 264: Net-(D3-Pad255) -> /Lattice MACHXO2/Digit Drivers/S1G
- D3 pad 265: /Lattice MACHXO2/Digit_3/D3A5 -> /Lattice MACHXO2/Digit Drivers/Digit 1/D1A5
- D3 pad 266: Net-(D3-Pad254) -> /Lattice MACHXO2/Digit Drivers/S1R
- D3 pad 267: Net-(D3-Pad255) -> /Lattice MACHXO2/Digit Drivers/S1G
- D3 pad 268: /Lattice MACHXO2/Digit_3/D3A6 -> /Lattice MACHXO2/Digit Drivers/Digit 1/D1A6
- D3 pad 269: Net-(D3-Pad254) -> /Lattice MACHXO2/Digit Drivers/S1R
- D3 pad 27: Net-(D3-Pad21) -> /Lattice MACHXO2/Digit Drivers/S2G
- D3 pad 270: Net-(D3-Pad255) -> /Lattice MACHXO2/Digit Drivers/S1G
- D3 pad 271: /Lattice MACHXO2/Digit_3/D3A1 -> /Lattice MACHXO2/Digit Drivers/Digit 1/D1A1
- D3 pad 272: Net-(D3-Pad272) -> /Lattice MACHXO2/Digit Drivers/S2R
- D3 pad 273: Net-(D3-Pad273) -> /Lattice MACHXO2/Digit Drivers/S2G
- D3 pad 274: /Lattice MACHXO2/Digit_3/D3A2 -> /Lattice MACHXO2/Digit Drivers/Digit 1/D1A2
- D3 pad 275: Net-(D3-Pad272) -> /Lattice MACHXO2/Digit Drivers/S2R
- D3 pad 276: Net-(D3-Pad273) -> /Lattice MACHXO2/Digit Drivers/S2G
- D3 pad 277: /Lattice MACHXO2/Digit_3/D3A3 -> /Lattice MACHXO2/Digit Drivers/Digit 1/D1A3
- D3 pad 278: Net-(D3-Pad272) -> /Lattice MACHXO2/Digit Drivers/S2R
- D3 pad 279: Net-(D3-Pad273) -> /Lattice MACHXO2/Digit Drivers/S2G
- D3 pad 28: /Lattice MACHXO2/Digit_1/D1A4 -> /Lattice MACHXO2/Digit Drivers/Digit 1/D1A4
- D3 pad 280: /Lattice MACHXO2/Digit_3/D3A4 -> /Lattice MACHXO2/Digit Drivers/Digit 1/D1A4
- D3 pad 281: Net-(D3-Pad272) -> /Lattice MACHXO2/Digit Drivers/S2R
- D3 pad 282: Net-(D3-Pad273) -> /Lattice MACHXO2/Digit Drivers/S2G
- D3 pad 283: /Lattice MACHXO2/Digit_3/D3A5 -> /Lattice MACHXO2/Digit Drivers/Digit 1/D1A5
- D3 pad 284: Net-(D3-Pad272) -> /Lattice MACHXO2/Digit Drivers/S2R
- D3 pad 285: Net-(D3-Pad273) -> /Lattice MACHXO2/Digit Drivers/S2G
- D3 pad 286: /Lattice MACHXO2/Digit_3/D3A6 -> /Lattice MACHXO2/Digit Drivers/Digit 1/D1A6
- D3 pad 287: Net-(D3-Pad272) -> /Lattice MACHXO2/Digit Drivers/S2R
- D3 pad 288: Net-(D3-Pad273) -> /Lattice MACHXO2/Digit Drivers/S2G
- D3 pad 289: /Lattice MACHXO2/Digit_3/D3A1 -> /Lattice MACHXO2/Digit Drivers/Digit 1/D1A1
- D3 pad 29: Net-(D3-Pad20) -> /Lattice MACHXO2/Digit Drivers/S2R
- D3 pad 290: Net-(D3-Pad290) -> /Lattice MACHXO2/Digit Drivers/S3R
- D3 pad 291: Net-(D3-Pad291) -> /Lattice MACHXO2/Digit Drivers/S3G
- D3 pad 292: /Lattice MACHXO2/Digit_3/D3A2 -> /Lattice MACHXO2/Digit Drivers/Digit 1/D1A2
- D3 pad 293: Net-(D3-Pad290) -> /Lattice MACHXO2/Digit Drivers/S3R
- D3 pad 294: Net-(D3-Pad291) -> /Lattice MACHXO2/Digit Drivers/S3G
- D3 pad 295: /Lattice MACHXO2/Digit_3/D3A3 -> /Lattice MACHXO2/Digit Drivers/Digit 1/D1A3
- D3 pad 296: Net-(D3-Pad290) -> /Lattice MACHXO2/Digit Drivers/S3R
- D3 pad 297: Net-(D3-Pad291) -> /Lattice MACHXO2/Digit Drivers/S3G
- D3 pad 298: /Lattice MACHXO2/Digit_3/D3A4 -> /Lattice MACHXO2/Digit Drivers/Digit 1/D1A4
- D3 pad 299: Net-(D3-Pad290) -> /Lattice MACHXO2/Digit Drivers/S3R
- D3 pad 3: Net-(D3-Pad12) -> /Lattice MACHXO2/Digit Drivers/S1G
- D3 pad 30: Net-(D3-Pad21) -> /Lattice MACHXO2/Digit Drivers/S2G
- D3 pad 300: Net-(D3-Pad291) -> /Lattice MACHXO2/Digit Drivers/S3G
- D3 pad 301: /Lattice MACHXO2/Digit_3/D3A5 -> /Lattice MACHXO2/Digit Drivers/Digit 1/D1A5
- D3 pad 302: Net-(D3-Pad290) -> /Lattice MACHXO2/Digit Drivers/S3R
- D3 pad 303: Net-(D3-Pad291) -> /Lattice MACHXO2/Digit Drivers/S3G
- D3 pad 304: /Lattice MACHXO2/Digit_3/D3A6 -> /Lattice MACHXO2/Digit Drivers/Digit 1/D1A6
- D3 pad 305: Net-(D3-Pad290) -> /Lattice MACHXO2/Digit Drivers/S3R
- D3 pad 306: Net-(D3-Pad291) -> /Lattice MACHXO2/Digit Drivers/S3G
- D3 pad 307: /Lattice MACHXO2/Digit_3/D3A1 -> /Lattice MACHXO2/Digit Drivers/Digit 1/D1A1
- D3 pad 308: Net-(D3-Pad308) -> /Lattice MACHXO2/Digit Drivers/S4R
- D3 pad 309: Net-(D3-Pad309) -> /Lattice MACHXO2/Digit Drivers/S4G
- D3 pad 31: /Lattice MACHXO2/Digit_1/D1A5 -> /Lattice MACHXO2/Digit Drivers/Digit 1/D1A5
- D3 pad 310: /Lattice MACHXO2/Digit_3/D3A2 -> /Lattice MACHXO2/Digit Drivers/Digit 1/D1A2
- D3 pad 311: Net-(D3-Pad308) -> /Lattice MACHXO2/Digit Drivers/S4R
- D3 pad 312: Net-(D3-Pad309) -> /Lattice MACHXO2/Digit Drivers/S4G
- D3 pad 313: /Lattice MACHXO2/Digit_3/D3A3 -> /Lattice MACHXO2/Digit Drivers/Digit 1/D1A3
- D3 pad 314: Net-(D3-Pad308) -> /Lattice MACHXO2/Digit Drivers/S4R
- D3 pad 315: Net-(D3-Pad309) -> /Lattice MACHXO2/Digit Drivers/S4G
- D3 pad 316: /Lattice MACHXO2/Digit_3/D3A4 -> /Lattice MACHXO2/Digit Drivers/Digit 1/D1A4
- D3 pad 317: Net-(D3-Pad308) -> /Lattice MACHXO2/Digit Drivers/S4R
- D3 pad 318: Net-(D3-Pad309) -> /Lattice MACHXO2/Digit Drivers/S4G
- D3 pad 319: /Lattice MACHXO2/Digit_3/D3A5 -> /Lattice MACHXO2/Digit Drivers/Digit 1/D1A5
- D3 pad 32: Net-(D3-Pad20) -> /Lattice MACHXO2/Digit Drivers/S2R
- D3 pad 320: Net-(D3-Pad308) -> /Lattice MACHXO2/Digit Drivers/S4R
- D3 pad 321: Net-(D3-Pad309) -> /Lattice MACHXO2/Digit Drivers/S4G
- D3 pad 322: /Lattice MACHXO2/Digit_3/D3A6 -> /Lattice MACHXO2/Digit Drivers/Digit 1/D1A6
- D3 pad 323: Net-(D3-Pad308) -> /Lattice MACHXO2/Digit Drivers/S4R
- D3 pad 324: Net-(D3-Pad309) -> /Lattice MACHXO2/Digit Drivers/S4G
- D3 pad 325: /Lattice MACHXO2/Digit_3/D3A1 -> /Lattice MACHXO2/Digit Drivers/Digit 1/D1A1
- D3 pad 326: Net-(D3-Pad326) -> /Lattice MACHXO2/Digit Drivers/S5R
- D3 pad 327: Net-(D3-Pad327) -> /Lattice MACHXO2/Digit Drivers/S5G
- D3 pad 328: /Lattice MACHXO2/Digit_3/D3A2 -> /Lattice MACHXO2/Digit Drivers/Digit 1/D1A2
- D3 pad 329: Net-(D3-Pad326) -> /Lattice MACHXO2/Digit Drivers/S5R
- D3 pad 33: Net-(D3-Pad21) -> /Lattice MACHXO2/Digit Drivers/S2G
- D3 pad 330: Net-(D3-Pad327) -> /Lattice MACHXO2/Digit Drivers/S5G
- D3 pad 331: /Lattice MACHXO2/Digit_3/D3A3 -> /Lattice MACHXO2/Digit Drivers/Digit 1/D1A3
- D3 pad 332: Net-(D3-Pad326) -> /Lattice MACHXO2/Digit Drivers/S5R
- D3 pad 333: Net-(D3-Pad327) -> /Lattice MACHXO2/Digit Drivers/S5G
- D3 pad 334: /Lattice MACHXO2/Digit_3/D3A4 -> /Lattice MACHXO2/Digit Drivers/Digit 1/D1A4
- D3 pad 335: Net-(D3-Pad326) -> /Lattice MACHXO2/Digit Drivers/S5R
- D3 pad 336: Net-(D3-Pad327) -> /Lattice MACHXO2/Digit Drivers/S5G
- D3 pad 337: /Lattice MACHXO2/Digit_3/D3A5 -> /Lattice MACHXO2/Digit Drivers/Digit 1/D1A5
- D3 pad 338: Net-(D3-Pad326) -> /Lattice MACHXO2/Digit Drivers/S5R
- D3 pad 339: Net-(D3-Pad327) -> /Lattice MACHXO2/Digit Drivers/S5G
- D3 pad 34: /Lattice MACHXO2/Digit_1/D1A6 -> /Lattice MACHXO2/Digit Drivers/Digit 1/D1A6
- D3 pad 340: /Lattice MACHXO2/Digit_3/D3A6 -> /Lattice MACHXO2/Digit Drivers/Digit 1/D1A6
- D3 pad 341: Net-(D3-Pad326) -> /Lattice MACHXO2/Digit Drivers/S5R
- D3 pad 342: Net-(D3-Pad327) -> /Lattice MACHXO2/Digit Drivers/S5G
- D3 pad 343: /Lattice MACHXO2/Digit_3/D3A1 -> /Lattice MACHXO2/Digit Drivers/Digit 1/D1A1
- D3 pad 344: Net-(D3-Pad344) -> /Lattice MACHXO2/Digit Drivers/S6R
- D3 pad 345: Net-(D3-Pad345) -> /Lattice MACHXO2/Digit Drivers/S6G
- D3 pad 346: /Lattice MACHXO2/Digit_3/D3A2 -> /Lattice MACHXO2/Digit Drivers/Digit 1/D1A2
- D3 pad 347: Net-(D3-Pad344) -> /Lattice MACHXO2/Digit Drivers/S6R
- D3 pad 348: Net-(D3-Pad345) -> /Lattice MACHXO2/Digit Drivers/S6G
- D3 pad 349: /Lattice MACHXO2/Digit_3/D3A3 -> /Lattice MACHXO2/Digit Drivers/Digit 1/D1A3
- D3 pad 35: Net-(D3-Pad20) -> /Lattice MACHXO2/Digit Drivers/S2R
- D3 pad 350: Net-(D3-Pad344) -> /Lattice MACHXO2/Digit Drivers/S6R
- D3 pad 351: Net-(D3-Pad345) -> /Lattice MACHXO2/Digit Drivers/S6G
- D3 pad 352: /Lattice MACHXO2/Digit_3/D3A4 -> /Lattice MACHXO2/Digit Drivers/Digit 1/D1A4
- D3 pad 353: Net-(D3-Pad344) -> /Lattice MACHXO2/Digit Drivers/S6R
- D3 pad 354: Net-(D3-Pad345) -> /Lattice MACHXO2/Digit Drivers/S6G
- D3 pad 355: /Lattice MACHXO2/Digit_3/D3A5 -> /Lattice MACHXO2/Digit Drivers/Digit 1/D1A5
- D3 pad 356: Net-(D3-Pad344) -> /Lattice MACHXO2/Digit Drivers/S6R
- D3 pad 357: Net-(D3-Pad345) -> /Lattice MACHXO2/Digit Drivers/S6G
- D3 pad 358: /Lattice MACHXO2/Digit_3/D3A6 -> /Lattice MACHXO2/Digit Drivers/Digit 1/D1A6
- D3 pad 359: Net-(D3-Pad344) -> /Lattice MACHXO2/Digit Drivers/S6R
- D3 pad 36: Net-(D3-Pad21) -> /Lattice MACHXO2/Digit Drivers/S2G
- D3 pad 360: Net-(D3-Pad345) -> /Lattice MACHXO2/Digit Drivers/S6G
- D3 pad 361: /Lattice MACHXO2/Digit_3/D3A1 -> /Lattice MACHXO2/Digit Drivers/Digit 1/D1A1
- D3 pad 362: Net-(D3-Pad362) -> /Lattice MACHXO2/Digit Drivers/S7R
- D3 pad 363: Net-(D3-Pad363) -> /Lattice MACHXO2/Digit Drivers/S7G
- D3 pad 364: /Lattice MACHXO2/Digit_3/D3A2 -> /Lattice MACHXO2/Digit Drivers/Digit 1/D1A2
- D3 pad 365: Net-(D3-Pad362) -> /Lattice MACHXO2/Digit Drivers/S7R
- D3 pad 366: Net-(D3-Pad363) -> /Lattice MACHXO2/Digit Drivers/S7G
- D3 pad 367: /Lattice MACHXO2/Digit_3/D3A3 -> /Lattice MACHXO2/Digit Drivers/Digit 1/D1A3
- D3 pad 368: Net-(D3-Pad368) -> /Lattice MACHXO2/Digit Drivers/S7R
- D3 pad 369: Net-(D3-Pad363) -> /Lattice MACHXO2/Digit Drivers/S7G
- D3 pad 37: /Lattice MACHXO2/Digit_1/D1A1 -> /Lattice MACHXO2/Digit Drivers/Digit 1/D1A1
- D3 pad 370: /Lattice MACHXO2/Digit_3/D3A4 -> /Lattice MACHXO2/Digit Drivers/Digit 1/D1A4
- D3 pad 371: Net-(D3-Pad362) -> /Lattice MACHXO2/Digit Drivers/S7R
- D3 pad 372: Net-(D3-Pad363) -> /Lattice MACHXO2/Digit Drivers/S7G
- D3 pad 373: /Lattice MACHXO2/Digit_3/D3A5 -> /Lattice MACHXO2/Digit Drivers/Digit 1/D1A5
- D3 pad 374: Net-(D3-Pad362) -> /Lattice MACHXO2/Digit Drivers/S7R
- D3 pad 375: Net-(D3-Pad363) -> /Lattice MACHXO2/Digit Drivers/S7G
- D3 pad 376: /Lattice MACHXO2/Digit_3/D3A6 -> /Lattice MACHXO2/Digit Drivers/Digit 1/D1A6
- D3 pad 377: Net-(D3-Pad362) -> /Lattice MACHXO2/Digit Drivers/S7R
- D3 pad 378: Net-(D3-Pad363) -> /Lattice MACHXO2/Digit Drivers/S7G
- D3 pad 379: /Lattice MACHXO2/Digit_4/D4A1 -> /Lattice MACHXO2/Digit Drivers/Digit 1/D1A1
- D3 pad 38: Net-(D3-Pad38) -> /Lattice MACHXO2/Digit Drivers/S3R
- D3 pad 380: Net-(D3-Pad380) -> /Lattice MACHXO2/Digit Drivers/S1R
- D3 pad 381: Net-(D3-Pad381) -> /Lattice MACHXO2/Digit Drivers/S1G
- D3 pad 382: /Lattice MACHXO2/Digit_4/D4A2 -> /Lattice MACHXO2/Digit Drivers/Digit 1/D1A2
- D3 pad 383: Net-(D3-Pad380) -> /Lattice MACHXO2/Digit Drivers/S1R
- D3 pad 384: Net-(D3-Pad381) -> /Lattice MACHXO2/Digit Drivers/S1G
- D3 pad 385: /Lattice MACHXO2/Digit_4/D4A3 -> /Lattice MACHXO2/Digit Drivers/Digit 1/D1A3
- D3 pad 386: Net-(D3-Pad380) -> /Lattice MACHXO2/Digit Drivers/S1R
- D3 pad 387: Net-(D3-Pad381) -> /Lattice MACHXO2/Digit Drivers/S1G
- D3 pad 388: /Lattice MACHXO2/Digit_4/D4A4 -> /Lattice MACHXO2/Digit Drivers/Digit 1/D1A4
- D3 pad 389: Net-(D3-Pad380) -> /Lattice MACHXO2/Digit Drivers/S1R
- D3 pad 39: Net-(D3-Pad39) -> /Lattice MACHXO2/Digit Drivers/S3G
- D3 pad 390: Net-(D3-Pad381) -> /Lattice MACHXO2/Digit Drivers/S1G
- D3 pad 391: /Lattice MACHXO2/Digit_4/D4A5 -> /Lattice MACHXO2/Digit Drivers/Digit 1/D1A5
- D3 pad 392: Net-(D3-Pad380) -> /Lattice MACHXO2/Digit Drivers/S1R
- D3 pad 393: Net-(D3-Pad381) -> /Lattice MACHXO2/Digit Drivers/S1G
- D3 pad 394: /Lattice MACHXO2/Digit_4/D4A6 -> /Lattice MACHXO2/Digit Drivers/Digit 1/D1A6
- D3 pad 395: Net-(D3-Pad380) -> /Lattice MACHXO2/Digit Drivers/S1R
- D3 pad 396: Net-(D3-Pad381) -> /Lattice MACHXO2/Digit Drivers/S1G
- D3 pad 397: /Lattice MACHXO2/Digit_4/D4A1 -> /Lattice MACHXO2/Digit Drivers/Digit 1/D1A1
- D3 pad 398: Net-(D3-Pad398) -> /Lattice MACHXO2/Digit Drivers/S2R
- D3 pad 399: Net-(D3-Pad399) -> /Lattice MACHXO2/Digit Drivers/S2G
- D3 pad 4: /Lattice MACHXO2/Digit_1/D1A2 -> /Lattice MACHXO2/Digit Drivers/Digit 1/D1A2
- D3 pad 40: /Lattice MACHXO2/Digit_1/D1A2 -> /Lattice MACHXO2/Digit Drivers/Digit 1/D1A2
- D3 pad 400: /Lattice MACHXO2/Digit_4/D4A2 -> /Lattice MACHXO2/Digit Drivers/Digit 1/D1A2
- D3 pad 401: Net-(D3-Pad398) -> /Lattice MACHXO2/Digit Drivers/S2R
- D3 pad 402: Net-(D3-Pad399) -> /Lattice MACHXO2/Digit Drivers/S2G
- D3 pad 403: /Lattice MACHXO2/Digit_4/D4A3 -> /Lattice MACHXO2/Digit Drivers/Digit 1/D1A3
- D3 pad 404: Net-(D3-Pad398) -> /Lattice MACHXO2/Digit Drivers/S2R
- D3 pad 405: Net-(D3-Pad399) -> /Lattice MACHXO2/Digit Drivers/S2G
- D3 pad 406: /Lattice MACHXO2/Digit_4/D4A4 -> /Lattice MACHXO2/Digit Drivers/Digit 1/D1A4
- D3 pad 407: Net-(D3-Pad398) -> /Lattice MACHXO2/Digit Drivers/S2R
- D3 pad 408: Net-(D3-Pad399) -> /Lattice MACHXO2/Digit Drivers/S2G
- D3 pad 409: /Lattice MACHXO2/Digit_4/D4A5 -> /Lattice MACHXO2/Digit Drivers/Digit 1/D1A5
- D3 pad 41: Net-(D3-Pad38) -> /Lattice MACHXO2/Digit Drivers/S3R
- D3 pad 410: Net-(D3-Pad398) -> /Lattice MACHXO2/Digit Drivers/S2R
- D3 pad 411: Net-(D3-Pad399) -> /Lattice MACHXO2/Digit Drivers/S2G
- D3 pad 412: /Lattice MACHXO2/Digit_4/D4A6 -> /Lattice MACHXO2/Digit Drivers/Digit 1/D1A6
- D3 pad 413: Net-(D3-Pad398) -> /Lattice MACHXO2/Digit Drivers/S2R
- D3 pad 414: Net-(D3-Pad399) -> /Lattice MACHXO2/Digit Drivers/S2G
- D3 pad 415: /Lattice MACHXO2/Digit_4/D4A1 -> /Lattice MACHXO2/Digit Drivers/Digit 1/D1A1
- D3 pad 416: Net-(D3-Pad416) -> /Lattice MACHXO2/Digit Drivers/S3R
- D3 pad 417: Net-(D3-Pad417) -> /Lattice MACHXO2/Digit Drivers/S3G
- D3 pad 418: /Lattice MACHXO2/Digit_4/D4A2 -> /Lattice MACHXO2/Digit Drivers/Digit 1/D1A2
- D3 pad 419: Net-(D3-Pad416) -> /Lattice MACHXO2/Digit Drivers/S3R
- D3 pad 42: Net-(D3-Pad39) -> /Lattice MACHXO2/Digit Drivers/S3G
- D3 pad 420: Net-(D3-Pad417) -> /Lattice MACHXO2/Digit Drivers/S3G
- D3 pad 421: /Lattice MACHXO2/Digit_4/D4A3 -> /Lattice MACHXO2/Digit Drivers/Digit 1/D1A3
- D3 pad 422: Net-(D3-Pad416) -> /Lattice MACHXO2/Digit Drivers/S3R
- D3 pad 423: Net-(D3-Pad417) -> /Lattice MACHXO2/Digit Drivers/S3G
- D3 pad 424: /Lattice MACHXO2/Digit_4/D4A4 -> /Lattice MACHXO2/Digit Drivers/Digit 1/D1A4
- D3 pad 425: Net-(D3-Pad416) -> /Lattice MACHXO2/Digit Drivers/S3R
- D3 pad 426: Net-(D3-Pad417) -> /Lattice MACHXO2/Digit Drivers/S3G
- D3 pad 427: /Lattice MACHXO2/Digit_4/D4A5 -> /Lattice MACHXO2/Digit Drivers/Digit 1/D1A5
- D3 pad 428: Net-(D3-Pad416) -> /Lattice MACHXO2/Digit Drivers/S3R
- D3 pad 429: Net-(D3-Pad417) -> /Lattice MACHXO2/Digit Drivers/S3G
- D3 pad 43: /Lattice MACHXO2/Digit_1/D1A3 -> /Lattice MACHXO2/Digit Drivers/Digit 1/D1A3
- D3 pad 430: /Lattice MACHXO2/Digit_4/D4A6 -> /Lattice MACHXO2/Digit Drivers/Digit 1/D1A6
- D3 pad 431: Net-(D3-Pad416) -> /Lattice MACHXO2/Digit Drivers/S3R
- D3 pad 432: Net-(D3-Pad417) -> /Lattice MACHXO2/Digit Drivers/S3G
- D3 pad 433: /Lattice MACHXO2/Digit_4/D4A1 -> /Lattice MACHXO2/Digit Drivers/Digit 1/D1A1
- D3 pad 434: Net-(D3-Pad434) -> /Lattice MACHXO2/Digit Drivers/S4R
- D3 pad 435: Net-(D3-Pad435) -> /Lattice MACHXO2/Digit Drivers/S4G
- D3 pad 436: /Lattice MACHXO2/Digit_4/D4A2 -> /Lattice MACHXO2/Digit Drivers/Digit 1/D1A2
- D3 pad 437: Net-(D3-Pad434) -> /Lattice MACHXO2/Digit Drivers/S4R
- D3 pad 438: Net-(D3-Pad435) -> /Lattice MACHXO2/Digit Drivers/S4G
- D3 pad 439: /Lattice MACHXO2/Digit_4/D4A3 -> /Lattice MACHXO2/Digit Drivers/Digit 1/D1A3
- D3 pad 44: Net-(D3-Pad38) -> /Lattice MACHXO2/Digit Drivers/S3R
- D3 pad 440: Net-(D3-Pad434) -> /Lattice MACHXO2/Digit Drivers/S4R
- D3 pad 441: Net-(D3-Pad435) -> /Lattice MACHXO2/Digit Drivers/S4G
- D3 pad 442: /Lattice MACHXO2/Digit_4/D4A4 -> /Lattice MACHXO2/Digit Drivers/Digit 1/D1A4
- D3 pad 443: Net-(D3-Pad434) -> /Lattice MACHXO2/Digit Drivers/S4R
- D3 pad 444: Net-(D3-Pad435) -> /Lattice MACHXO2/Digit Drivers/S4G
- D3 pad 445: /Lattice MACHXO2/Digit_4/D4A5 -> /Lattice MACHXO2/Digit Drivers/Digit 1/D1A5
- D3 pad 446: Net-(D3-Pad434) -> /Lattice MACHXO2/Digit Drivers/S4R
- D3 pad 447: Net-(D3-Pad435) -> /Lattice MACHXO2/Digit Drivers/S4G
- D3 pad 448: /Lattice MACHXO2/Digit_4/D4A6 -> /Lattice MACHXO2/Digit Drivers/Digit 1/D1A6
- D3 pad 449: Net-(D3-Pad434) -> /Lattice MACHXO2/Digit Drivers/S4R
- D3 pad 45: Net-(D3-Pad39) -> /Lattice MACHXO2/Digit Drivers/S3G
- D3 pad 450: Net-(D3-Pad435) -> /Lattice MACHXO2/Digit Drivers/S4G
- D3 pad 451: /Lattice MACHXO2/Digit_4/D4A1 -> /Lattice MACHXO2/Digit Drivers/Digit 1/D1A1
- D3 pad 452: Net-(D3-Pad452) -> /Lattice MACHXO2/Digit Drivers/S5R
- D3 pad 453: Net-(D3-Pad453) -> /Lattice MACHXO2/Digit Drivers/S5G
- D3 pad 454: /Lattice MACHXO2/Digit_4/D4A2 -> /Lattice MACHXO2/Digit Drivers/Digit 1/D1A2
- D3 pad 455: Net-(D3-Pad452) -> /Lattice MACHXO2/Digit Drivers/S5R
- D3 pad 456: Net-(D3-Pad453) -> /Lattice MACHXO2/Digit Drivers/S5G
- D3 pad 457: /Lattice MACHXO2/Digit_4/D4A3 -> /Lattice MACHXO2/Digit Drivers/Digit 1/D1A3
- D3 pad 458: Net-(D3-Pad452) -> /Lattice MACHXO2/Digit Drivers/S5R
- D3 pad 459: Net-(D3-Pad453) -> /Lattice MACHXO2/Digit Drivers/S5G
- D3 pad 46: /Lattice MACHXO2/Digit_1/D1A4 -> /Lattice MACHXO2/Digit Drivers/Digit 1/D1A4
- D3 pad 460: /Lattice MACHXO2/Digit_4/D4A4 -> /Lattice MACHXO2/Digit Drivers/Digit 1/D1A4
- D3 pad 461: Net-(D3-Pad452) -> /Lattice MACHXO2/Digit Drivers/S5R
- D3 pad 462: Net-(D3-Pad453) -> /Lattice MACHXO2/Digit Drivers/S5G
- D3 pad 463: /Lattice MACHXO2/Digit_4/D4A5 -> /Lattice MACHXO2/Digit Drivers/Digit 1/D1A5
- D3 pad 464: Net-(D3-Pad452) -> /Lattice MACHXO2/Digit Drivers/S5R
- D3 pad 465: Net-(D3-Pad453) -> /Lattice MACHXO2/Digit Drivers/S5G
- D3 pad 466: /Lattice MACHXO2/Digit_4/D4A6 -> /Lattice MACHXO2/Digit Drivers/Digit 1/D1A6
- D3 pad 467: Net-(D3-Pad452) -> /Lattice MACHXO2/Digit Drivers/S5R
- D3 pad 468: Net-(D3-Pad453) -> /Lattice MACHXO2/Digit Drivers/S5G
- D3 pad 469: /Lattice MACHXO2/Digit_4/D4A1 -> /Lattice MACHXO2/Digit Drivers/Digit 1/D1A1
- D3 pad 47: Net-(D3-Pad38) -> /Lattice MACHXO2/Digit Drivers/S3R
- D3 pad 470: Net-(D3-Pad470) -> /Lattice MACHXO2/Digit Drivers/S6R
- D3 pad 471: Net-(D3-Pad471) -> /Lattice MACHXO2/Digit Drivers/S6G
- D3 pad 472: /Lattice MACHXO2/Digit_4/D4A2 -> /Lattice MACHXO2/Digit Drivers/Digit 1/D1A2
- D3 pad 473: Net-(D3-Pad470) -> /Lattice MACHXO2/Digit Drivers/S6R
- D3 pad 474: Net-(D3-Pad471) -> /Lattice MACHXO2/Digit Drivers/S6G
- D3 pad 475: /Lattice MACHXO2/Digit_4/D4A3 -> /Lattice MACHXO2/Digit Drivers/Digit 1/D1A3
- D3 pad 476: Net-(D3-Pad470) -> /Lattice MACHXO2/Digit Drivers/S6R
- D3 pad 477: Net-(D3-Pad471) -> /Lattice MACHXO2/Digit Drivers/S6G
- D3 pad 478: /Lattice MACHXO2/Digit_4/D4A4 -> /Lattice MACHXO2/Digit Drivers/Digit 1/D1A4
- D3 pad 479: Net-(D3-Pad470) -> /Lattice MACHXO2/Digit Drivers/S6R
- D3 pad 48: Net-(D3-Pad39) -> /Lattice MACHXO2/Digit Drivers/S3G
- D3 pad 480: Net-(D3-Pad471) -> /Lattice MACHXO2/Digit Drivers/S6G
- D3 pad 481: /Lattice MACHXO2/Digit_4/D4A5 -> /Lattice MACHXO2/Digit Drivers/Digit 1/D1A5
- D3 pad 482: Net-(D3-Pad470) -> /Lattice MACHXO2/Digit Drivers/S6R
- D3 pad 483: Net-(D3-Pad471) -> /Lattice MACHXO2/Digit Drivers/S6G
- D3 pad 484: /Lattice MACHXO2/Digit_4/D4A6 -> /Lattice MACHXO2/Digit Drivers/Digit 1/D1A6
- D3 pad 485: Net-(D3-Pad470) -> /Lattice MACHXO2/Digit Drivers/S6R
- D3 pad 486: Net-(D3-Pad471) -> /Lattice MACHXO2/Digit Drivers/S6G
- D3 pad 487: /Lattice MACHXO2/Digit_4/D4A1 -> /Lattice MACHXO2/Digit Drivers/Digit 1/D1A1
- D3 pad 488: Net-(D3-Pad488) -> /Lattice MACHXO2/Digit Drivers/S7R
- D3 pad 489: Net-(D3-Pad489) -> /Lattice MACHXO2/Digit Drivers/S7G
- D3 pad 49: /Lattice MACHXO2/Digit_1/D1A5 -> /Lattice MACHXO2/Digit Drivers/Digit 1/D1A5
- D3 pad 490: /Lattice MACHXO2/Digit_4/D4A2 -> /Lattice MACHXO2/Digit Drivers/Digit 1/D1A2
- D3 pad 491: Net-(D3-Pad488) -> /Lattice MACHXO2/Digit Drivers/S7R
- D3 pad 492: Net-(D3-Pad489) -> /Lattice MACHXO2/Digit Drivers/S7G
- D3 pad 493: /Lattice MACHXO2/Digit_4/D4A3 -> /Lattice MACHXO2/Digit Drivers/Digit 1/D1A3
- D3 pad 494: Net-(D3-Pad488) -> /Lattice MACHXO2/Digit Drivers/S7R
- D3 pad 495: Net-(D3-Pad489) -> /Lattice MACHXO2/Digit Drivers/S7G
- D3 pad 496: /Lattice MACHXO2/Digit_4/D4A4 -> /Lattice MACHXO2/Digit Drivers/Digit 1/D1A4
- D3 pad 497: Net-(D3-Pad488) -> /Lattice MACHXO2/Digit Drivers/S7R
- D3 pad 498: Net-(D3-Pad489) -> /Lattice MACHXO2/Digit Drivers/S7G
- D3 pad 499: /Lattice MACHXO2/Digit_4/D4A5 -> /Lattice MACHXO2/Digit Drivers/Digit 1/D1A5
- D3 pad 5: Net-(D3-Pad11) -> /Lattice MACHXO2/Digit Drivers/S1R
- D3 pad 50: Net-(D3-Pad38) -> /Lattice MACHXO2/Digit Drivers/S3R
- D3 pad 500: Net-(D3-Pad488) -> /Lattice MACHXO2/Digit Drivers/S7R
- D3 pad 501: Net-(D3-Pad489) -> /Lattice MACHXO2/Digit Drivers/S7G
- D3 pad 502: /Lattice MACHXO2/Digit_4/D4A6 -> /Lattice MACHXO2/Digit Drivers/Digit 1/D1A6
- D3 pad 503: Net-(D3-Pad488) -> /Lattice MACHXO2/Digit Drivers/S7R
- D3 pad 504: Net-(D3-Pad489) -> /Lattice MACHXO2/Digit Drivers/S7G
- D3 pad 51: Net-(D3-Pad39) -> /Lattice MACHXO2/Digit Drivers/S3G
- D3 pad 52: /Lattice MACHXO2/Digit_1/D1A6 -> /Lattice MACHXO2/Digit Drivers/Digit 1/D1A6
- D3 pad 53: Net-(D3-Pad38) -> /Lattice MACHXO2/Digit Drivers/S3R
- D3 pad 54: Net-(D3-Pad39) -> /Lattice MACHXO2/Digit Drivers/S3G
- D3 pad 55: /Lattice MACHXO2/Digit_1/D1A1 -> /Lattice MACHXO2/Digit Drivers/Digit 1/D1A1
- D3 pad 56: Net-(D3-Pad56) -> /Lattice MACHXO2/Digit Drivers/S4R
- D3 pad 57: Net-(D3-Pad57) -> /Lattice MACHXO2/Digit Drivers/S4G
- D3 pad 58: /Lattice MACHXO2/Digit_1/D1A2 -> /Lattice MACHXO2/Digit Drivers/Digit 1/D1A2
- D3 pad 59: Net-(D3-Pad56) -> /Lattice MACHXO2/Digit Drivers/S4R
- D3 pad 6: Net-(D3-Pad12) -> /Lattice MACHXO2/Digit Drivers/S1G
- D3 pad 60: Net-(D3-Pad57) -> /Lattice MACHXO2/Digit Drivers/S4G
- D3 pad 61: /Lattice MACHXO2/Digit_1/D1A3 -> /Lattice MACHXO2/Digit Drivers/Digit 1/D1A3
- D3 pad 62: Net-(D3-Pad56) -> /Lattice MACHXO2/Digit Drivers/S4R
- D3 pad 63: Net-(D3-Pad57) -> /Lattice MACHXO2/Digit Drivers/S4G
- D3 pad 64: /Lattice MACHXO2/Digit_1/D1A4 -> /Lattice MACHXO2/Digit Drivers/Digit 1/D1A4
- D3 pad 65: Net-(D3-Pad56) -> /Lattice MACHXO2/Digit Drivers/S4R
- D3 pad 66: Net-(D3-Pad57) -> /Lattice MACHXO2/Digit Drivers/S4G
- D3 pad 67: /Lattice MACHXO2/Digit_1/D1A5 -> /Lattice MACHXO2/Digit Drivers/Digit 1/D1A5
- D3 pad 68: Net-(D3-Pad56) -> /Lattice MACHXO2/Digit Drivers/S4R
- D3 pad 69: Net-(D3-Pad57) -> /Lattice MACHXO2/Digit Drivers/S4G
- D3 pad 7: /Lattice MACHXO2/Digit_1/D1A3 -> /Lattice MACHXO2/Digit Drivers/Digit 1/D1A3
- D3 pad 70: /Lattice MACHXO2/Digit_1/D1A6 -> /Lattice MACHXO2/Digit Drivers/Digit 1/D1A6
- D3 pad 71: Net-(D3-Pad56) -> /Lattice MACHXO2/Digit Drivers/S4R
- D3 pad 72: Net-(D3-Pad57) -> /Lattice MACHXO2/Digit Drivers/S4G
- D3 pad 73: /Lattice MACHXO2/Digit_1/D1A1 -> /Lattice MACHXO2/Digit Drivers/Digit 1/D1A1
- D3 pad 74: Net-(D3-Pad74) -> /Lattice MACHXO2/Digit Drivers/S5R
- D3 pad 75: Net-(D3-Pad75) -> /Lattice MACHXO2/Digit Drivers/S5G
- D3 pad 76: /Lattice MACHXO2/Digit_1/D1A2 -> /Lattice MACHXO2/Digit Drivers/Digit 1/D1A2
- D3 pad 77: Net-(D3-Pad74) -> /Lattice MACHXO2/Digit Drivers/S5R
- D3 pad 78: Net-(D3-Pad75) -> /Lattice MACHXO2/Digit Drivers/S5G
- D3 pad 79: /Lattice MACHXO2/Digit_1/D1A3 -> /Lattice MACHXO2/Digit Drivers/Digit 1/D1A3
- D3 pad 8: Net-(D3-Pad11) -> /Lattice MACHXO2/Digit Drivers/S1R
- D3 pad 80: Net-(D3-Pad74) -> /Lattice MACHXO2/Digit Drivers/S5R
- D3 pad 81: Net-(D3-Pad75) -> /Lattice MACHXO2/Digit Drivers/S5G
- D3 pad 82: /Lattice MACHXO2/Digit_1/D1A4 -> /Lattice MACHXO2/Digit Drivers/Digit 1/D1A4
- D3 pad 83: Net-(D3-Pad74) -> /Lattice MACHXO2/Digit Drivers/S5R
- D3 pad 84: Net-(D3-Pad75) -> /Lattice MACHXO2/Digit Drivers/S5G
- D3 pad 85: /Lattice MACHXO2/Digit_1/D1A5 -> /Lattice MACHXO2/Digit Drivers/Digit 1/D1A5
- D3 pad 86: Net-(D3-Pad74) -> /Lattice MACHXO2/Digit Drivers/S5R
- D3 pad 87: Net-(D3-Pad75) -> /Lattice MACHXO2/Digit Drivers/S5G
- D3 pad 88: /Lattice MACHXO2/Digit_1/D1A6 -> /Lattice MACHXO2/Digit Drivers/Digit 1/D1A6
- D3 pad 89: Net-(D3-Pad74) -> /Lattice MACHXO2/Digit Drivers/S5R
- D3 pad 9: Net-(D3-Pad12) -> /Lattice MACHXO2/Digit Drivers/S1G
- D3 pad 90: Net-(D3-Pad75) -> /Lattice MACHXO2/Digit Drivers/S5G
- D3 pad 91: /Lattice MACHXO2/Digit_1/D1A1 -> /Lattice MACHXO2/Digit Drivers/Digit 1/D1A1
- D3 pad 92: Net-(D3-Pad101) -> /Lattice MACHXO2/Digit Drivers/S6R
- D3 pad 93: Net-(D3-Pad102) -> /Lattice MACHXO2/Digit Drivers/S6G
- D3 pad 94: /Lattice MACHXO2/Digit_1/D1A2 -> /Lattice MACHXO2/Digit Drivers/Digit 1/D1A2
- D3 pad 95: Net-(D3-Pad101) -> /Lattice MACHXO2/Digit Drivers/S6R
- D3 pad 96: Net-(D3-Pad102) -> /Lattice MACHXO2/Digit Drivers/S6G
- D3 pad 97: /Lattice MACHXO2/Digit_1/D1A3 -> /Lattice MACHXO2/Digit Drivers/Digit 1/D1A3
- D3 pad 98: Net-(D3-Pad101) -> /Lattice MACHXO2/Digit Drivers/S6R
- D3 pad 99: Net-(D3-Pad102) -> /Lattice MACHXO2/Digit Drivers/S6G
- Q10 pad 1: GND -> Net-(Q10-Pad1)
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Routing:
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
Commit message: PCB work.
Parts:
- moved D1 164.8 mm to (102.5, 31.7)
- moved C3 164.8 mm to (93.9, 38.3)
- moved C5 164.8 mm to (93.4, 32.3)
- moved C6 164.8 mm to (89.1, 38.3)
- moved R4 164.8 mm to (84.2, 32.3)
- moved C1 164.8 mm to (88.9, 44.3)
- moved C2 164.8 mm to (98.2, 32.3)
- moved C4 164.8 mm to (84.3, 44.3)
- moved C7 164.8 mm to (84.3, 38.3)
- moved D2 164.8 mm to (92.9, 43.7)
- moved Q1 164.8 mm to (98.2, 37.6)
- moved R1 164.8 mm to (88.8, 32.3)
- moved R2 164.8 mm to (79.7, 44.3)
- moved R3 164.8 mm to (108.2, 31.8)
- moved R5 164.8 mm to (79.7, 38.3)
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Routing:
- net /Lattice MACHXO2/Digit Drivers/Digit 1/D1A4: track 439.9 -> 588.2 mm
- net /Lattice MACHXO2/Digit Drivers/Digit 1/D1A5: track 447.2 -> 591.3 mm
- net /Lattice MACHXO2/Digit Drivers/Digit 1/D1A3: track 259.2 -> 399.5 mm
- net /Lattice MACHXO2/Digit Drivers/Digit 1/D1A2: track 217.2 -> 351.2 mm
- net /Lattice MACHXO2/Digit Drivers/Digit 1/D1A1: track 159.0 -> 262.8 mm
- net /Lattice MACHXO2/Digit Drivers/Digit 1/D1A6: track 408.9 -> 494.7 mm
