File: PCB_1.1/Digit2.sch (KiCad schematic (older format))
At the start: 37 parts, among them Q2 DMN2041LSD-13, Q3 DMN2041LSD-13, Q33 DMN2041LSD-13, Q34 DMN2041LSD-13, Q35 DMN2041LSD-13, Q4 DMN2041LSD-13, Q5 DMN2041LSD-13, Q6 DMN2041LSD-13, Q7 DMN2041LSD-13, Q8 DMN2041LSD-13

Commit message: PCB work.
Parts:
- removed Q2, Q3, Q4, Q5, Q6, Q7, Q8: DMN2041LSD-13, Power_Integrations:SO-8, symbol DMN2041LSD-13
- removed Q33, Q34, Q35: DMN2041LSD-13, SO-8, symbol DMN2041LSD-13
- removed R10, R11, R12, R13, R14, R15, R16, R17, R18, R19, R20, R7, R75, R76, R79, R8, R80, R83, R84, R9: 10K, Resistors_SMD:R_0603_HandSoldering, symbol R
- removed R77, R78, R81, R82, R85, R86: 150, Resistors_SMD:R_0603_HandSoldering, symbol R
Connections:
- net labels removed: +5V, A1, A2, A3, A4, A5, A6, D2S1G, D2S1R, D2S2G, D2S2R, D2S3G, D2S3R, D2S4G, D2S4R, D2S5G, D2S5R, D2S6G, D2S6R, D2S7G, D2S7R, GND
- wire segments 293 -> 152

Commit message: PCB work.
Connections:
- net labels added: D2S1G, D2S1R, D2S2G, D2S2R, D2S3G, D2S3R, D2S4G, D2S4R, D2S5G, D2S5R, D2S6G, D2S6R, D2S7G, D2S7R
- wire segments 152 -> 158
